File: Slave/V1/Isolated_BMS_Slave_Front_End.sch (KiCad schematic (older format))
At the start: 25 parts, among them J501 649002227222, Q501 CPH6347-TL-W, Q502 CPH6347-TL-W, U501 LTV-816S, U502 SI8641AB-B-IS1

Commit message: front end done
Connections:
- net AGND: now also C503.1
Changed lines of the file:
@@
 AR Path="/59400152/591B47DF" Ref="Q2501"  Part="1"
 AR Path="/59400D56/591B47DF" Ref="Q2901"  Part="1"
-F 0 "Q1301" V 3300 1300 60  0000 C CNN
+F 0 "Q501" V 3300 1300 60  0000 C CNN
 F 1 "CPH6347-TL-W" V 3200 1200 60  0000 C CNN
 F 2 "IC:TSOT-23-6" H 3000 400 60  0001 C CNN
@@
 AR Path="/59400152/591D60B1" Ref="U2502"  Part="1"
 AR Path="/59400D56/591D60B1" Ref="U2902"  Part="1"
-F 0 "U1302" H 6200 5400 60  0000 C CNN
+F 0 "U502" H 6200 5400 60  0000 C CNN
 F 1 "SI8641AB-B-IS1" H 6200 3750 60  0000 C CNN
 F 2 "IC:SOIC-16" H 6200 2800 60  0001 C CNN
@@
 AR Path="/59400152/591D614C" Ref="C2502"  Part="1"
 AR Path="/59400D56/591D614C" Ref="C2902"  Part="1"
-F 0 "C1302" H 7050 4060 60  0000 C CNN
+F 0 "C502" H 7050 4060 60  0000 C CNN
 F 1 "885012207098" H 7050 3550 60  0001 C CNN
 F 2 "Capacitors:C0805" H 7050 2950 60  0001 C CNN
@@
 AR Path="/59400152/591D641D" Ref="C2501"  Part="1"
 AR Path="/59400D56/591D641D" Ref="C2901"  Part="1"
-F 0 "C1301" H 5350 4060 60  0000 C CNN
+F 0 "C501" H 5350 4060 60  0000 C CNN
 F 1 "885012207098" H 5350 3550 60  0001 C CNN
 F 2 "Capacitors:C0805" H 5350 2950 60  0001 C CNN
@@
 AR Path="/59400152/591D91BB" Ref="R2513"  Part="1"
 AR Path="/59400D56/591D91BB" Ref="R2913"  Part="1"
-F 0 "R1313" H 4700 5380 60  0000 C CNN
+F 0 "R513" H 4700 5380 60  0000 C CNN
 F 1 "RC0805JR-074K7L" H 4700 5000 50  0001 C CNN
 F 2 "Resistors:R0805" H 4700 4400 30  0001 C CNN
@@
 AR Path="/59400152/591D91D0" Ref="C2504"  Part="1"
 AR Path="/59400D56/591D91D0" Ref="C2904"  Part="1"
-F 0 "C1304" H 4950 5660 60  0000 C CNN
+F 0 "C504" H 4950 5660 60  0000 C CNN
 F 1 "885012207098" H 4950 5150 60  0001 C CNN
 F 2 "Capacitors:C0805" H 4950 4550 60  0001 C CNN
@@
 AR Path="/59400152/5938F00C" Ref="Q2502"  Part="1"
 AR Path="/59400D56/5938F00C" Ref="Q2902"  Part="1"
-F 0 "Q1302" V 4500 1300 60  0000 C CNN
+F 0 "Q502" V 4500 1300 60  0000 C CNN
 F 1 "CPH6347-TL-W" V 4400 1200 60  0000 C CNN
 F 2 "IC:TSOT-23-6" H 4200 400 60  0001 C CNN
@@
 AR Path="/59400152/593917FE" Ref="R2512"  Part="1"
 AR Path="/59400D56/593917FE" Ref="R2912"  Part="1"
-F 0 "R1312" H 3800 5280 60  0000 C CNN
+F 0 "R512" H 3800 5280 60  0000 C CNN
 F 1 "RC0805JR-074K7L" H 3800 4900 50  0001 C CNN
 F 2 "Resistors:R0805" H 3800 4300 30  0001 C CNN
@@
 AR Path="/59400152/593919F1" Ref="R2509"  Part="1"
 AR Path="/59400D56/593919F1" Ref="R2909"  Part="1"
-F 0 "R1309" H 4300 4980 60  0000 C CNN
+F 0 "R509" H 4300 4980 60  0000 C CNN
 F 1 "RC0805JR-07100RL" H 4300 4600 50  0001 C CNN
 F 2 "Resistors:R0805" H 4300 4000 30  0001 C CNN
@@
 AR Path="/59400152/59391AB0" Ref="R2507"  Part="1"
 AR Path="/59400D56/59391AB0" Ref="R2907"  Part="1"
-F 0 "R1307" H 4700 4780 60  0000 C CNN
+F 0 "R507" H 4700 4780 60  0000 C CNN
 F 1 "RC0805JR-07100RL" H 4700 4400 50  0001 C CNN
 F 2 "Resistors:R0805" H 4700 3800 30  0001 C CNN
@@
 AR Path="/59400152/59391AED" Ref="R2505"  Part="1"
 AR Path="/59400D56/59391AED" Ref="R2905"  Part="1"
-F 0 "R1305" H 4300 4580 60  0000 C CNN
+F 0 "R505" H 4300 4580 60  0000 C CNN
 F 1 "RC0805JR-07100RL" H 4300 4200 50  0001 C CNN
 F 2 "Resistors:R0805" H 4300 3600 30  0001 C CNN
@@
 AR Path="/59400152/59392BA0" Ref="R2504"  Part="1"
 AR Path="/59400D56/59392BA0" Ref="R2904"  Part="1"
-F 0 "R1304" H 7400 4380 60  0000 C CNN
+F 0 "R504" H 7400 4380 60  0000 C CNN
 F 1 "RC0805JR-07100RL" H 7400 4000 50  0001 C CNN
 F 2 "Resistors:R0805" H 7400 3400 30  0001 C CNN
@@
 AR Path="/59400152/593932C5" Ref="R2506"  Part="1"
 AR Path="/59400D56/593932C5" Ref="R2906"  Part="1"
-F 0 "R1306" H 7000 4580 60  0000 C CNN
+F 0 "R506" H 7000 4580 60  0000 C CNN
 F 1 "RC0805JR-07100RL" H 7000 4200 50  0001 C CNN
 F 2 "Resistors:R0805" H 7000 3600 30  0001 C CNN
@@
 AR Path="/59400152/593934E8" Ref="R2508"  Part="1"
 AR Path="/59400D56/593934E8" Ref="R2908"  Part="1"
-F 0 "R1308" H 7400 4780 60  0000 C CNN
+F 0 "R508" H 7400 4780 60  0000 C CNN
 F 1 "RC0805JR-07100RL" H 7400 4400 50  0001 C CNN
 F 2 "Resistors:R0805" H 7400 3800 30  0001 C CNN
@@
 AR Path="/59400152/59395C7C" Ref="U2501"  Part="1"
 AR Path="/59400D56/59395C7C" Ref="U2901"  Part="1"
-F 0 "U1301" H 4100 2500 60  0000 C CNN
+F 0 "U501" H 4100 2500 60  0000 C CNN
 F 1 "LTV-816S" H 4100 2000 60  0000 C CNN
 F 2 "IC:4-SMD" H 4100 1300 60  0001 C CNN
@@
 AR Path="/59400152/59396188" Ref="R2503"  Part="1"
 AR Path="/59400D56/59396188" Ref="R2903"  Part="1"
-F 0 "R1303" H 4700 2080 60  0000 C CNN
+F 0 "R503" H 4700 2080 60  0000 C CNN
 F 1 "RC0805JR-07330RL" H 4700 1700 50  0001 C CNN
 F 2 "Resistors:R0805" H 4700 1100 30  0001 C CNN
@@
 AR Path="/59400152/5939743F" Ref="D2502"  Part="1"
 AR Path="/59400D56/5939743F" Ref="D2902"  Part="1"
-F 0 "D1302" H 3150 2350 60  0000 C CNN
+F 0 "D502" H 3150 2350 60  0000 C CNN
 F 1 "NSR0530HT1G" H 3200 2050 60  0000 C CNN
 F 2 "Diodes:SOD-323" H 3180 1200 60  0001 C CNN
@@
 AR Path="/59400152/5939A33B" Ref="C2503"  Part="1"
 AR Path="/59400D56/5939A33B" Ref="C2903"  Part="1"
-F 0 "C1303" H 7650 5460 60  0000 C CNN
+F 0 "C503" H 7650 5460 60  0000 C CNN
 F 1 "885012207080" H 7650 4950 60  0001 C CNN
 F 2 "Capacitors:C0805" H 7650 4350 60  0001 C CNN
@@
 AR Path="/59400152/59397104" Ref="R2502"  Part="1"
 AR Path="/59400D56/59397104" Ref="R2902"  Part="1"
-F 0 "R1302" H 3500 1580 60  0000 C CNN
+F 0 "R502" H 3500 1580 60  0000 C CNN
 F 1 "RC0805JR-07470KL" H 3500 1200 50  0001 C CNN
 F 2 "Resistors:R0805" H 3500 600 30  0001 C CNN
@@
 AR Path="/59400152/593A1551" Ref="D2501"  Part="1"
 AR Path="/59400D56/593A1551" Ref="D2901"  Part="1"
-F 0 "D1301" H 1950 2050 60  0000 C CNN
+F 0 "D501" H 1950 2050 60  0000 C CNN
 F 1 "150080RS75000" H 2000 1700 60  0001 C CNN
 F 2 "Diodes:LED_0805_RED" H 2010 820 60  0001 C CNN
@@
 AR Path="/59400152/593A2339" Ref="R2501"  Part="1"
 AR Path="/59400D56/593A2339" Ref="R2901"  Part="1"
-F 0 "R1301" H 2000 1580 60  0000 C CNN
+F 0 "R501" H 2000 1580 60  0000 C CNN
 F 1 "RC0805JR-071KL" H 2000 1200 50  0001 C CNN
 F 2 "Resistors:R0805" H 2000 600 30  0001 C CNN
@@
 AR Path="/59400152/593D0FB3" Ref="R2510"  Part="1"
 AR Path="/59400D56/593D0FB3" Ref="R2910"  Part="1"
-F 0 "R1310" H 7000 4980 60  0000 C CNN
+F 0 "R510" H 7000 4980 60  0000 C CNN
 F 1 "RC0805JR-074K7L" H 7000 4600 50  0001 C CNN
 F 2 "Resistors:R0805" H 7000 4000 30  0001 C CNN
@@
 AR Path="/59400152/593D1688" Ref="R2511"  Part="1"
 AR Path="/59400D56/593D1688" Ref="R2911"  Part="1"
-F 0 "R1311" H 8000 5180 60  0000 C CNN
+F 0 "R511" H 8000 5180 60  0000 C CNN
 F 1 "RC0805JR-074K7L" H 8000 4800 50  0001 C CNN
 F 2 "Resistors:R0805" H 8000 4200 30  0001 C CNN
@@
 AR Path="/59400152/593D16CF" Ref="R2514"  Part="1"
 AR Path="/59400D56/593D16CF" Ref="R2914"  Part="1"
-F 0 "R1314" H 7300 5480 60  0000 C CNN
+F 0 "R514" H 7300 5480 60  0000 C CNN
 F 1 "RC0805JR-07470KL" H 7300 5100 50  0001 C CNN
 F 2 "Resistors:R0805" H 7300 4500 30  0001 C CNN
@@
 AR Path="/59400152/593D9852" Ref="J2501"  Part="1"
 AR Path="/59400D56/593D9852" Ref="J2901"  Part="1"
-F 0 "J1301" H 800 1500 60  0000 C CNN
+F 0 "J501" H 800 1500 60  0000 C CNN
 F 1 "649002227222" H 900 1100 60  0000 C CNN
 F 2 "Connectors:649002227222" H 800 400 60  0001 C CNN
@@
 Wire Wire Line
 	5600 3600 5600 3900
+Connection ~ 7700 5700
 $EndSCHEMATC
