File: Slave/V1/balancing.sch (KiCad schematic (older format))
At the start: 10 parts, among them Q401 CPH6347-TL-W, Q402 BSS806NH6327XTSA1, U401 ADCMP350YKSZ-REEL7

Commit message: clear annotation
Parts:
- renumbered C401 to C?, D401 to D?, Q402 to Q?, Q401 to Q?, R401 to R?, R403 to R?, R405 to R?, R402 to R?, R404 to R?, U401 to U?
Connections:
- net GND: now also D?.1 (Cathode); no longer D?.2 (Cathode)
Changed lines of the file:
@@
 Vin
 $Comp
-L BSS806NH6327XTSA1 Q402
+L BSS806NH6327XTSA1 Q?
 U 1 1 591DDB89
 P 4200 4200
-F 0 "Q402" H 3800 4400 60  0000 C CNN
+F 0 "Q?" H 3800 4400 60  0000 C CNN
 F 1 "BSS806NH6327XTSA1" H 3700 4300 60  0000 C CNN
 F 2 "IC:SOT-23-3" H 4350 3300 60  0001 C CNN
@@
 	4300 5400 4300 4500
 $Comp
-L CPH6347-TL-W Q401
+L CPH6347-TL-W Q?
 U 1 1 591DE34E
 P 4500 2800
-F 0 "Q401" H 5500 2900 60  0000 C CNN
+F 0 "Q?" H 5500 2900 60  0000 C CNN
 F 1 "CPH6347-TL-W" H 5200 3000 60  0000 C CNN
 F 2 "IC:TSOT-23-6" H 4600 1900 60  0001 C CNN
@@
 $EndComp
 $Comp
-L ADCMP350YKSZ-REEL7 U401
+L ADCMP350YKSZ-REEL7 U?
 U 1 1 591DE79A
 P 6400 3700
-F 0 "U401" H 6400 3900 60  0000 C CNN
+F 0 "U?" H 6400 3900 60  0000 C CNN
 F 1 "ADCMP350YKSZ-REEL7" H 6400 3450 60  0000 C CNN
 F 2 "IC:SC70-4" H 6400 2800 60  0001 C CNN
@@
 $EndComp
 $Comp
-L BGND #PWR040
+L BGND #PWR?
 U 1 1 591DE86C
 P 6400 3100
-F 0 "#PWR040" H 6400 2930 50  0001 C CNN
+F 0 "#PWR?" H 6400 2930 50  0001 C CNN
 F 1 "BGND" H 6400 3000 50  0000 C CNN
 F 2 "" H 6400 3200 60  0000 C CNN
@@
 Vin
 $Comp
-L 885012207098 C401
+L 885012207098 C?
 U 1 1 591DE88A
 P 6100 2900
-F 0 "C401" H 6050 3060 60  0000 C CNN
+F 0 "C?" H 6050 3060 60  0000 C CNN
 F 1 "885012207098" H 6050 2550 60  0001 C CNN
 F 2 "Capacitors:C0805" H 6050 1950 60  0001 C CNN
@@
 	7100 3800 7100 4400
 $Comp
-L RC0805JR-07470KL R401
+L RC0805JR-07470KL R?
 U 1 1 591DEB54
 P 5200 2500
-F 0 "R401" H 5200 2580 60  0000 C CNN
+F 0 "R?" H 5200 2580 60  0000 C CNN
 F 1 "RC0805JR-07470KL" H 5200 2200 50  0001 C CNN
 F 2 "Resistors:R0805" H 5200 1600 30  0001 C CNN
@@
 	6700 3600 7600 3600
 $Comp
-L 352210RJT R403
+L 352210RJT R?
 U 1 1 591DF793
 P 4300 3600
-F 0 "R403" H 4300 3680 60  0000 C CNN
+F 0 "R?" H 4300 3680 60  0000 C CNN
 F 1 "352210RJT" H 4300 3300 50  0001 C CNN
 F 2 "Resistors:R2512" H 4300 2700 30  0001 C CNN
@@
 	3200 4200 4000 4200
 $Comp
-L RC0805JR-076K8L R405
+L RC0805JR-076K8L R?
 U 1 1 591DF8F9
 P 3000 4200
-F 0 "R405" H 3000 4280 60  0000 C CNN
+F 0 "R?" H 3000 4280 60  0000 C CNN
 F 1 "RC0805JR-076K8L" H 3000 3900 50  0001 C CNN
 F 2 "Resistors:R0805" H 3000 3300 30  0001 C CNN
@@
 	2600 4200 2800 4200
 $Comp
-L MMBZ12VALT1G D401
+L MMBZ12VALT1G D?
 U 1 1 591DFFE8
 P 3700 4500
-F 0 "D401" H 3700 4700 60  0000 C CNN
+F 0 "D?" H 3700 4700 60  0000 C CNN
 F 1 "MMBZ12VALT1G" H 3400 4300 60  0000 C CNN
 F 2 "IC:SOT-23-3" H 3710 3310 60  0001 C CNN
@@
 $EndComp
 $Comp
-L MMBZ12VALT1G D401
-U 2 1 591E0165
+L MMBZ12VALT1G D?
+U 1 1 591E0165
 P 3700 5000
-F 0 "D401" H 3600 4800 60  0000 C CNN
+F 0 "D?" H 3600 4800 60  0000 C CNN
 F 1 "MMBZ12VALT1G" H 3700 4850 60  0001 C CNN
 F 2 "IC:SOT-23-3" H 3710 3810 60  0001 C CNN
@@
 F 8 "TVS DIODE 8.5VWM 17VC SOT23" H 3710 3910 60  0001 C CNN "Description"
 F 9 "11.4V" H 3700 4750 60  0001 C CNN "Voltage - Breakdown (Min)"
-	2    3700 5000
+	1    3700 5000
 	0    1    1    0
 $EndComp
@@
 Connection ~ 4300 5200
 $Comp
-L Resistor_Generic R402
+L Resistor_Generic R?
 U 1 1 591E091E
 P 7600 3300
-F 0 "R402" H 7600 3400 60  0000 C CNN
+F 0 "R?" H 7600 3400 60  0000 C CNN
 F 1 "Resistor_Generic" H 7650 3000 50  0001 C CNN
 F 2 "Resistors:R0805" H 7650 2400 30  0001 C CNN
@@
 $EndComp
 $Comp
-L Resistor_Generic R404
+L Resistor_Generic R?
 U 1 1 591E0A2D
 P 7600 3900
-F 0 "R404" H 7600 4000 60  0000 C CNN
+F 0 "R?" H 7600 4000 60  0000 C CNN
 F 1 "Resistor_Generic" H 7650 3600 50  0001 C CNN
 F 2 "Resistors:R0805" H 7650 3000 30  0001 C CNN

Commit message: add notes
Other:
- note added: "Mettre LED en || avec la load"
Changed lines of the file:
@@
 Text HLabel 7600 4700 2    60   Input ~ 0
 GND
+Text Notes 2700 3500 0    60   ~ 0
+Mettre LED en || avec la load
 $EndSCHEMATC

Commit message: add LED to reverse protection + balancing
Parts:
- added D?: 150080RS75000, Diodes:LED_0805_RED, symbol 150080RS75000
- added R?: RC0805JR-071KL, Resistors:R0805, symbol RC0805JR-071KL
Connections:
- net at Q?.3 (D), R?.1: now also D?.1 (Cathode)
- net at Q?.1 (D), Q?.2 (D), Q?.5 (D)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: now also R?.1
- new net: D?.2 (Anode), R?.2
Other:
- note added: "Circuit de protection pour\nque le P-MOSFET soit OFF \nlorsque Vin < 3.8V \n"
- note removed: "Circuit de protection pour\nque le P-MOSFET soit OFF \nlorsque Vin < 3.6V \n(Resistance a calculer)\n"
- note removed: "Mettre LED en || avec la load"
- moved on the sheet: D?A, Q?, R?

Commit message: placing components
Parts:
- removed D?: 150080RS75000, Diodes:LED_0805_RED, symbol 150080RS75000
- removed R? (x2): Resistor_Generic, Resistors:R0805, symbol Resistor_Generic
- added D801: 150080VS75000, Diodes:LED_0805_GREEN, symbol 150080VS75000
- added R803: RC0805JR-07560KL, Resistors:R0805, symbol RC0805JR-07560KL
- added R805: RC0805JR-07100KL, Resistors:R0805, symbol RC0805JR-07100KL
- gave numbers to parts that had none: 9
Connections:
- net GND: now also D802.2 (Cathode), R805.1; no longer D802.1 (Cathode)
- net Vin: now also R803.2
- net at Q802.3 (D), R804.1: now also D801.1 (Cathode)
- net at U801.1 (Vin): now also R803.1, R805.2
- net at R802.2: now also D801.2 (Anode)
Changed lines of the file:
@@
 Vin
 $Comp
-L BSS806NH6327XTSA1 Q?
+L BSS806NH6327XTSA1 Q802
 U 1 1 591DDB89
 P 4200 4300
-F 0 "Q?" H 3800 4500 60  0000 C CNN
+F 0 "Q802" H 3800 4500 60  0000 C CNN
 F 1 "BSS806NH6327XTSA1" H 3700 4400 60  0000 C CNN
 F 2 "IC:SOT-23-3" H 4350 3400 60  0001 C CNN
@@
 $EndComp
 Wire Wire Line
-	4300 4600 4300 5300
-Wire Wire Line
-	4300 5300 4300 5500
-$Comp
-L CPH6347-TL-W Q?
+	4300 4600 4300 5500
+$Comp
+L CPH6347-TL-W Q801
 U 1 1 591DE34E
 P 4500 2800
-F 0 "Q?" H 5500 2900 60  0000 C CNN
+F 0 "Q801" H 5500 2900 60  0000 C CNN
 F 1 "CPH6347-TL-W" H 5200 3000 60  0000 C CNN
 F 2 "IC:TSOT-23-6" H 4600 1900 60  0001 C CNN
@@
 $EndComp
 $Comp
-L ADCMP350YKSZ-REEL7 U?
+L ADCMP350YKSZ-REEL7 U801
 U 1 1 591DE79A
 P 6400 3700
-F 0 "U?" H 6400 3900 60  0000 C CNN
+F 0 "U801" H 6400 3900 60  0000 C CNN
 F 1 "ADCMP350YKSZ-REEL7" H 6400 3450 60  0000 C CNN
 F 2 "IC:SC70-4" H 6400 2800 60  0001 C CNN
@@
 $EndComp
 $Comp
-L BGND #PWR?
+L BGND #PWR063
 U 1 1 591DE86C
 P 6400 3100
-F 0 "#PWR?" H 6400 2930 50  0001 C CNN
+F 0 "#PWR063" H 6400 2930 50  0001 C CNN
 F 1 "BGND" H 6400 3000 50  0000 C CNN
 F 2 "" H 6400 3200 60  0000 C CNN
@@
 Vin
 $Comp
-L 885012207098 C?
+L 885012207098 C801
 U 1 1 591DE88A
 P 6100 2900
-F 0 "C?" H 6050 3060 60  0000 C CNN
+F 0 "C801" H 6050 3060 60  0000 C CNN
 F 1 "885012207098" H 6050 2550 60  0001 C CNN
 F 2 "Capacitors:C0805" H 6050 1950 60  0001 C CNN
@@
 $EndComp
 Wire Wire Line
-	5600 2900 5800 2900
-Wire Wire Line
-	5800 2900 5900 2900
+	5600 2900 5900 2900
 Wire Wire Line
 	6200 2900 6400 2900
@@
 	6700 3800 7100 3800
 Wire Wire Line
-	7100 3800 7100 4200
-Wire Wire Line
-	7100 4200 7100 4400
-$Comp
-L RC0805JR-07470KL R?
+	7100 3800 7100 4400
+$Comp
+L RC0805JR-07470KL R801
 U 1 1 591DEB54
 P 5200 2500
-F 0 "R?" H 5200 2580 60  0000 C CNN
+F 0 "R801" H 5200 2580 60  0000 C CNN
 F 1 "RC0805JR-07470KL" H 5200 2200 50  0001 C CNN
 F 2 "Resistors:R0805" H 5200 1600 30  0001 C CNN
@@
 	4400 2500 4400 2200
 Wire Wire Line
-	4200 2200 4400 2200
-Wire Wire Line
-	4400 2200 5200 2200
+	4200 2200 5200 2200
 Wire Wire Line
 	5200 2200 5200 2300
@@
 	4700 2800 5200 2800
 Wire Wire Line
-	5200 2700 5200 2800
-Wire Wire Line
-	5200 2800 5200 3800
+	5200 2700 5200 3800
 Connection ~ 5200 2800
 Connection ~ 4400 2200
@@
 	6700 3600 7600 3600
 $Comp
-L 352210RJT R?
+L 352210RJT R804
 U 1 1 591DF793
 P 4300 3600
-F 0 "R?" H 4300 3680 60  0000 C CNN
+F 0 "R804" H 4300 3680 60  0000 C CNN
 F 1 "352210RJT" H 4300 3300 50  0001 C CNN
 F 2 "Resistors:R2512" H 4300 2700 30  0001 C CNN
@@
 $EndComp
 Wire Wire Line
-	4300 3100 4300 3200
-Wire Wire Line
-	4300 3200 4300 3300
-Wire Wire Line
-	4300 3300 4300 3400
+	4300 3100 4300 3400
 Wire Wire Line
 	4400 3100 4400 3200
 Wire Wire Line
-	4300 3200 4400 3200
-Wire Wire Line
-	4400 3200 4500 3200
-Wire Wire Line
-	4500 3200 4600 3200
+	4300 3200 4600 3200
 Connection ~ 4300 3200
 Wire Wire Line
@@
 Connection ~ 4500 3200
 Wire Wire Line
-	4300 3800 4300 3900
-Wire Wire Line
-	4300 3900 4300 4000
-Wire Wire Line
-	3200 4300 3700 4300
-Wire Wire Line
-	3700 4300 4000 4300
-$Comp
-L RC0805JR-076K8L R?
+	4300 3800 4300 4000
+Wire Wire Line
+	3200 4300 4000 4300
+$Comp
+L RC0805JR-076K8L R806
 U 1 1 591DF8F9
 P 3000 4300
-F 0 "R?" H 3000 4380 60  0000 C CNN
+F 0 "R806" H 3000 4380 60  0000 C CNN
 F 1 "RC0805JR-076K8L" H 3000 4000 50  0001 C CNN
 F 2 "Resistors:R0805" H 3000 3400 30  0001 C CNN
@@
 	2600 4300 2800 4300
 $Comp
-L MMBZ12VALT1G D?
+L MMBZ12VALT1G D802
 U 1 1 591DFFE8
 P 3700 4600
-F 0 "D?" H 3700 4800 60  0000 C CNN
+F 0 "D802" H 3700 4800 60  0000 C CNN
 F 1 "MMBZ12VALT1G" H 3400 4400 60  0000 C CNN
 F 2 "IC:SOT-23-3" H 3710 3410 60  0001 C CNN
@@
 $EndComp
 $Comp
-L MMBZ12VALT1G D?
-U 1 1 591E0165
+L MMBZ12VALT1G D802
+U 2 1 591E0165
 P 3700 5100
-F 0 "D?" H 3600 4900 60  0000 C CNN
+F 0 "D802" H 3600 4900 60  0000 C CNN
 F 1 "MMBZ12VALT1G" H 3700 4950 60  0001 C CNN
 F 2 "IC:SOT-23-3" H 3710 3910 60  0001 C CNN
@@
 F 8 "TVS DIODE 8.5VWM 17VC SOT23" H 3710 4010 60  0001 C CNN "Description"
 F 9 "11.4V" H 3700 4850 60  0001 C CNN "Voltage - Breakdown (Min)"
-	1    3700 5100
+	2    3700 5100
 	0    1    1    0
 $EndComp
@@
 	3700 5300 4300 5300
 Connection ~ 4300 5300
-$Comp
-L Resistor_Generic R?
-U 1 1 591E091E
-P 7600 3300
-F 0 "R?" H 7600 3400 60  0000 C CNN
-F 1 "Resistor_Generic" H 7650 3000 50  0001 C CNN
-F 2 "Resistors:R0805" H 7650 2400 30  0001 C CNN
-F 3 "D" H 7650 2350 30  0001 C CNN
-F 4 "Supplier" H 7650 2900 60  0001 C CNN "Supplier"
-F 5 "Supplier Part Number" H 7650 2800 60  0001 C CNN "Supplier Part Number"
-F 6 "Manufacturer" H 7650 2700 60  0001 C CNN "Manufacturer"
-F 7 "Manufacturer Part Number" H 7650 2600 60  0001 C CNN "Manufacturer Part Number"
-F 8 "Description" H 7650 2500 60  0001 C CNN "Description"
-F 9 "Resistance" H 7600 3220 50  0000 C CNN "Resistance (Ohms)"
-F 10 "Puissance" H 7600 3100 50  0001 C CNN "Puissance (Watts)"
-F 11 "Tolerance" H 7600 3160 50  0001 C CNN "Tolerance (%)"
-	1    7600 3300
-	0    -1   -1   0
-$EndComp
-$Comp
-L Resistor_Generic R?
-U 1 1 591E0A2D
-P 7600 3900
-F 0 "R?" H 7600 4000 60  0000 C CNN
-F 1 "Resistor_Generic" H 7650 3600 50  0001 C CNN
-F 2 "Resistors:R0805" H 7650 3000 30  0001 C CNN
-F 3 "D" H 7650 2950 30  0001 C CNN
-F 4 "Supplier" H 7650 3500 60  0001 C CNN "Supplier"
-F 5 "Supplier Part Number" H 7650 3400 60  0001 C CNN "Supplier Part Number"
-F 6 "Manufacturer" H 7650 3300 60  0001 C CNN "Manufacturer"
-F 7 "Manufacturer Part Number" H 7650 3200 60  0001 C CNN "Manufacturer Part Number"
-F 8 "Description" H 7650 3100 60  0001 C CNN "Description"
-F 9 "Resistance" H 7600 3820 50  0000 C CNN "Resistance (Ohms)"
-F 10 "Puissance" H 7600 3700 50  0001 C CNN "Puissance (Watts)"
-F 11 "Tolerance" H 7600 3760 50  0001 C CNN "Tolerance (%)"
-	1    7600 3900
-	0    -1   -1   0
-$EndComp
 Wire Wire Line
 	7600 4100 7600 4200
@@
 Connection ~ 7100 4200
 Wire Wire Line
-	7600 3500 7600 3600
-Wire Wire Line
-	7600 3600 7600 3700
+	7600 3500 7600 3700
 Connection ~ 7600 3600
 Text HLabel 7400 3000 0    60   Input ~ 0
@@
 GND
 $Comp
-L RC0805JR-071KL R?
+L RC0805JR-071KL R802
 U 1 1 593A32C1
 P 3800 3300
-F 0 "R?" H 3800 3380 60  0000 C CNN
+F 0 "R802" H 3800 3380 60  0000 C CNN
 F 1 "RC0805JR-071KL" H 3800 3000 50  0001 C CNN
 F 2 "Resistors:R0805" H 3800 2400 30  0001 C CNN
@@
 	-1   0    0    -1
 $EndComp
-$Comp
-L 150080RS75000 D?
-U 1 1 593A3338
+Wire Wire Line
+	3400 3500 3400 3300
+Wire Wire Line
+	3400 3300 3600 3300
+Wire Wire Line
+	4000 3300 4300 3300
+Connection ~ 4300 3300
+Wire Wire Line
+	3400 3800 3400 3900
+Wire Wire Line
+	3400 3900 4300 3900
+Connection ~ 4300 3900
+$Comp
+L RC0805JR-07100KL R805
+U 1 1 593E2823
+P 7600 3900
+F 0 "R805" H 7600 3980 60  0000 C CNN
+F 1 "RC0805JR-07100KL" H 7600 3600 50  0001 C CNN
+F 2 "Resistors:R0805" H 7600 3000 30  0001 C CNN
+F 3 "http://www.yageo.com/documents/recent/PYu-RC_Group_51_RoHS_L_7.pdf" H 7600 2950 30  0001 C CNN
+F 4 "Digikey" H 7600 3500 60  0001 C CNN "Supplier"
+F 5 "311-100KARCT-ND" H 7600 3400 60  0001 C CNN "Supplier Part Number"
+F 6 "Yageo" H 7600 3300 60  0001 C CNN "Manufacturer"
+F 7 "RC0805JR-07100KL" H 7600 3200 60  0001 C CNN "Manufacturer Part Number"
+F 8 "RES SMD 100K OHM 5% 1/8W 0805" H 7600 3100 60  0001 C CNN "Description"
+F 9 "100k" H 7600 3830 50  0000 C CNN "Resistance (Ohms)"
+F 10 "±5%" H 8010 3820 50  0001 C CNN "Tolerance (%)"
+F 11 "1/8W" H 7600 3760 50  0001 C CNN "Puissance (Watts)"
+	1    7600 3900
+	0    -1   -1   0
+$EndComp
+$Comp
+L RC0805JR-07560KL R803
+U 1 1 593E4220
+P 7600 3300
+F 0 "R803" H 7600 3380 60  0000 C CNN
+F 1 "RC0805JR-07560KL" H 7600 3000 50  0001 C CNN
+F 2 "Resistors:R0805" H 7600 2400 30  0001 C CNN
+F 3 "http://www.yageo.com/documents/recent/PYu-RC_Group_51_RoHS_L_7.pdf" H 7600 2350 30  0001 C CNN
+F 4 "Digikey" H 7600 2900 60  0001 C CNN "Supplier"
+F 5 "311-560KARCT-ND" H 7600 2800 60  0001 C CNN "Supplier Part Number"
+F 6 "Yageo" H 7600 2700 60  0001 C CNN "Manufacturer"
+F 7 "RC0805JR-07560KL" H 7600 2600 60  0001 C CNN "Manufacturer Part Number"
+F 8 "RES SMD 560K OHM 5% 1/8W 0805" H 7600 2500 60  0001 C CNN "Description"
+F 9 "560k" H 7600 3230 50  0000 C CNN "Resistance (Ohms)"
+F 10 "±5%" H 8010 3220 50  0001 C CNN "Tolerance (%)"
+F 11 "1/8W" H 7600 3160 50  0001 C CNN "Puissance (Watts)"
+	1    7600 3300
+	0    -1   -1   0
+$EndComp
+$Comp
+L 150080VS75000 D801
+U 1 1 593E53C5
 P 3400 3700
-F 0 "D?" H 3350 3850 60  0000 C CNN
-F 1 "150080RS75000" H 3400 3500 60  0001 C CNN
-F 2 "Diodes:LED_0805_RED" H 3410 2620 60  0001 C CNN
-F 3 "http://katalog.we-online.de/led/datasheet/150080RS75000.pdf" H 3410 2520 60  0001 C CNN
+F 0 "D801" H 3350 3850 60  0000 C CNN
+F 1 "150080VS75000" H 3400 3500 60  0001 C CNN
+F 2 "Diodes:LED_0805_GREEN" H 3410 2620 60  0001 C CNN
+F 3 "http://katalog.we-online.de/led/datasheet/150080VS75000.pdf" H 3410 2520 60  0001 C CNN
 F 4 "Digikey" H 3410 3120 60  0001 C CNN "Supplier"
-F 5 "732-4984-1-ND" H 3410 3020 60  0001 C CNN "Supplier Part Number"
+F 5 "732-4986-1-ND" H 3410 3020 60  0001 C CNN "Supplier Part Number"
 F 6 "Wurth Electronics Inc." H 3410 2920 60  0001 C CNN "Manufacturer"
-F 7 "150080RS75000" H 3410 2820 60  0001 C CNN "Manufacturer Part Number"
-F 8 "LED RED CLEAR 0805 SMD" H 3410 2720 60  0001 C CNN "Description"
-F 9 "RED" H 3300 3500 60  0000 C CNN "Color"
+F 7 "150080VS75000" H 3410 2820 60  0001 C CNN "Manufacturer Part Number"
+F 8 "LED GREEN CLEAR 0805 SMD" H 3410 2720 60  0001 C CNN "Description"
+F 9 "GREEN" H 3400 3500 60  0000 C CNN "Color"
 F 10 "2V" H 3400 3300 60  0001 C CNN "Voltage - Forward (Vf) (Typ)"
 	1    3400 3700
 	0    -1   1    0
 $EndComp
-Wire Wire Line
-	3400 3500 3400 3300
-Wire Wire Line
-	3400 3300 3600 3300
-Wire Wire Line
-	4000 3300 4300 3300
-Connection ~ 4300 3300
-Wire Wire Line
-	3400 3800 3400 3900
-Wire Wire Line
-	3400 3900 4300 3900
-Connection ~ 4300 3900
 $EndSCHEMATC

Commit message: adding 8 front end
Connections:
- net BGND is gone; now on net GND: C801.2
- net GND: now also D802.1 (Cathode); no longer D802.2 (Cathode)
Changed lines of the file:
@@
 $Descr A4 11693 8268
 encoding utf-8
-Sheet 8 8
+Sheet 16 16
 Title "Isolated BMS Slave Front End"
 Date ""
@@
 U 1 1 591DDB89
 P 4200 4300
-F 0 "Q802" H 3800 4500 60  0000 C CNN
+AR Path="/5938E2BF/591D23A3/591DDB89" Ref="Q802"  Part="1"
+AR Path="/593ED6BB/591D23A3/591DDB89" Ref="Q1202"  Part="1"
+AR Path="/593EFAB4/591D23A3/591DDB89" Ref="Q1602"  Part="1"
+AR Path="/593F9F72/591D23A3/591DDB89" Ref="Q1202"  Part="1"
+AR Path="/593FDFB1/591D23A3/591DDB89" Ref="Q?"  Part="1"
+F 0 "Q?" H 3800 4500 60  0000 C CNN
 F 1 "BSS806NH6327XTSA1" H 3700 4400 60  0000 C CNN
 F 2 "IC:SOT-23-3" H 4350 3400 60  0001 C CNN
@@
 U 1 1 591DE34E
 P 4500 2800
-F 0 "Q801" H 5500 2900 60  0000 C CNN
+AR Path="/5938E2BF/591D23A3/591DE34E" Ref="Q801"  Part="1"
+AR Path="/593ED6BB/591D23A3/591DE34E" Ref="Q1201"  Part="1"
+AR Path="/593EFAB4/591D23A3/591DE34E" Ref="Q1601"  Part="1"
+AR Path="/593F9F72/591D23A3/591DE34E" Ref="Q1201"  Part="1"
+AR Path="/593FDFB1/591D23A3/591DE34E" Ref="Q?"  Part="1"
+F 0 "Q?" H 5500 2900 60  0000 C CNN
 F 1 "CPH6347-TL-W" H 5200 3000 60  0000 C CNN
 F 2 "IC:TSOT-23-6" H 4600 1900 60  0001 C CNN
@@
 U 1 1 591DE79A
 P 6400 3700
-F 0 "U801" H 6400 3900 60  0000 C CNN
+AR Path="/5938E2BF/591D23A3/591DE79A" Ref="U801"  Part="1"
+AR Path="/593ED6BB/591D23A3/591DE79A" Ref="U1201"  Part="1"
+AR Path="/593EFAB4/591D23A3/591DE79A" Ref="U1601"  Part="1"
+AR Path="/593F9F72/591D23A3/591DE79A" Ref="U1201"  Part="1"
+AR Path="/593FDFB1/591D23A3/591DE79A" Ref="U?"  Part="1"
+F 0 "U?" H 6400 3900 60  0000 C CNN
 F 1 "ADCMP350YKSZ-REEL7" H 6400 3450 60  0000 C CNN
 F 2 "IC:SC70-4" H 6400 2800 60  0001 C CNN
@@
 	-1   0    0    -1
 $EndComp
-$Comp
-L BGND #PWR060
-U 1 1 591DE86C
-P 6400 3100
-F 0 "#PWR060" H 6400 2930 50  0001 C CNN
-F 1 "BGND" H 6400 3000 50  0000 C CNN
-F 2 "" H 6400 3200 60  0000 C CNN
-F 3 "" H 6380 3010 60  0000 C CNN
-	1    6400 3100
-	1    0    0    -1
-$EndComp
 Text HLabel 5600 2900 0    60   Input ~ 0
 Vin
@@
 U 1 1 591DE88A
 P 6100 2900
-F 0 "C801" H 6050 3060 60  0000 C CNN
+AR Path="/5938E2BF/591D23A3/591DE88A" Ref="C801"  Part="1"
+AR Path="/593ED6BB/591D23A3/591DE88A" Ref="C1201"  Part="1"
+AR Path="/593EFAB4/591D23A3/591DE88A" Ref="C1601"  Part="1"
+AR Path="/593F9F72/591D23A3/591DE88A" Ref="C1201"  Part="1"
+AR Path="/593FDFB1/591D23A3/591DE88A" Ref="C?"  Part="1"
+F 0 "C?" H 6050 3060 60  0000 C CNN
 F 1 "885012207098" H 6050 2550 60  0001 C CNN
 F 2 "Capacitors:C0805" H 6050 1950 60  0001 C CNN
@@
 	6200 2900 6400 2900
 Wire Wire Line
-	6400 2900 6400 3000
-Wire Wire Line
 	6100 3600 5800 3600
 Wire Wire Line
@@
 U 1 1 591DEB54
 P 5200 2500
-F 0 "R801" H 5200 2580 60  0000 C CNN
+AR Path="/5938E2BF/591D23A3/591DEB54" Ref="R801"  Part="1"
+AR Path="/593ED6BB/591D23A3/591DEB54" Ref="R1201"  Part="1"
+AR Path="/593EFAB4/591D23A3/591DEB54" Ref="R1601"  Part="1"
+AR Path="/593F9F72/591D23A3/591DEB54" Ref="R1201"  Part="1"
+AR Path="/593FDFB1/591D23A3/591DEB54" Ref="R?"  Part="1"
+F 0 "R?" H 5200 2580 60  0000 C CNN
 F 1 "RC0805JR-07470KL" H 5200 2200 50  0001 C CNN
 F 2 "Resistors:R0805" H 5200 1600 30  0001 C CNN
@@
 U 1 1 591DF793
 P 4300 3600
-F 0 "R804" H 4300 3680 60  0000 C CNN
+AR Path="/5938E2BF/591D23A3/591DF793" Ref="R804"  Part="1"
+AR Path="/593ED6BB/591D23A3/591DF793" Ref="R1204"  Part="1"
+AR Path="/593EFAB4/591D23A3/591DF793" Ref="R1604"  Part="1"
+AR Path="/593F9F72/591D23A3/591DF793" Ref="R1204"  Part="1"
+AR Path="/593FDFB1/591D23A3/591DF793" Ref="R?"  Part="1"
+F 0 "R?" H 4300 3680 60  0000 C CNN
 F 1 "352210RJT" H 4300 3300 50  0001 C CNN
 F 2 "Resistors:R2512" H 4300 2700 30  0001 C CNN
@@
 U 1 1 591DF8F9
 P 3000 4300
-F 0 "R806" H 3000 4380 60  0000 C CNN
+AR Path="/5938E2BF/591D23A3/591DF8F9" Ref="R806"  Part="1"
+AR Path="/593ED6BB/591D23A3/591DF8F9" Ref="R1206"  Part="1"
+AR Path="/593EFAB4/591D23A3/591DF8F9" Ref="R1606"  Part="1"
+AR Path="/593F9F72/591D23A3/591DF8F9" Ref="R1206"  Part="1"
+AR Path="/593FDFB1/591D23A3/591DF8F9" Ref="R?"  Part="1"
+F 0 "R?" H 3000 4380 60  0000 C CNN
 F 1 "RC0805JR-076K8L" H 3000 4000 50  0001 C CNN
 F 2 "Resistors:R0805" H 3000 3400 30  0001 C CNN
@@
 U 1 1 591DFFE8
 P 3700 4600
-F 0 "D802" H 3700 4800 60  0000 C CNN
+AR Path="/5938E2BF/591D23A3/591DFFE8" Ref="D802"  Part="1"
+AR Path="/593ED6BB/591D23A3/591DFFE8" Ref="D1202"  Part="1"
+AR Path="/593EFAB4/591D23A3/591DFFE8" Ref="D1602"  Part="1"
+AR Path="/593F9F72/591D23A3/591DFFE8" Ref="D1202"  Part="1"
+AR Path="/593FDFB1/591D23A3/591DFFE8" Ref="D?"  Part="1"
+F 0 "D?" H 3700 4800 60  0000 C CNN
 F 1 "MMBZ12VALT1G" H 3400 4400 60  0000 C CNN
 F 2 "IC:SOT-23-3" H 3710 3410 60  0001 C CNN
@@
 $Comp
 L MMBZ12VALT1G D802
-U 2 1 591E0165
+U 1 1 591E0165
 P 3700 5100
-F 0 "D802" H 3600 4900 60  0000 C CNN
+AR Path="/5938E2BF/591D23A3/591E0165" Ref="D802"  Part="2"
+AR Path="/593ED6BB/591D23A3/591E0165" Ref="D1202"  Part="2"
+AR Path="/593EFAB4/591D23A3/591E0165" Ref="D1602"  Part="2"
+AR Path="/593F9F72/591D23A3/591E0165" Ref="D1202"  Part="2"
+AR Path="/593FDFB1/591D23A3/591E0165" Ref="D?"  Part="1"
+F 0 "D?" H 3600 4900 60  0000 C CNN
 F 1 "MMBZ12VALT1G" H 3700 4950 60  0001 C CNN
 F 2 "IC:SOT-23-3" H 3710 3910 60  0001 C CNN
@@
 F 8 "TVS DIODE 8.5VWM 17VC SOT23" H 3710 4010 60  0001 C CNN "Description"
 F 9 "11.4V" H 3700 4850 60  0001 C CNN "Voltage - Breakdown (Min)"
-	2    3700 5100
+	1    3700 5100
 	0    1    1    0
 $EndComp
@@
 U 1 1 593A32C1
 P 3800 3300
-F 0 "R802" H 3800 3380 60  0000 C CNN
+AR Path="/5938E2BF/591D23A3/593A32C1" Ref="R802"  Part="1"
+AR Path="/593ED6BB/591D23A3/593A32C1" Ref="R1202"  Part="1"
+AR Path="/593EFAB4/591D23A3/593A32C1" Ref="R1602"  Part="1"
+AR Path="/593F9F72/591D23A3/593A32C1" Ref="R1202"  Part="1"
+AR Path="/593FDFB1/591D23A3/593A32C1" Ref="R?"  Part="1"
+F 0 "R?" H 3800 3380 60  0000 C CNN
 F 1 "RC0805JR-071KL" H 3800 3000 50  0001 C CNN
 F 2 "Resistors:R0805" H 3800 2400 30  0001 C CNN
@@
 U 1 1 593E2823
 P 7600 3900
-F 0 "R805" H 7600 3980 60  0000 C CNN
+AR Path="/5938E2BF/591D23A3/593E2823" Ref="R805"  Part="1"
+AR Path="/593ED6BB/591D23A3/593E2823" Ref="R1205"  Part="1"
+AR Path="/593EFAB4/591D23A3/593E2823" Ref="R1605"  Part="1"
+AR Path="/593F9F72/591D23A3/593E2823" Ref="R1205"  Part="1"
+AR Path="/593FDFB1/591D23A3/593E2823" Ref="R?"  Part="1"
+F 0 "R?" H 7600 3980 60  0000 C CNN
 F 1 "RC0805JR-07100KL" H 7600 3600 50  0001 C CNN
 F 2 "Resistors:R0805" H 7600 3000 30  0001 C CNN
@@
 U 1 1 593E4220
 P 7600 3300
-F 0 "R803" H 7600 3380 60  0000 C CNN
+AR Path="/5938E2BF/591D23A3/593E4220" Ref="R803"  Part="1"
+AR Path="/593ED6BB/591D23A3/593E4220" Ref="R1203"  Part="1"
+AR Path="/593EFAB4/591D23A3/593E4220" Ref="R1603"  Part="1"
+AR Path="/593F9F72/591D23A3/593E4220" Ref="R1203"  Part="1"
+AR Path="/593FDFB1/591D23A3/593E4220" Ref="R?"  Part="1"
+F 0 "R?" H 7600 3380 60  0000 C CNN
 F 1 "RC0805JR-07560KL" H 7600 3000 50  0001 C CNN
 F 2 "Resistors:R0805" H 7600 2400 30  0001 C CNN
@@
 U 1 1 593E53C5
 P 3400 3700
-F 0 "D801" H 3350 3850 60  0000 C CNN
+AR Path="/5938E2BF/591D23A3/593E53C5" Ref="D801"  Part="1"
+AR Path="/593ED6BB/591D23A3/593E53C5" Ref="D1201"  Part="1"
+AR Path="/593EFAB4/591D23A3/593E53C5" Ref="D1601"  Part="1"
+AR Path="/593F9F72/591D23A3/593E53C5" Ref="D1201"  Part="1"
+AR Path="/593FDFB1/591D23A3/593E53C5" Ref="D?"  Part="1"
+F 0 "D?" H 3350 3850 60  0000 C CNN
 F 1 "150080VS75000" H 3400 3500 60  0001 C CNN
 F 2 "Diodes:LED_0805_GREEN" H 3410 2620 60  0001 C CNN
@@
 	0    -1   1    0
 $EndComp
+Text Label 6400 3100 0    60   ~ 0
+GND
+Wire Wire Line
+	6400 2900 6400 3100
+Wire Wire Line
+	6400 3100 6600 3100
 $EndSCHEMATC

Commit message: placed front end 1 to 5
Connections:
- net GND: now also D802.2 (Cathode); no longer D802.1 (Cathode)
- net Drain_P_Mosfet: now reaches Q801.1 (D), Q801.2 (D), Q801.5 (D), Q801.6 (D), R802.1, R804.2
