File: Slave/V1/balancing.sch (KiCad schematic (older format))
At the start: 12 parts, among them Q801 CPH6347-TL-W, Q802 BSS806NH6327XTSA1, U801 ADCMP350YKSZ-REEL7

Commit message: front end done
Changed lines of the file:
@@
 AR Path="/59400D56/591D23A3/591DDB89" Ref="Q3202"  Part="1"
 AR Path="/59400D60/591D23A3/591DDB89" Ref="Q3602"  Part="1"
-F 0 "Q802" H 3800 4500 60  0000 C CNN
+F 0 "Q3602" H 3800 4500 60  0000 C CNN
 F 1 "BSS806NH6327XTSA1" H 3700 4400 60  0000 C CNN
 F 2 "IC:SOT-23-3" H 4350 3400 60  0001 C CNN
@@
 AR Path="/59400D56/591D23A3/591DE34E" Ref="Q3201"  Part="1"
 AR Path="/59400D60/591D23A3/591DE34E" Ref="Q3601"  Part="1"
-F 0 "Q801" H 5500 2900 60  0000 C CNN
+F 0 "Q3601" H 5500 2900 60  0000 C CNN
 F 1 "CPH6347-TL-W" H 5200 3000 60  0000 C CNN
 F 2 "IC:TSOT-23-6" H 4600 1900 60  0001 C CNN
@@
 AR Path="/59400D56/591D23A3/591DE79A" Ref="U3201"  Part="1"
 AR Path="/59400D60/591D23A3/591DE79A" Ref="U3601"  Part="1"
-F 0 "U801" H 6400 3900 60  0000 C CNN
+F 0 "U3601" H 6400 3900 60  0000 C CNN
 F 1 "ADCMP350YKSZ-REEL7" H 6400 3450 60  0000 C CNN
 F 2 "IC:SC70-4" H 6400 2800 60  0001 C CNN
@@
 AR Path="/59400D56/591D23A3/591DE88A" Ref="C3201"  Part="1"
 AR Path="/59400D60/591D23A3/591DE88A" Ref="C3601"  Part="1"
-F 0 "C801" H 6050 3060 60  0000 C CNN
+F 0 "C3601" H 6050 3060 60  0000 C CNN
 F 1 "885012207098" H 6050 2550 60  0001 C CNN
 F 2 "Capacitors:C0805" H 6050 1950 60  0001 C CNN
@@
 AR Path="/59400D56/591D23A3/591DEB54" Ref="R3201"  Part="1"
 AR Path="/59400D60/591D23A3/591DEB54" Ref="R3601"  Part="1"
-F 0 "R801" H 5200 2580 60  0000 C CNN
+F 0 "R3601" H 5200 2580 60  0000 C CNN
 F 1 "RC0805JR-07470KL" H 5200 2200 50  0001 C CNN
 F 2 "Resistors:R0805" H 5200 1600 30  0001 C CNN
@@
 AR Path="/59400D56/591D23A3/591DF793" Ref="R3204"  Part="1"
 AR Path="/59400D60/591D23A3/591DF793" Ref="R3604"  Part="1"
-F 0 "R804" H 4300 3680 60  0000 C CNN
+F 0 "R3604" H 4300 3680 60  0000 C CNN
 F 1 "352210RJT" H 4300 3300 50  0001 C CNN
 F 2 "Resistors:R2512" H 4300 2700 30  0001 C CNN
@@
 AR Path="/59400D56/591D23A3/591DF8F9" Ref="R3206"  Part="1"
 AR Path="/59400D60/591D23A3/591DF8F9" Ref="R3606"  Part="1"
-F 0 "R806" H 3000 4380 60  0000 C CNN
+F 0 "R3606" H 3000 4380 60  0000 C CNN
 F 1 "RC0805JR-076K8L" H 3000 4000 50  0001 C CNN
 F 2 "Resistors:R0805" H 3000 3400 30  0001 C CNN
@@
 AR Path="/59400D56/591D23A3/591DFFE8" Ref="D3202"  Part="1"
 AR Path="/59400D60/591D23A3/591DFFE8" Ref="D3602"  Part="1"
-F 0 "D802" H 3700 4800 60  0000 C CNN
+F 0 "D3602" H 3700 4800 60  0000 C CNN
 F 1 "MMBZ12VALT1G" H 3400 4400 60  0000 C CNN
 F 2 "IC:SOT-23-3" H 3710 3410 60  0001 C CNN
@@
 AR Path="/59400D56/591D23A3/591E0165" Ref="D3202"  Part="2"
 AR Path="/59400D60/591D23A3/591E0165" Ref="D3602"  Part="2"
-F 0 "D802" H 3600 4900 60  0000 C CNN
+F 0 "D3602" H 3600 4900 60  0000 C CNN
 F 1 "MMBZ12VALT1G" H 3700 4950 60  0001 C CNN
 F 2 "IC:SOT-23-3" H 3710 3910 60  0001 C CNN
@@
 AR Path="/59400D56/591D23A3/593A32C1" Ref="R3202"  Part="1"
 AR Path="/59400D60/591D23A3/593A32C1" Ref="R3602"  Part="1"
-F 0 "R802" H 3800 3380 60  0000 C CNN
+F 0 "R3602" H 3800 3380 60  0000 C CNN
 F 1 "RC0805JR-071KL" H 3800 3000 50  0001 C CNN
 F 2 "Resistors:R0805" H 3800 2400 30  0001 C CNN
@@
 AR Path="/59400D56/591D23A3/593E2823" Ref="R3205"  Part="1"
 AR Path="/59400D60/591D23A3/593E2823" Ref="R3605"  Part="1"
-F 0 "R805" H 7600 3980 60  0000 C CNN
+F 0 "R3605" H 7600 3980 60  0000 C CNN
 F 1 "RC0805JR-07100KL" H 7600 3600 50  0001 C CNN
 F 2 "Resistors:R0805" H 7600 3000 30  0001 C CNN
@@
 AR Path="/59400D56/591D23A3/593E4220" Ref="R3203"  Part="1"
 AR Path="/59400D60/591D23A3/593E4220" Ref="R3603"  Part="1"
-F 0 "R803" H 7600 3380 60  0000 C CNN
+F 0 "R3603" H 7600 3380 60  0000 C CNN
 F 1 "RC0805JR-07560KL" H 7600 3000 50  0001 C CNN
 F 2 "Resistors:R0805" H 7600 2400 30  0001 C CNN
@@
 AR Path="/59400D56/591D23A3/593E53C5" Ref="D3201"  Part="1"
 AR Path="/59400D60/591D23A3/593E53C5" Ref="D3601"  Part="1"
-F 0 "D801" H 3350 3850 60  0000 C CNN
+F 0 "D3601" H 3350 3850 60  0000 C CNN
 F 1 "150080VS75000" H 3400 3500 60  0001 C CNN
 F 2 "Diodes:LED_0805_GREEN" H 3410 2620 60  0001 C CNN
