File: Slave/V1/voltage_reading.sch (KiCad schematic (older format))
At the start: 5 parts, among them U301 ADC121S021CIMF/NOPB

Commit message: clear annotation
Parts:
- renumbered C302 to C?, C301 to C?, C303 to C?, R301 to R?, U301 to U?
Changed lines of the file:
@@
 $EndDescr
 $Comp
-L 885012207098 C302
+L 885012207098 C?
 U 1 1 591B6F4E
 P 5400 3300
-F 0 "C302" H 5350 3460 60  0000 C CNN
+F 0 "C?" H 5350 3460 60  0000 C CNN
 F 1 "885012207098" H 5350 2950 60  0001 C CNN
 F 2 "Capacitors:C0805" H 5350 2350 60  0001 C CNN
@@
 $EndComp
 $Comp
-L 885012107015 C301
+L 885012107015 C?
 U 1 1 591B6FC1
 P 5400 2900
-F 0 "C301" H 5350 3060 60  0000 C CNN
+F 0 "C?" H 5350 3060 60  0000 C CNN
 F 1 "885012107015" H 5350 2550 60  0001 C CNN
 F 2 "Capacitors:C0805" H 5350 1950 60  0001 C CNN
@@
 $EndComp
 $Comp
-L RC0805JR-07100RL R301
+L RC0805JR-07100RL R?
 U 1 1 591BAB3B
 P 4100 4000
-F 0 "R301" H 4100 4080 60  0000 C CNN
+F 0 "R?" H 4100 4080 60  0000 C CNN
 F 1 "RC0805JR-07100RL" H 4100 3700 50  0001 C CNN
 F 2 "Resistors:R0805" H 4100 3100 30  0001 C CNN
@@
 $EndComp
 $Comp
-L 885012207047 C303
+L 885012207047 C?
 U 1 1 591BB052
 P 4500 4200
-F 0 "C303" H 4450 4360 60  0000 C CNN
+F 0 "C?" H 4450 4360 60  0000 C CNN
 F 1 "885012207047" H 4450 3850 60  0001 C CNN
 F 2 "Capacitors:C0805" H 4450 3250 60  0001 C CNN
@@
 VCell
 $Comp
-L ADC121S021CIMF/NOPB U301
+L ADC121S021CIMF/NOPB U?
 U 1 1 591D3EBF
 P 5500 4000
-F 0 "U301" H 5500 4300 60  0000 C CNN
+F 0 "U?" H 5500 4300 60  0000 C CNN
 F 1 "ADC121S021CIMF/NOPB" H 5550 3640 60  0000 C CNN
 F 2 "IC:SOT-23-6" H 5500 2800 60  0001 C CNN

Commit message: placing components
Parts:
- gave numbers to parts that had none: 5
Changed lines of the file:
@@
 $EndDescr
 $Comp
-L 885012207098 C?
+L 885012207098 C702
 U 1 1 591B6F4E
 P 5400 3300
-F 0 "C?" H 5350 3460 60  0000 C CNN
+F 0 "C702" H 5350 3460 60  0000 C CNN
 F 1 "885012207098" H 5350 2950 60  0001 C CNN
 F 2 "Capacitors:C0805" H 5350 2350 60  0001 C CNN
@@
 $EndComp
 $Comp
-L 885012107015 C?
+L 885012107015 C701
 U 1 1 591B6FC1
 P 5400 2900
-F 0 "C?" H 5350 3060 60  0000 C CNN
+F 0 "C701" H 5350 3060 60  0000 C CNN
 F 1 "885012107015" H 5350 2550 60  0001 C CNN
 F 2 "Capacitors:C0805" H 5350 1950 60  0001 C CNN
@@
 $EndComp
 $Comp
-L RC0805JR-07100RL R?
+L RC0805JR-07100RL R701
 U 1 1 591BAB3B
 P 4100 4000
-F 0 "R?" H 4100 4080 60  0000 C CNN
+F 0 "R701" H 4100 4080 60  0000 C CNN
 F 1 "RC0805JR-07100RL" H 4100 3700 50  0001 C CNN
 F 2 "Resistors:R0805" H 4100 3100 30  0001 C CNN
@@
 $EndComp
 $Comp
-L 885012207047 C?
+L 885012207047 C703
 U 1 1 591BB052
 P 4500 4200
-F 0 "C?" H 4450 4360 60  0000 C CNN
+F 0 "C703" H 4450 4360 60  0000 C CNN
 F 1 "885012207047" H 4450 3850 60  0001 C CNN
 F 2 "Capacitors:C0805" H 4450 3250 60  0001 C CNN
@@
 VCell
 $Comp
-L ADC121S021CIMF/NOPB U?
+L ADC121S021CIMF/NOPB U701
 U 1 1 591D3EBF
 P 5500 4000
-F 0 "U?" H 5500 4300 60  0000 C CNN
+F 0 "U701" H 5500 4300 60  0000 C CNN
 F 1 "ADC121S021CIMF/NOPB" H 5550 3640 60  0000 C CNN
 F 2 "IC:SOT-23-6" H 5500 2800 60  0001 C CNN

Commit message: placed front end 1 to 5
Changed lines of the file:
@@
 $Descr USLetter 11000 8500
 encoding utf-8
-Sheet 15 16
+Sheet 15 36
 Title "Isolated BMS Slave Front End"
 Date ""
@@
 AR Path="/593EFAB4/591D0796/591B6F4E" Ref="C1502"  Part="1"
 AR Path="/593F9F72/591D0796/591B6F4E" Ref="C1102"  Part="1"
-AR Path="/593FDFB1/591D0796/591B6F4E" Ref="C?"  Part="1"
-F 0 "C?" H 5350 3460 60  0000 C CNN
+AR Path="/593FDFB1/591D0796/591B6F4E" Ref="C1502"  Part="1"
+AR Path="/593FF1B1/591D0796/591B6F4E" Ref="C1902"  Part="1"
+AR Path="/593FF93E/591D0796/591B6F4E" Ref="C2302"  Part="1"
+AR Path="/59400152/591D0796/591B6F4E" Ref="C2702"  Part="1"
+AR Path="/59400D56/591D0796/591B6F4E" Ref="C3102"  Part="1"
+AR Path="/59400D60/591D0796/591B6F4E" Ref="C3502"  Part="1"
+F 0 "C1502" H 5350 3460 60  0000 C CNN
 F 1 "885012207098" H 5350 2950 60  0001 C CNN
 F 2 "Capacitors:C0805" H 5350 2350 60  0001 C CNN
@@
 AR Path="/593EFAB4/591D0796/591B6FC1" Ref="C1501"  Part="1"
 AR Path="/593F9F72/591D0796/591B6FC1" Ref="C1101"  Part="1"
-AR Path="/593FDFB1/591D0796/591B6FC1" Ref="C?"  Part="1"
-F 0 "C?" H 5350 3060 60  0000 C CNN
+AR Path="/593FDFB1/591D0796/591B6FC1" Ref="C1501"  Part="1"
+AR Path="/593FF1B1/591D0796/591B6FC1" Ref="C1901"  Part="1"
+AR Path="/593FF93E/591D0796/591B6FC1" Ref="C2301"  Part="1"
+AR Path="/59400152/591D0796/591B6FC1" Ref="C2701"  Part="1"
+AR Path="/59400D56/591D0796/591B6FC1" Ref="C3101"  Part="1"
+AR Path="/59400D60/591D0796/591B6FC1" Ref="C3501"  Part="1"
+F 0 "C1501" H 5350 3060 60  0000 C CNN
 F 1 "885012107015" H 5350 2550 60  0001 C CNN
 F 2 "Capacitors:C0805" H 5350 1950 60  0001 C CNN
@@
 AR Path="/593EFAB4/591D0796/591BAB3B" Ref="R1501"  Part="1"
 AR Path="/593F9F72/591D0796/591BAB3B" Ref="R1101"  Part="1"
-AR Path="/593FDFB1/591D0796/591BAB3B" Ref="R?"  Part="1"
-F 0 "R?" H 4100 4080 60  0000 C CNN
+AR Path="/593FDFB1/591D0796/591BAB3B" Ref="R1501"  Part="1"
+AR Path="/593FF1B1/591D0796/591BAB3B" Ref="R1901"  Part="1"
+AR Path="/593FF93E/591D0796/591BAB3B" Ref="R2301"  Part="1"
+AR Path="/59400152/591D0796/591BAB3B" Ref="R2701"  Part="1"
+AR Path="/59400D56/591D0796/591BAB3B" Ref="R3101"  Part="1"
+AR Path="/59400D60/591D0796/591BAB3B" Ref="R3501"  Part="1"
+F 0 "R1501" H 4100 4080 60  0000 C CNN
 F 1 "RC0805JR-07100RL" H 4100 3700 50  0001 C CNN
 F 2 "Resistors:R0805" H 4100 3100 30  0001 C CNN
@@
 AR Path="/593EFAB4/591D0796/591BB052" Ref="C1503"  Part="1"
 AR Path="/593F9F72/591D0796/591BB052" Ref="C1103"  Part="1"
-AR Path="/593FDFB1/591D0796/591BB052" Ref="C?"  Part="1"
-F 0 "C?" H 4450 4360 60  0000 C CNN
+AR Path="/593FDFB1/591D0796/591BB052" Ref="C1503"  Part="1"
+AR Path="/593FF1B1/591D0796/591BB052" Ref="C1903"  Part="1"
+AR Path="/593FF93E/591D0796/591BB052" Ref="C2303"  Part="1"
+AR Path="/59400152/591D0796/591BB052" Ref="C2703"  Part="1"
+AR Path="/59400D56/591D0796/591BB052" Ref="C3103"  Part="1"
+AR Path="/59400D60/591D0796/591BB052" Ref="C3503"  Part="1"
+F 0 "C1503" H 4450 4360 60  0000 C CNN
 F 1 "885012207047" H 4450 3850 60  0001 C CNN
 F 2 "Capacitors:C0805" H 4450 3250 60  0001 C CNN
@@
 AR Path="/593EFAB4/591D0796/591D3EBF" Ref="U1501"  Part="1"
 AR Path="/593F9F72/591D0796/591D3EBF" Ref="U1101"  Part="1"
-AR Path="/593FDFB1/591D0796/591D3EBF" Ref="U?"  Part="1"
-F 0 "U?" H 5500 4300 60  0000 C CNN
+AR Path="/593FDFB1/591D0796/591D3EBF" Ref="U1501"  Part="1"
+AR Path="/593FF1B1/591D0796/591D3EBF" Ref="U1901"  Part="1"
+AR Path="/593FF93E/591D0796/591D3EBF" Ref="U2301"  Part="1"
+AR Path="/59400152/591D0796/591D3EBF" Ref="U2701"  Part="1"
+AR Path="/59400D56/591D0796/591D3EBF" Ref="U3101"  Part="1"
+AR Path="/59400D60/591D0796/591D3EBF" Ref="U3501"  Part="1"
+F 0 "U1501" H 5500 4300 60  0000 C CNN
 F 1 "ADC121S021CIMF/NOPB" H 5550 3640 60  0000 C CNN
 F 2 "IC:SOT-23-6" H 5500 2800 60  0001 C CNN

Commit message: front end done
Changed lines of the file:
@@
 AR Path="/59400D56/591D0796/591B6F4E" Ref="C3102"  Part="1"
 AR Path="/59400D60/591D0796/591B6F4E" Ref="C3502"  Part="1"
-F 0 "C1502" H 5350 3460 60  0000 C CNN
+F 0 "C3102" H 5350 3460 60  0000 C CNN
 F 1 "885012207098" H 5350 2950 60  0001 C CNN
 F 2 "Capacitors:C0805" H 5350 2350 60  0001 C CNN
@@
 AR Path="/59400D56/591D0796/591B6FC1" Ref="C3101"  Part="1"
 AR Path="/59400D60/591D0796/591B6FC1" Ref="C3501"  Part="1"
-F 0 "C1501" H 5350 3060 60  0000 C CNN
+F 0 "C3101" H 5350 3060 60  0000 C CNN
 F 1 "885012107015" H 5350 2550 60  0001 C CNN
 F 2 "Capacitors:C0805" H 5350 1950 60  0001 C CNN
@@
 AR Path="/59400D56/591D0796/591BAB3B" Ref="R3101"  Part="1"
 AR Path="/59400D60/591D0796/591BAB3B" Ref="R3501"  Part="1"
-F 0 "R1501" H 4100 4080 60  0000 C CNN
+F 0 "R3101" H 4100 4080 60  0000 C CNN
 F 1 "RC0805JR-07100RL" H 4100 3700 50  0001 C CNN
 F 2 "Resistors:R0805" H 4100 3100 30  0001 C CNN
@@
 AR Path="/59400D56/591D0796/591BB052" Ref="C3103"  Part="1"
 AR Path="/59400D60/591D0796/591BB052" Ref="C3503"  Part="1"
-F 0 "C1503" H 4450 4360 60  0000 C CNN
+F 0 "C3103" H 4450 4360 60  0000 C CNN
 F 1 "885012207047" H 4450 3850 60  0001 C CNN
 F 2 "Capacitors:C0805" H 4450 3250 60  0001 C CNN
@@
 AR Path="/59400D56/591D0796/591D3EBF" Ref="U3101"  Part="1"
 AR Path="/59400D60/591D0796/591D3EBF" Ref="U3501"  Part="1"
-F 0 "U1501" H 5500 4300 60  0000 C CNN
+F 0 "U3101" H 5500 4300 60  0000 C CNN
 F 1 "ADC121S021CIMF/NOPB" H 5550 3640 60  0000 C CNN
 F 2 "IC:SOT-23-6" H 5500 2800 60  0001 C CNN

Commit message: minor
Other:
- note added: "1k"
Changed lines of the file:
@@
 $Descr USLetter 11000 8500
 encoding utf-8
-Sheet 15 36
+Sheet 7 36
 Title "Isolated BMS Slave Front End"
 Date ""
@@
 AR Path="/59400D56/591D0796/591B6F4E" Ref="C3102"  Part="1"
 AR Path="/59400D60/591D0796/591B6F4E" Ref="C3502"  Part="1"
-F 0 "C3102" H 5350 3460 60  0000 C CNN
+F 0 "C702" H 5350 3460 60  0000 C CNN
 F 1 "885012207098" H 5350 2950 60  0001 C CNN
 F 2 "Capacitors:C0805" H 5350 2350 60  0001 C CNN
@@
 AR Path="/59400D56/591D0796/591B6FC1" Ref="C3101"  Part="1"
 AR Path="/59400D60/591D0796/591B6FC1" Ref="C3501"  Part="1"
-F 0 "C3101" H 5350 3060 60  0000 C CNN
+F 0 "C701" H 5350 3060 60  0000 C CNN
 F 1 "885012107015" H 5350 2550 60  0001 C CNN
 F 2 "Capacitors:C0805" H 5350 1950 60  0001 C CNN
@@
 AR Path="/59400D56/591D0796/591BAB3B" Ref="R3101"  Part="1"
 AR Path="/59400D60/591D0796/591BAB3B" Ref="R3501"  Part="1"
-F 0 "R3101" H 4100 4080 60  0000 C CNN
+F 0 "R701" H 4100 4080 60  0000 C CNN
 F 1 "RC0805JR-07100RL" H 4100 3700 50  0001 C CNN
 F 2 "Resistors:R0805" H 4100 3100 30  0001 C CNN
@@
 AR Path="/59400D56/591D0796/591BB052" Ref="C3103"  Part="1"
 AR Path="/59400D60/591D0796/591BB052" Ref="C3503"  Part="1"
-F 0 "C3103" H 4450 4360 60  0000 C CNN
+F 0 "C703" H 4450 4360 60  0000 C CNN
 F 1 "885012207047" H 4450 3850 60  0001 C CNN
 F 2 "Capacitors:C0805" H 4450 3250 60  0001 C CNN
@@
 AR Path="/59400D56/591D0796/591D3EBF" Ref="U3101"  Part="1"
 AR Path="/59400D60/591D0796/591D3EBF" Ref="U3501"  Part="1"
-F 0 "U3101" H 5500 4300 60  0000 C CNN
+F 0 "U701" H 5500 4300 60  0000 C CNN
 F 1 "ADC121S021CIMF/NOPB" H 5550 3640 60  0000 C CNN
 F 2 "IC:SOT-23-6" H 5500 2800 60  0001 C CNN
@@
 Wire Wire Line
 	6800 3100 7200 3100
+Text Notes 4100 3800 0    60   ~ 0
+1k
 $EndSCHEMATC

Commit message: add comment with new ADC RC filter values
Other:
- note added: "100nF"
- note added: "16k"
- note removed: "1k"
Changed lines of the file:
@@
 	6800 3100 7200 3100
 Text Notes 4100 3800 0    60   ~ 0
-1k
+16k
+Text Notes 4600 4500 0    60   ~ 0
+100nF
 $EndSCHEMATC

Commit message: Changed CAN to CAN2, add LED ID
Changed lines of the file:
@@
 AR Path="/59400D56/591D0796/591B6F4E" Ref="C3102"  Part="1"
 AR Path="/59400D60/591D0796/591B6F4E" Ref="C3502"  Part="1"
-F 0 "C702" H 5350 3460 60  0000 C CNN
+F 0 "C3502" H 5350 3460 60  0000 C CNN
 F 1 "885012207098" H 5350 2950 60  0001 C CNN
 F 2 "Capacitors:C0805" H 5350 2350 60  0001 C CNN
@@
 AR Path="/59400D56/591D0796/591B6FC1" Ref="C3101"  Part="1"
 AR Path="/59400D60/591D0796/591B6FC1" Ref="C3501"  Part="1"
-F 0 "C701" H 5350 3060 60  0000 C CNN
+F 0 "C3501" H 5350 3060 60  0000 C CNN
 F 1 "885012107015" H 5350 2550 60  0001 C CNN
 F 2 "Capacitors:C0805" H 5350 1950 60  0001 C CNN
@@
 AR Path="/59400D56/591D0796/591BAB3B" Ref="R3101"  Part="1"
 AR Path="/59400D60/591D0796/591BAB3B" Ref="R3501"  Part="1"
-F 0 "R701" H 4100 4080 60  0000 C CNN
+F 0 "R3501" H 4100 4080 60  0000 C CNN
 F 1 "RC0805JR-07100RL" H 4100 3700 50  0001 C CNN
 F 2 "Resistors:R0805" H 4100 3100 30  0001 C CNN
@@
 AR Path="/59400D56/591D0796/591BB052" Ref="C3103"  Part="1"
 AR Path="/59400D60/591D0796/591BB052" Ref="C3503"  Part="1"
-F 0 "C703" H 4450 4360 60  0000 C CNN
+F 0 "C3503" H 4450 4360 60  0000 C CNN
 F 1 "885012207047" H 4450 3850 60  0001 C CNN
 F 2 "Capacitors:C0805" H 4450 3250 60  0001 C CNN
@@
 AR Path="/59400D56/591D0796/591D3EBF" Ref="U3101"  Part="1"
 AR Path="/59400D60/591D0796/591D3EBF" Ref="U3501"  Part="1"
-F 0 "U701" H 5500 4300 60  0000 C CNN
+F 0 "U3501" H 5500 4300 60  0000 C CNN
 F 1 "ADC121S021CIMF/NOPB" H 5550 3640 60  0000 C CNN
 F 2 "IC:SOT-23-6" H 5500 2800 60  0001 C CNN
