File: Master_Board/V1/Power Supply.sch (KiCad schematic (older format))
At the start: 19 parts, among them J301 Header_Male_Pin_2.54mm_1X2_,_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, U301 OKI-78SR-5/1.5-W36-C, U302 AZ1117IH-3.3TRG1

Commit message: Add page LedDriver
Parts:
- renumbered C302 to C301, C303 to C302, C304 to C303, C301 to C304, TP302 to TP301, TP304 to TP302, TP301 to TP304
Changed lines of the file:
@@
 $Descr USLetter 11000 8500
 encoding utf-8
-Sheet 3 10
+Sheet 3 11
 Title "Power Supply"
 Date ""
@@
 3.3V (LDO)
 $Comp
-L VDD #PWR034
+L VDD #PWR312
 U 1 1 58F7F090
 P 8000 3500
-F 0 "#PWR034" H 8000 3350 50  0001 C CNN
+F 0 "#PWR312" H 8000 3350 50  0001 C CNN
 F 1 "VDD" H 7990 3640 50  0000 C CNN
 F 2 "" H 8000 3500 60  0000 C CNN
@@
 $EndComp
 $Comp
-L PWR_FLAG #FLG035
+L PWR_FLAG #FLG305
 U 1 1 58F88B2C
 P 6800 3500
-F 0 "#FLG035" H 6800 3400 60  0001 C CNN
+F 0 "#FLG305" H 6800 3400 60  0001 C CNN
 F 1 "PWR_FLAG" H 6800 3700 30  0000 C CNN
 F 2 "" H 6800 3500 60  0000 C CNN
@@
 $EndComp
 $Comp
-L PWR_FLAG #FLG036
+L PWR_FLAG #FLG304
 U 1 1 58F88B3E
 P 5100 3600
-F 0 "#FLG036" H 5100 3500 60  0001 C CNN
+F 0 "#FLG304" H 5100 3500 60  0001 C CNN
 F 1 "PWR_FLAG" H 5100 3800 30  0000 C CNN
 F 2 "" H 5100 3600 60  0000 C CNN
@@
 $EndComp
 $Comp
-L 5V #PWR037
+L 5V #PWR305
 U 1 1 58F88B47
 P 4900 3600
-F 0 "#PWR037" H 4900 3450 50  0001 C CNN
+F 0 "#PWR305" H 4900 3450 50  0001 C CNN
 F 1 "5V" H 4890 3740 50  0000 C CNN
 F 2 "" H 4900 3600 60  0000 C CNN
@@
 $EndComp
 $Comp
-L DGND #PWR038
+L DGND #PWR304
 U 1 1 58F88F61
 P 4200 4400
-F 0 "#PWR038" H 4200 4230 50  0001 C CNN
+F 0 "#PWR304" H 4200 4230 50  0001 C CNN
 F 1 "DGND" H 4200 4300 50  0000 C CNN
 F 2 "" H 4200 4500 60  0000 C CNN
@@
 Connection ~ 4900 3700
 $Comp
-L 885012107018 C302
+L 885012107018 C301
 U 1 1 58F8900A
 P 3600 3900
-F 0 "C302" V 3600 4125 60  0000 C CNN
+F 0 "C301" V 3600 4125 60  0000 C CNN
 F 1 "885012107018" H 3550 3550 60  0001 C CNN
 F 2 "Capacitors:C0805" H 3550 2950 60  0001 C CNN
@@
 $EndComp
 $Comp
-L 885012107018 C303
+L 885012107018 C302
 U 1 1 58F89140
 P 4800 3900
-F 0 "C303" V 4800 4125 60  0000 C CNN
+F 0 "C302" V 4800 4125 60  0000 C CNN
 F 1 "885012107018" H 4750 3550 60  0001 C CNN
 F 2 "Capacitors:C0805" H 4750 2950 60  0001 C CNN
@@
 Connection ~ 5100 3700
 $Comp
-L 885012107014 C304
+L 885012107014 C303
 U 1 1 58F8A222
 P 5700 3900
-F 0 "C304" V 5700 4125 60  0000 C CNN
+F 0 "C303" V 5700 4125 60  0000 C CNN
 F 1 "885012107014" H 5650 3550 60  0001 C CNN
 F 2 "Capacitors:C0805" H 5650 2950 60  0001 C CNN
@@
 	5700 4100 5700 4200
 $Comp
-L DGND #PWR039
+L DGND #PWR307
 U 1 1 58F8A321
 P 5700 4300
-F 0 "#PWR039" H 5700 4130 50  0001 C CNN
+F 0 "#PWR307" H 5700 4130 50  0001 C CNN
 F 1 "DGND" H 5700 4200 50  0000 C CNN
 F 2 "" H 5700 4400 60  0000 C CNN
@@
 $EndComp
 $Comp
-L DGND #PWR040
+L DGND #PWR308
 U 1 1 58F8A33F
 P 6200 4200
-F 0 "#PWR040" H 6200 4030 50  0001 C CNN
+F 0 "#PWR308" H 6200 4030 50  0001 C CNN
 F 1 "DGND" H 6200 4100 50  0000 C CNN
 F 2 "" H 6200 4300 60  0000 C CNN
@@
 Connection ~ 6600 3600
 $Comp
-L 885012107005 C301
+L 885012107005 C304
 U 1 1 58F8A3EF
 P 7000 3800
-F 0 "C301" V 7000 4025 60  0000 C CNN
+F 0 "C304" V 7000 4025 60  0000 C CNN
 F 1 "885012107005" H 6950 3450 60  0001 C CNN
 F 2 "Capacitors:C0805" H 6950 2850 60  0001 C CNN
@@
 $EndComp
 $Comp
-L DGND #PWR041
+L DGND #PWR309
 U 1 1 58F8A4C9
 P 7000 4200
-F 0 "#PWR041" H 7000 4030 50  0001 C CNN
+F 0 "#PWR309" H 7000 4030 50  0001 C CNN
 F 1 "DGND" H 7000 4100 50  0000 C CNN
 F 2 "" H 7000 4300 60  0000 C CNN
@@
 Connection ~ 7000 3600
 $Comp
-L PWR_FLAG #FLG042
+L PWR_FLAG #FLG301
 U 1 1 58F8B845
 P 1900 3600
-F 0 "#FLG042" H 1900 3500 60  0001 C CNN
+F 0 "#FLG301" H 1900 3500 60  0001 C CNN
 F 1 "PWR_FLAG" H 1900 3800 30  0000 C CNN
 F 2 "" H 1900 3600 60  0000 C CNN
@@
 Connection ~ 1900 3700
 $Comp
-L PWR_FLAG #FLG043
+L PWR_FLAG #FLG303
 U 1 1 58F8B88C
 P 3900 4300
-F 0 "#FLG043" H 3900 4200 60  0001 C CNN
+F 0 "#FLG303" H 3900 4200 60  0001 C CNN
 F 1 "PWR_FLAG" H 3900 4500 30  0000 C CNN
 F 2 "" H 3900 4300 60  0000 C CNN
@@
 $EndComp
 $Comp
-L DGND #PWR044
+L DGND #PWR306
 U 1 1 58F8E9CC
 P 5000 5100
-F 0 "#PWR044" H 5000 4930 50  0001 C CNN
+F 0 "#PWR306" H 5000 4930 50  0001 C CNN
 F 1 "DGND" H 5000 5000 50  0000 C CNN
 F 2 "" H 5000 5200 60  0000 C CNN
@@
 	5000 4100 5000 3700
 Connection ~ 5000 3700
-Wire Wire Line
-	1600 3700 2000 3700
 $Comp
 L RC0805JR-07470RL R303
@@
 $EndComp
 $Comp
-L DGND #PWR045
+L DGND #PWR311
 U 1 1 58F8EC42
 P 7500 5100
-F 0 "#PWR045" H 7500 4930 50  0001 C CNN
+F 0 "#PWR311" H 7500 4930 50  0001 C CNN
 F 1 "DGND" H 7500 5000 50  0000 C CNN
 F 2 "" H 7500 5200 60  0000 C CNN
@@
 $EndComp
 $Comp
-L DGND #PWR046
+L DGND #PWR303
 U 1 1 58F8E20A
 P 3200 5100
-F 0 "#PWR046" H 3200 4930 50  0001 C CNN
+F 0 "#PWR303" H 3200 4930 50  0001 C CNN
 F 1 "DGND" H 3200 5000 50  0000 C CNN
 F 2 "" H 3200 5200 60  0000 C CNN
@@
 Connection ~ 3200 3700
 $Comp
-L Test_Point_THM TP302
+L Test_Point_THM TP301
 U 1 1 58F8E348
 P 3400 3400
-F 0 "TP302" V 3300 3400 60  0000 C CNN
+F 0 "TP301" V 3300 3400 60  0000 C CNN
 F 1 "Test_Point_THM" H 3400 3100 60  0001 C CNN
 F 2 "Connectors:Keystone_5001" H 3400 2500 60  0001 C CNN
@@
 Connection ~ 5400 3700
 $Comp
-L Test_Point_THM TP301
+L Test_Point_THM TP304
 U 1 1 58F8E9A6
 P 7300 3300
-F 0 "TP301" V 7175 3300 60  0000 C CNN
+F 0 "TP304" V 7175 3300 60  0000 C CNN
 F 1 "Test_Point_THM" H 7300 3000 60  0001 C CNN
 F 2 "Connectors:Keystone_5001" H 7300 2400 60  0001 C CNN
@@
 Connection ~ 7300 3600
 $Comp
-L Test_Point_THM TP304
+L Test_Point_THM TP302
 U 1 1 58F8EB6B
 P 3600 4500
-F 0 "TP304" V 3475 4500 60  0000 C CNN
+F 0 "TP302" V 3475 4500 60  0000 C CNN
 F 1 "Test_Point_THM" H 3600 4200 60  0001 C CNN
 F 2 "Connectors:Keystone_5001" H 3600 3600 60  0001 C CNN
@@
 	2500 3700 3900 3700
 Wire Wire Line
-	1900 3700 2100 3700
+	1600 3700 2100 3700
 Wire Wire Line
 	6500 3600 7700 3600
 $Comp
-L 12V #PWR047
+L 12V #PWR302
 U 1 1 58FEC80D
 P 2600 3600
-F 0 "#PWR047" H 2600 3450 50  0001 C CNN
+F 0 "#PWR302" H 2600 3450 50  0001 C CNN
 F 1 "12V" H 2590 3740 50  0000 C CNN
 F 2 "" H 2600 3600 60  0000 C CNN
@@
 $EndComp
 $Comp
-L PWR_FLAG #FLG048
+L PWR_FLAG #FLG302
 U 1 1 58FEC813
 P 2900 3600
-F 0 "#FLG048" H 2900 3500 60  0001 C CNN
+F 0 "#FLG302" H 2900 3500 60  0001 C CNN
 F 1 "PWR_FLAG" H 2900 3800 30  0000 C CNN
 F 2 "" H 2900 3600 60  0000 C CNN
@@
 	1600 3600 1600 3700
 $Comp
-L CAN_PWR #PWR049
+L CAN_PWR #PWR301
 U 1 1 58FEC94F
 P 1600 3600
-F 0 "#PWR049" H 1600 3450 50  0001 C CNN
+F 0 "#PWR301" H 1600 3450 50  0001 C CNN
 F 1 "CAN_PWR" H 1590 3740 50  0000 C CNN
 F 2 "" H 1600 3600 60  0000 C CNN
@@
 $EndComp
 $Comp
-L 3.3V #PWR050
+L 3.3V #PWR310
 U 1 1 58FF65C4
 P 7100 3500
-F 0 "#PWR050" H 7100 3350 50  0001 C CNN
+F 0 "#PWR310" H 7100 3350 50  0001 C CNN
 F 1 "3.3V" H 7090 3640 50  0000 C CNN
 F 2 "" H 7100 3500 60  0000 C CNN
@@
 Connection ~ 8000 3600
 $Comp
-L PWR_FLAG #FLG051
+L PWR_FLAG #FLG306
 U 1 1 58FF7333
 P 8500 3500
-F 0 "#FLG051" H 8500 3400 60  0001 C CNN
+F 0 "#FLG306" H 8500 3400 60  0001 C CNN
 F 1 "PWR_FLAG" H 8500 3700 30  0000 C CNN
 F 2 "" H 8500 3500 60  0000 C CNN

Commit message: Modify MasterBoard.sch
Parts:
- D301, D302, D303: symbol 150080VS75000 -> 150080VS75000-RESCUE-Master_Board
Changed lines of the file:
@@
 EESchema Schematic File Version 2
+LIBS:Master_Board-rescue
 LIBS:ADC
 LIBS:Amplifiers
@@
 Connection ~ 3900 4200
 $Comp
-L 150080VS75000 D302
+L 150080VS75000-RESCUE-Master_Board D302
 U 1 1 58F8E86A
 P 5000 4800
@@
 $EndComp
 $Comp
-L 150080VS75000 D303
+L 150080VS75000-RESCUE-Master_Board D303
 U 1 1 58F8EC30
 P 7500 4800
@@
 Connection ~ 7500 3600
 $Comp
-L 150080VS75000 D301
+L 150080VS75000-RESCUE-Master_Board D301
 U 1 1 58F8E204
 P 3200 4800
