File: Current_Sense/V1/power_supply.sch (KiCad schematic (older format))
At the start: 33 parts, among them U401 PQMC3-D12-D15-S, U402 NCP1117LPST33T3G, U403 NCP1117ST50T3G

Commit message: start to place pin on uC
Parts:
- added C418, C419: 885012107018, Capacitors:C0805, symbol 885012107018
- added C420: 885012107014, Capacitors:C0805, symbol 885012107014
- added J401: Header_Male_Pin_2.54mm_1X2_,_Unshrouded, Connectors:Headers_2.54mm_1X2, symbol Header_Male_Pin_2.54mm_1X2_,_Unshrouded
- added TP407: Test_Point_THM, Connectors:Keystone_5001, symbol Test_Point_THM
- added U404: NCP1117LPST33T3G, IC:SOT-223-3, symbol NCP1117LPST33T3G
Connections:
- net 5VB: now also C418.2, C419.2, U404.3 (Vin)
- net GNDB: now also C418.1, C419.1, C420.1, U404.1 (GND)
- new net: C420.2, J401.1, TP407.1 (TP), U404.2 (Vout), U404.4 (Vout_(TAB))
- new net VDD: J401.2

Commit message: placing power supply
Parts:
- added TP408: Test_Point_THM, Connectors:Keystone_5001, symbol Test_Point_THM
Connections:
- net -15VB: now also TP408.1 (TP)
Changed lines of the file:
@@
 Isolated DC-DC
 $Comp
-L PWR_FLAG #FLG049
+L PWR_FLAG #FLG402
 U 1 1 592CA09E
 P 2300 1900
-F 0 "#FLG049" H 2300 1800 60  0001 C CNN
+F 0 "#FLG402" H 2300 1800 60  0001 C CNN
 F 1 "PWR_FLAG" H 2300 2100 30  0000 C CNN
 F 2 "" H 2300 1900 60  0000 C CNN
@@
 $EndComp
 $Comp
-L PWR_FLAG #FLG050
+L PWR_FLAG #FLG404
 U 1 1 592CA0B8
 P 5400 2500
-F 0 "#FLG050" H 5400 2400 60  0001 C CNN
+F 0 "#FLG404" H 5400 2400 60  0001 C CNN
 F 1 "PWR_FLAG" H 5400 2700 30  0000 C CNN
 F 2 "" H 5400 2500 60  0000 C CNN
@@
 $EndComp
 $Comp
-L GNDA #PWR051
+L GNDA #PWR415
 U 1 1 592CAB5C
 P 3000 4900
-F 0 "#PWR051" H 3000 4730 50  0001 C CNN
+F 0 "#PWR415" H 3000 4730 50  0001 C CNN
 F 1 "GNDA" H 3000 4800 50  0000 C CNN
 F 2 "" H 3000 5000 60  0000 C CNN
@@
 $EndComp
 $Comp
-L 3.3VA #PWR052
+L 3.3VA #PWR412
 U 1 1 592CACD3
 P 4300 4000
-F 0 "#PWR052" H 4300 3850 50  0001 C CNN
+F 0 "#PWR412" H 4300 3850 50  0001 C CNN
 F 1 "3.3VA" H 4290 4140 50  0000 C CNN
 F 2 "" H 4300 4000 60  0000 C CNN
@@
 Connection ~ 3700 4100
 $Comp
-L 15VB #PWR053
+L 15VB #PWR401
 U 1 1 592CB5E5
 P 8400 1600
-F 0 "#PWR053" H 8400 1450 50  0001 C CNN
+F 0 "#PWR401" H 8400 1450 50  0001 C CNN
 F 1 "15VB" H 8390 1740 50  0000 C CNN
 F 2 "" H 8400 1600 60  0000 C CNN
@@
 $EndComp
 $Comp
-L -15VB #PWR054
+L -15VB #PWR408
 U 1 1 592CB605
 P 8300 2800
-F 0 "#PWR054" H 8300 2520 50  0001 C CNN
+F 0 "#PWR408" H 8300 2520 50  0001 C CNN
 F 1 "-15VB" H 8290 2660 50  0000 C CNN
 F 2 "" H 8300 2800 60  0000 C CNN
@@
 $EndComp
 $Comp
-L PWR_FLAG #FLG055
+L PWR_FLAG #FLG405
 U 1 1 592CB62F
 P 8000 2800
-F 0 "#FLG055" H 8000 2700 60  0001 C CNN
+F 0 "#FLG405" H 8000 2700 60  0001 C CNN
 F 1 "PWR_FLAG" H 8000 3000 30  0000 C CNN
 F 2 "" H 8000 2800 60  0000 C CNN
@@
 $EndComp
 $Comp
-L PWR_FLAG #FLG056
+L PWR_FLAG #FLG401
 U 1 1 592CB63B
 P 8100 1600
-F 0 "#FLG056" H 8100 1500 60  0001 C CNN
+F 0 "#FLG401" H 8100 1500 60  0001 C CNN
 F 1 "PWR_FLAG" H 8100 1800 30  0000 C CNN
 F 2 "" H 8100 1600 60  0000 C CNN
@@
 $EndComp
 $Comp
-L GNDB #PWR057
+L GNDB #PWR404
 U 1 1 592CB709
 P 9000 2400
-F 0 "#PWR057" H 9000 2230 50  0001 C CNN
+F 0 "#PWR404" H 9000 2230 50  0001 C CNN
 F 1 "GNDB" H 9000 2300 50  0000 C CNN
 F 2 "" H 9000 2500 60  0000 C CNN
@@
 $EndComp
 $Comp
-L PWR_FLAG #FLG058
+L PWR_FLAG #FLG403
 U 1 1 592CB727
 P 8700 2300
-F 0 "#FLG058" H 8700 2200 60  0001 C CNN
+F 0 "#FLG403" H 8700 2200 60  0001 C CNN
 F 1 "PWR_FLAG" H 8700 2500 30  0000 C CNN
 F 2 "" H 8700 2300 60  0000 C CNN
@@
 	5400 2400 5400 2500
 $Comp
-L GNDA #PWR059
+L GNDA #PWR407
 U 1 1 592CC36E
 P 5100 2800
-F 0 "#PWR059" H 5100 2630 50  0001 C CNN
+F 0 "#PWR407" H 5100 2630 50  0001 C CNN
 F 1 "GNDA" H 5100 2700 50  0000 C CNN
 F 2 "" H 5100 2900 60  0000 C CNN
@@
 $EndComp
 $Comp
-L GNDA #PWR060
+L GNDA #PWR410
 U 1 1 592CD2BA
 P 4300 2900
-F 0 "#PWR060" H 4300 2730 50  0001 C CNN
+F 0 "#PWR410" H 4300 2730 50  0001 C CNN
 F 1 "GNDA" H 4300 2800 50  0000 C CNN
 F 2 "" H 4300 3000 60  0000 C CNN
@@
 	3600 2500 3600 2400
 $Comp
-L GNDA #PWR061
+L GNDA #PWR406
 U 1 1 592CDE1C
 P 2000 2700
-F 0 "#PWR061" H 2000 2530 50  0001 C CNN
+F 0 "#PWR406" H 2000 2530 50  0001 C CNN
 F 1 "GNDA" H 2000 2600 50  0000 C CNN
 F 2 "" H 2000 2800 60  0000 C CNN
@@
 $EndComp
 $Comp
-L GNDB #PWR062
+L GNDB #PWR416
 U 1 1 592CE794
 P 7900 4900
-F 0 "#PWR062" H 7900 4730 50  0001 C CNN
+F 0 "#PWR416" H 7900 4730 50  0001 C CNN
 F 1 "GNDB" H 7900 4800 50  0000 C CNN
 F 2 "" H 7900 5000 60  0000 C CNN
@@
 Connection ~ 8300 4100
 $Comp
-L 15VB #PWR063
+L 15VB #PWR413
 U 1 1 592CEBA4
 P 6900 4000
-F 0 "#PWR063" H 6900 3850 50  0001 C CNN
+F 0 "#PWR413" H 6900 3850 50  0001 C CNN
 F 1 "15VB" H 6890 4140 50  0000 C CNN
 F 2 "" H 6900 4000 60  0000 C CNN
@@
 Connection ~ 6900 4100
 $Comp
-L 5VB #PWR064
+L 5VB #PWR414
 U 1 1 592CF13F
 P 9300 4000
-F 0 "#PWR064" H 9300 3850 50  0001 C CNN
+F 0 "#PWR414" H 9300 3850 50  0001 C CNN
 F 1 "5VB" H 9290 4140 50  0000 C CNN
 F 2 "" H 9300 4000 60  0000 C CNN
@@
 Connection ~ 8900 2200
 $Comp
-L 12VA #PWR065
+L 12VA #PWR411
 U 1 1 592CA984
 P 2000 4000
-F 0 "#PWR065" H 2000 3850 50  0001 C CNN
+F 0 "#PWR411" H 2000 3850 50  0001 C CNN
 F 1 "12VA" H 1990 4140 50  0000 C CNN
 F 2 "" H 2000 4000 60  0000 C CNN
@@
 $EndComp
 $Comp
-L 12VA #PWR066
+L 12VA #PWR403
 U 1 1 592CA068
 P 2000 1900
-F 0 "#PWR066" H 2000 1750 50  0001 C CNN
+F 0 "#PWR403" H 2000 1750 50  0001 C CNN
 F 1 "12VA" H 1990 2040 50  0000 C CNN
 F 2 "" H 2000 1900 60  0000 C CNN
@@
 $EndComp
 $Comp
-L PWR_FLAG #FLG067
+L PWR_FLAG #FLG406
 U 1 1 59300390
 P 4000 4000
-F 0 "#FLG067" H 4000 3900 60  0001 C CNN
+F 0 "#FLG406" H 4000 3900 60  0001 C CNN
 F 1 "PWR_FLAG" H 4000 4200 30  0000 C CNN
 F 2 "" H 4000 4000 60  0000 C CNN
@@
 Connection ~ 4000 4100
 $Comp
-L PWR_FLAG #FLG068
+L PWR_FLAG #FLG407
 U 1 1 59301548
 P 9000 4000
-F 0 "#FLG068" H 9000 3900 60  0001 C CNN
+F 0 "#FLG407" H 9000 3900 60  0001 C CNN
 F 1 "PWR_FLAG" H 9000 4200 30  0000 C CNN
 F 2 "" H 9000 4000 60  0000 C CNN
@@
 $EndComp
 $Comp
-L 15VB #PWR069
+L 15VB #PWR402
 U 1 1 592F48C4
 P 9400 1600
-F 0 "#PWR069" H 9400 1450 50  0001 C CNN
+F 0 "#PWR402" H 9400 1450 50  0001 C CNN
 F 1 "15VB" H 9390 1740 50  0000 C CNN
 F 2 "" H 9400 1600 60  0000 C CNN
@@
 	9400 2100 9400 2300
 $Comp
-L -15VB #PWR070
+L -15VB #PWR409
 U 1 1 592F4A81
 P 9400 2800
-F 0 "#PWR070" H 9400 2520 50  0001 C CNN
+F 0 "#PWR409" H 9400 2520 50  0001 C CNN
 F 1 "-15VB" H 9390 2660 50  0000 C CNN
 F 2 "" H 9400 2800 60  0000 C CNN
@@
 	9400 2700 9400 2800
 $Comp
-L GNDB #PWR071
+L GNDB #PWR405
 U 1 1 592F4B78
 P 9700 2400
-F 0 "#PWR071" H 9700 2230 50  0001 C CNN
+F 0 "#PWR405" H 9700 2230 50  0001 C CNN
 F 1 "GNDB" H 9700 2300 50  0000 C CNN
 F 2 "" H 9700 2500 60  0000 C CNN
@@
 	9300 5600 10000 5600
 $Comp
-L VDD #PWR072
+L VDD #PWR418
 U 1 1 595BD90E
 P 10000 5500
-F 0 "#PWR072" H 10000 5350 50  0001 C CNN
+F 0 "#PWR418" H 10000 5350 50  0001 C CNN
 F 1 "VDD" H 9990 5640 50  0000 C CNN
 F 2 "" H 10000 5500 60  0000 C CNN
@@
 	10000 5600 10000 5500
 $Comp
-L PWR_FLAG #FLG073
+L PWR_FLAG #FLG409
 U 1 1 595BDADB
 P 9600 5500
-F 0 "#FLG073" H 9600 5400 60  0001 C CNN
+F 0 "#FLG409" H 9600 5400 60  0001 C CNN
 F 1 "PWR_FLAG" H 9600 5700 30  0000 C CNN
 F 2 "" H 9600 5500 60  0000 C CNN
@@
 Connection ~ 8700 5600
 $Comp
-L PWR_FLAG #FLG074
+L PWR_FLAG #FLG408
 U 1 1 595C219D
 P 8900 5500
-F 0 "#FLG074" H 8900 5400 60  0001 C CNN
+F 0 "#FLG408" H 8900 5400 60  0001 C CNN
 F 1 "PWR_FLAG" H 8900 5700 30  0000 C CNN
 F 2 "" H 8900 5500 60  0000 C CNN
@@
 	9200 5600 9200 5500
 $Comp
-L GNDB #PWR075
+L GNDB #PWR419
 U 1 1 595C48E8
 P 7900 6400
-F 0 "#PWR075" H 7900 6230 50  0001 C CNN
+F 0 "#PWR419" H 7900 6230 50  0001 C CNN
 F 1 "GNDB" H 7900 6300 50  0000 C CNN
 F 2 "" H 7900 6500 60  0000 C CNN
@@
 $EndComp
 $Comp
-L 5VB #PWR076
+L 5VB #PWR417
 U 1 1 595C4BF8
 P 6900 5500
-F 0 "#PWR076" H 6900 5350 50  0001 C CNN
+F 0 "#PWR417" H 6900 5350 50  0001 C CNN
 F 1 "5VB" H 6890 5640 50  0000 C CNN
 F 2 "" H 6900 5500 60  0000 C CNN
@@
 	1    0    0    -1
 $EndComp
+$Comp
+L Test_Point_THM TP408
+U 1 1 595EE28F
+P 7650 3000
+F 0 "TP408" H 7650 2900 60  0000 C CNN
+F 1 "Test_Point_THM" H 7650 2700 60  0001 C CNN
+F 2 "Connectors:Keystone_5001" H 7650 2100 60  0001 C CNN
+F 3 "http://keyelco.com/userAssets/file/M65p56.pdf" H 7650 2000 60  0001 C CNN
+F 4 "Digikey" H 7650 2600 60  0001 C CNN "Supplier"
+F 5 "36-5001-ND" H 7650 2500 60  0001 C CNN "Supplier Part Number"
+F 6 "Keystone Electronics" H 7650 2400 60  0001 C CNN "Manufacturer"
+F 7 "5001" H 7650 2300 60  0001 C CNN "Manufacturer Part Number"
+F 8 "TEST POINT PC MINI .040\"D BLACK" H 7650 2200 60  0001 C CNN "Description"
+	1    7650 3000
+	0    -1   -1   0
+$EndComp
+Wire Wire Line
+	7650 2800 7650 2700
+Connection ~ 7650 2700
 $EndSCHEMATC
