File: Master_Board/V2/CAN2.sch (KiCad schematic (older format))
At the start: 13 parts, among them U501 SN65HVD232DR

Commit message: Place part in PCB
Connections:
- net CAN2_H: now also D501.2 (CH2); no longer D501.1 (CH1)
- net CAN2_L: now also D501.1 (CH1); no longer D501.2 (CH2)
Changed lines of the file:
@@
 $EndDescr
 $Comp
-L VDD #PWR077
+L VDD #PWR059
 U 1 1 597095FA
 P 2900 2900
-F 0 "#PWR077" H 2900 2750 50  0001 C CNN
+F 0 "#PWR059" H 2900 2750 50  0001 C CNN
 F 1 "VDD" H 2890 3040 50  0000 C CNN
 F 2 "" H 2900 2900 60  0000 C CNN
@@
 $EndComp
 $Comp
-L DGND #PWR078
+L DGND #PWR060
 U 1 1 58F7D8B1
 P 2900 4600
-F 0 "#PWR078" H 2900 4430 50  0001 C CNN
+F 0 "#PWR060" H 2900 4430 50  0001 C CNN
 F 1 "DGND" H 2900 4500 50  0000 C CNN
 F 2 "" H 2900 4700 60  0000 C CNN
@@
 $EndComp
 $Comp
-L DGND #PWR079
+L DGND #PWR061
 U 1 1 597095FE
 P 1800 4600
-F 0 "#PWR079" H 1800 4430 50  0001 C CNN
+F 0 "#PWR061" H 1800 4430 50  0001 C CNN
 F 1 "DGND" H 1800 4500 50  0000 C CNN
 F 2 "" H 1800 4700 60  0000 C CNN
@@
 $EndComp
 $Comp
-L DGND #PWR080
+L DGND #PWR062
 U 1 1 59709600
 P 2400 3600
-F 0 "#PWR080" H 2400 3430 50  0001 C CNN
+F 0 "#PWR062" H 2400 3430 50  0001 C CNN
 F 1 "DGND" H 2400 3500 50  0000 C CNN
 F 2 "" H 2400 3700 60  0000 C CNN
@@
 U 1 1 58F808C0
 P 7000 4100
-F 0 "D501" H 7000 4300 60  0000 C CNN
-F 1 "D1213A-02SOL-7" H 7000 3850 60  0000 C CNN
+F 0 "D501" H 7000 3900 60  0000 C CNN
+F 1 "D1213A-02SOL-7" H 7000 4350 60  0000 C CNN
 F 2 "IC:SOT-23-3" H 7000 3080 60  0001 C CNN
 F 3 "https://www.diodes.com/assets/Datasheets/D1213A_02SOL.pdf" H 7000 2980 60  0001 C CNN
@@
 F 8 "TVS DIODE 3.3VWM 10VC SOT23" H 7000 3180 60  0001 C CNN "Description"
 	1    7000 4100
-	1    0    0    -1
+	1    0    0    1
 $EndComp
 $Comp
-L DGND #PWR081
+L DGND #PWR063
 U 1 1 58F808C6
 P 6050 4900
-F 0 "#PWR081" H 6050 4730 50  0001 C CNN
+F 0 "#PWR063" H 6050 4730 50  0001 C CNN
 F 1 "DGND" H 6050 4800 50  0000 C CNN
 F 2 "" H 6050 5000 60  0000 C CNN
@@
 $EndComp
 $Comp
-L DGND #PWR082
+L DGND #PWR064
 U 1 1 58F808CC
 P 5350 4900
-F 0 "#PWR082" H 5350 4730 50  0001 C CNN
+F 0 "#PWR064" H 5350 4730 50  0001 C CNN
 F 1 "DGND" H 5350 4800 50  0000 C CNN
 F 2 "" H 5350 5000 60  0000 C CNN
@@
 $EndComp
 $Comp
-L DGND #PWR083
+L DGND #PWR065
 U 1 1 58F81672
 P 7500 4400
-F 0 "#PWR083" H 7500 4230 50  0001 C CNN
+F 0 "#PWR065" H 7500 4230 50  0001 C CNN
 F 1 "DGND" H 7500 4300 50  0000 C CNN
 F 2 "" H 7500 4500 60  0000 C CNN
