File: Master_Board/V2/Power Supply.sch (KiCad schematic (older format))
At the start: 19 parts, among them J301 Header_Male_Pin_2.54mm_1X2_,_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, U301 OKI-78SR-5/1.5-W36-C, U302 AZ1117IH-3.3TRG1

Commit message: Place part in PCB
Changed lines of the file:
@@
 3.3V (LDO)
 $Comp
-L VDD #PWR049
+L VDD #PWR031
 U 1 1 58F7F090
 P 8000 3500
-F 0 "#PWR049" H 8000 3350 50  0001 C CNN
+F 0 "#PWR031" H 8000 3350 50  0001 C CNN
 F 1 "VDD" H 7990 3640 50  0000 C CNN
 F 2 "" H 8000 3500 60  0000 C CNN
@@
 $EndComp
 $Comp
-L PWR_FLAG #FLG050
+L PWR_FLAG #FLG032
 U 1 1 58F88B2C
 P 6800 3500
-F 0 "#FLG050" H 6800 3400 60  0001 C CNN
+F 0 "#FLG032" H 6800 3400 60  0001 C CNN
 F 1 "PWR_FLAG" H 6800 3700 30  0000 C CNN
 F 2 "" H 6800 3500 60  0000 C CNN
@@
 $EndComp
 $Comp
-L PWR_FLAG #FLG051
+L PWR_FLAG #FLG033
 U 1 1 58F88B3E
 P 5100 3600
-F 0 "#FLG051" H 5100 3500 60  0001 C CNN
+F 0 "#FLG033" H 5100 3500 60  0001 C CNN
 F 1 "PWR_FLAG" H 5100 3800 30  0000 C CNN
 F 2 "" H 5100 3600 60  0000 C CNN
@@
 $EndComp
 $Comp
-L 5V #PWR052
+L 5V #PWR034
 U 1 1 58F88B47
 P 4900 3600
-F 0 "#PWR052" H 4900 3450 50  0001 C CNN
+F 0 "#PWR034" H 4900 3450 50  0001 C CNN
 F 1 "5V" H 4890 3740 50  0000 C CNN
 F 2 "" H 4900 3600 60  0000 C CNN
@@
 $EndComp
 $Comp
-L DGND #PWR053
+L DGND #PWR035
 U 1 1 58F88F61
 P 4200 4400
-F 0 "#PWR053" H 4200 4230 50  0001 C CNN
+F 0 "#PWR035" H 4200 4230 50  0001 C CNN
 F 1 "DGND" H 4200 4300 50  0000 C CNN
 F 2 "" H 4200 4500 60  0000 C CNN
@@
 	5700 4100 5700 4200
 $Comp
-L DGND #PWR054
+L DGND #PWR036
 U 1 1 58F8A321
 P 5700 4300
-F 0 "#PWR054" H 5700 4130 50  0001 C CNN
+F 0 "#PWR036" H 5700 4130 50  0001 C CNN
 F 1 "DGND" H 5700 4200 50  0000 C CNN
 F 2 "" H 5700 4400 60  0000 C CNN
@@
 $EndComp
 $Comp
-L DGND #PWR055
+L DGND #PWR037
 U 1 1 58F8A33F
 P 6200 4200
-F 0 "#PWR055" H 6200 4030 50  0001 C CNN
+F 0 "#PWR037" H 6200 4030 50  0001 C CNN
 F 1 "DGND" H 6200 4100 50  0000 C CNN
 F 2 "" H 6200 4300 60  0000 C CNN
@@
 $EndComp
 $Comp
-L DGND #PWR056
+L DGND #PWR038
 U 1 1 58F8A4C9
 P 7000 4200
-F 0 "#PWR056" H 7000 4030 50  0001 C CNN
+F 0 "#PWR038" H 7000 4030 50  0001 C CNN
 F 1 "DGND" H 7000 4100 50  0000 C CNN
 F 2 "" H 7000 4300 60  0000 C CNN
@@
 Connection ~ 7000 3600
 $Comp
-L PWR_FLAG #FLG057
+L PWR_FLAG #FLG039
 U 1 1 58F8B845
 P 1900 3600
-F 0 "#FLG057" H 1900 3500 60  0001 C CNN
+F 0 "#FLG039" H 1900 3500 60  0001 C CNN
 F 1 "PWR_FLAG" H 1900 3800 30  0000 C CNN
 F 2 "" H 1900 3600 60  0000 C CNN
@@
 Connection ~ 1900 3700
 $Comp
-L PWR_FLAG #FLG058
+L PWR_FLAG #FLG040
 U 1 1 58F8B88C
 P 3900 4300
-F 0 "#FLG058" H 3900 4200 60  0001 C CNN
+F 0 "#FLG040" H 3900 4200 60  0001 C CNN
 F 1 "PWR_FLAG" H 3900 4500 30  0000 C CNN
 F 2 "" H 3900 4300 60  0000 C CNN
@@
 $EndComp
 $Comp
-L DGND #PWR059
+L DGND #PWR041
 U 1 1 58F8E9CC
 P 5000 5100
-F 0 "#PWR059" H 5000 4930 50  0001 C CNN
+F 0 "#PWR041" H 5000 4930 50  0001 C CNN
 F 1 "DGND" H 5000 5000 50  0000 C CNN
 F 2 "" H 5000 5200 60  0000 C CNN
@@
 $EndComp
 $Comp
-L DGND #PWR060
+L DGND #PWR042
 U 1 1 58F8EC42
 P 7500 5100
-F 0 "#PWR060" H 7500 4930 50  0001 C CNN
+F 0 "#PWR042" H 7500 4930 50  0001 C CNN
 F 1 "DGND" H 7500 5000 50  0000 C CNN
 F 2 "" H 7500 5200 60  0000 C CNN
@@
 $EndComp
 $Comp
-L DGND #PWR061
+L DGND #PWR043
 U 1 1 58F8E20A
 P 3200 5100
-F 0 "#PWR061" H 3200 4930 50  0001 C CNN
+F 0 "#PWR043" H 3200 4930 50  0001 C CNN
 F 1 "DGND" H 3200 5000 50  0000 C CNN
 F 2 "" H 3200 5200 60  0000 C CNN
@@
 	6500 3600 7700 3600
 $Comp
-L 12V #PWR062
+L 12V #PWR044
 U 1 1 58FEC80D
 P 2600 3600
-F 0 "#PWR062" H 2600 3450 50  0001 C CNN
+F 0 "#PWR044" H 2600 3450 50  0001 C CNN
 F 1 "12V" H 2590 3740 50  0000 C CNN
 F 2 "" H 2600 3600 60  0000 C CNN
@@
 $EndComp
 $Comp
-L PWR_FLAG #FLG063
+L PWR_FLAG #FLG045
 U 1 1 58FEC813
 P 2900 3600
-F 0 "#FLG063" H 2900 3500 60  0001 C CNN
+F 0 "#FLG045" H 2900 3500 60  0001 C CNN
 F 1 "PWR_FLAG" H 2900 3800 30  0000 C CNN
 F 2 "" H 2900 3600 60  0000 C CNN
@@
 	1600 3600 1600 3700
 $Comp
-L CAN_PWR #PWR064
+L CAN_PWR #PWR046
 U 1 1 58FEC94F
 P 1600 3600
-F 0 "#PWR064" H 1600 3450 50  0001 C CNN
+F 0 "#PWR046" H 1600 3450 50  0001 C CNN
 F 1 "CAN_PWR" H 1590 3740 50  0000 C CNN
 F 2 "" H 1600 3600 60  0000 C CNN
@@
 $EndComp
 $Comp
-L 3.3V #PWR065
+L 3.3V #PWR047
 U 1 1 58FF65C4
 P 7100 3500
-F 0 "#PWR065" H 7100 3350 50  0001 C CNN
+F 0 "#PWR047" H 7100 3350 50  0001 C CNN
 F 1 "3.3V" H 7090 3640 50  0000 C CNN
 F 2 "" H 7100 3500 60  0000 C CNN
@@
 Connection ~ 8000 3600
 $Comp
-L PWR_FLAG #FLG066
+L PWR_FLAG #FLG048
 U 1 1 58FF7333
 P 8500 3500
-F 0 "#FLG066" H 8500 3400 60  0001 C CNN
+F 0 "#FLG048" H 8500 3400 60  0001 C CNN
 F 1 "PWR_FLAG" H 8500 3700 30  0000 C CNN
 F 2 "" H 8500 3500 60  0000 C CNN
@@
 U 1 1 59347B67
 P 5000 4300
-F 0 "R302" H 5000 4380 60  0000 C CNN
+F 0 "R302" V 5050 4350 60  0000 L CNN
 F 1 "RC0805JR-071KL" H 5000 4000 50  0001 C CNN
 F 2 "Resistors:R0805" H 5000 3400 30  0001 C CNN
@@
 F 7 "RC0805JR-071KL" H 5000 3600 60  0001 C CNN "Manufacturer Part Number"
 F 8 "RES SMD 1K OHM 5% 1/8W 0805" H 5000 3500 60  0001 C CNN "Description"
-F 9 "1k" H 5000 4230 50  0000 C CNN "Resistance (Ohms)"
+F 9 "1k" V 4950 4350 50  0000 L CNN "Resistance (Ohms)"
 F 10 "±5%" H 5410 4220 50  0001 C CNN "Tolerance (%)"
 F 11 "1/8W" H 5000 4160 50  0001 C CNN "Puissance (Watts)"
@@
 U 1 1 59347DB4
 P 3200 4300
-F 0 "R301" H 3200 4380 60  0000 C CNN
+F 0 "R301" V 3250 4350 60  0000 L CNN
 F 1 "RC0805JR-074K7L" H 3200 4000 50  0001 C CNN
 F 2 "Resistors:R0805" H 3200 3400 30  0001 C CNN
@@
 F 7 "RC0805JR-074K7L" H 3200 3600 60  0001 C CNN "Manufacturer Part Number"
 F 8 "RES SMD 4.7K OHM 5% 1/8W 0805" H 3200 3500 60  0001 C CNN "Description"
-F 9 "4.7k" H 3200 4230 50  0000 C CNN "Resistance (Ohms)"
+F 9 "4.7k" V 3150 4350 50  0000 L CNN "Resistance (Ohms)"
 F 10 "±5%" H 3400 4200 50  0001 C CNN "Tolerance (%)"
 F 11 "1/8W" H 3200 4160 50  0001 C CNN "Puissance (Watts)"
