File: Master_Board/V2/VoltageSense.sch (KiCad schematic (older format))
At the start: 41 parts, among them J801 649002227222, J802 649002227222, J803 649002227222, J804 649002227222, U801 ACPL-C87A-500E, U802 NCS1S2405SC, U803 ACPL-C87A-500E, U804 LMV321RILT, U805 LMV321RILT

Commit message: Place part in PCB
Parts:
- renumbered C801 to C901, C802 to C902, C803 to C903, C804 to C904, C805 to C905, C806 to C906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
Connections:
- net BP_VSense renamed VSENSE_BP
- net GND renamed AGND
- net MPPT_VSense renamed VSENSE_MPPT
- net VSense_EN renamed VSENSE_EN
