File: Master_Board/V3/LedDriver.sch (KiCad schematic (older format))
At the start: 2 parts

Commit message: Rooting Master V3
Parts:
- renumbered D901 to D1001, R901 to R1001
Changed lines of the file:
@@
 LED Error
 $Comp
-L 150080RS75000 D901
+L 150080RS75000 D1001
 U 1 1 594D45D6
 P 6100 3700
-F 0 "D901" H 6100 3500 60  0000 C CNN
+F 0 "D1001" H 6100 3500 60  0000 C CNN
 F 1 "150080RS75000" H 6050 3850 60  0001 C CNN
 F 2 "Diodes:LED_0805_RED" H 6110 2620 60  0001 C CNN
@@
 $EndComp
 $Comp
-L RC0805JR-07330RL R901
+L RC0805JR-07330RL R1001
 U 1 1 594D472A
 P 5450 3700
-F 0 "R901" H 5450 3780 60  0000 C CNN
+F 0 "R1001" H 5450 3780 60  0000 C CNN
 F 1 "RC0805JR-07330RL" H 5450 3400 50  0001 C CNN
 F 2 "Resistors:R0805" H 5450 2800 30  0001 C CNN
@@
 	5250 3700 4550 3700
 $Comp
-L DGND #PWR087
+L DGND #PWR086
 U 1 1 594D4935
 P 4550 4000
-F 0 "#PWR087" H 4550 3830 50  0001 C CNN
+F 0 "#PWR086" H 4550 3830 50  0001 C CNN
 F 1 "DGND" H 4550 3900 50  0000 C CNN
 F 2 "" H 4550 4100 60  0000 C CNN
