File: Master_Board/V4/TempSens.sch (KiCad schematic (older format))
At the start: 3 parts

Commit message: Repair broken librairy references
Parts:
- C601: symbol 885012107015 -> Capacitors:885012107015
- R601: symbol RC0805JR-0733KL -> Resistors:RC0805JR-0733KL
- RT601: symbol NCP15WB473F03RC -> Sensors:NCP15WB473F03RC
Changed lines of the file:
@@
 NTC_1_ADC
 $Comp
-L RC0805JR-0733KL R601
+L Resistors:RC0805JR-0733KL R601
 U 1 1 5947B1C3
 P 6000 3400
@@
 $EndComp
 $Comp
-L 885012107015 C601
+L Capacitors:885012107015 C601
 U 1 1 5947B23E
 P 5450 3700
@@
 $EndComp
 $Comp
-L DGND #PWR0601
+L Power_Port:DGND #PWR0601
 U 1 1 5947B3D9
 P 5100 4100
@@
 	5100 3900 5100 4000
 $Comp
-L NCP15WB473F03RC RT601
+L Sensors:NCP15WB473F03RC RT601
 U 1 1 5947BCAB
 P 4650 3450
