File: Master_Board/V4/CAN1.sch (KiCad schematic (older format))
At the start: 15 parts, among them J401 649006227222, U401 SN65HVD232DR

Commit message: Repair broken librairy references
Parts:
- C401: symbol 885012207080 -> Capacitors:885012207080
- C402: symbol 885012107015 -> Capacitors:885012107015
- C403: symbol 885012207098 -> Capacitors:885012207098
- C404, C405: symbol 885012007053 -> Capacitors:885012007053
- D401: symbol D1213A-02SOL-7 -> Diodes:D1213A-02SOL-7
- J401: symbol 649006227222 -> Connectors:649006227222
- R401: symbol RC0805JR-07100RL -> Resistors:RC0805JR-07100RL
- R402: symbol RC1206JR-07120RL -> Resistors:RC1206JR-07120RL
- R403: symbol RC0805JR-070RL -> Resistors:RC0805JR-070RL
- TP401, TP402, TP403, TP404: symbol Test_Point_THM -> Connectors:Test_Point_THM
- U401: symbol SN65HVD232DR -> Interface:SN65HVD232DR
Changed lines of the file:
@@
 $EndDescr
 $Comp
-L VDD #PWR0403
+L Power_Port:VDD #PWR0403
 U 1 1 58F7D88D
 P 2900 2900
@@
 $EndComp
 $Comp
-L DGND #PWR0404
+L Power_Port:DGND #PWR0404
 U 1 1 597095FB
 P 2900 4600
@@
 $EndComp
 $Comp
-L DGND #PWR0401
+L Power_Port:DGND #PWR0401
 U 1 1 58F7E8BB
 P 1800 4600
@@
 	1800 4100 1800 4000
 $Comp
-L 885012207098 C403
+L Capacitors:885012207098 C403
 U 1 1 58F7ED24
 P 2700 3400
@@
 Connection ~ 2900 3400
 $Comp
-L DGND #PWR0402
+L Power_Port:DGND #PWR0402
 U 1 1 58F7EE1E
 P 2400 3600
@@
 	2400 3400 2500 3400
 $Comp
-L 885012107015 C402
+L Capacitors:885012107015 C402
 U 1 1 59709601
 P 2700 3000
@@
 Connection ~ 2400 3400
 $Comp
-L D1213A-02SOL-7 D401
+L Diodes:D1213A-02SOL-7 D401
 U 1 1 58F7FD89
 P 6700 4100
@@
 $EndComp
 $Comp
-L DGND #PWR0407
+L Power_Port:DGND #PWR0407
 U 1 1 58F7FE79
 P 7200 4500
@@
 	7200 4100 7200 4400
 $Comp
-L DGND #PWR0406
+L Power_Port:DGND #PWR0406
 U 1 1 58F80304
 P 6200 4900
@@
 $EndComp
 $Comp
-L DGND #PWR0405
+L Power_Port:DGND #PWR0405
 U 1 1 58F80376
 P 5600 4900
@@
 NoConn ~ 3800 4400
 $Comp
-L Test_Point_THM TP403
+L Connectors:Test_Point_THM TP403
 U 1 1 58F8F52D
 P 4200 3600
@@
 $EndComp
 $Comp
-L Test_Point_THM TP404
+L Connectors:Test_Point_THM TP404
 U 1 1 59709603
 P 4200 4500
@@
 CAN_H
 $Comp
-L Test_Point_THM TP401
+L Connectors:Test_Point_THM TP401
 U 1 1 58F8FB78
 P 1900 3700
@@
 TXD
 $Comp
-L Test_Point_THM TP402
+L Connectors:Test_Point_THM TP402
 U 1 1 59709605
 P 2500 4600
@@
 Connection ~ 2500 4200
 $Comp
-L RC1206JR-07120RL R402
+L Resistors:RC1206JR-07120RL R402
 U 1 1 59709606
 P 4600 5100
@@
 Connection ~ 6200 4000
 $Comp
-L SN65HVD232DR U401
+L Interface:SN65HVD232DR U401
 U 1 1 5938BD72
 P 3500 4400
@@
 	6300 3100 6300 4000
 $Comp
-L DGND #PWR0409
+L Power_Port:DGND #PWR0409
 U 1 1 593D5B09
 P 7400 3400
@@
 	7400 3200 7400 3300
 $Comp
-L CAN_PWR #PWR0408
+L Power_Port:CAN_PWR #PWR0408
 U 1 1 593D5B11
 P 7350 2800
@@
 CAN_N
 $Comp
-L RC0805JR-07100RL R401
+L Resistors:RC0805JR-07100RL R401
 U 1 1 597A434D
 P 1500 4000
@@
 $EndComp
 $Comp
-L 885012207080 C401
+L Capacitors:885012207080 C401
 U 1 1 597A447F
 P 1800 4200
@@
 $EndComp
 $Comp
-L 885012007053 C404
+L Capacitors:885012007053 C404
 U 1 1 597A4A3D
 P 5600 4600
@@
 $EndComp
 $Comp
-L 885012007053 C405
+L Capacitors:885012007053 C405
 U 1 1 597A4B6F
 P 6200 4600
@@
 $EndComp
 $Comp
-L 649006227222 J401
+L Connectors:649006227222 J401
 U 1 1 597A4DAE
 P 6900 3200
@@
 	6700 3000 6300 3000
 $Comp
-L RC0805JR-070RL R403
+L Resistors:RC0805JR-070RL R403
 U 1 1 597A4F67
 P 7800 3100
@@
 Shield1
 $Comp
-L DGND #PWR0410
+L Power_Port:DGND #PWR0410
 U 1 1 597A52DE
 P 8100 3400

Commit message: Add pull-up and connector to Master V4 circuit
Connections:
- wire segments 40 -> 54
Changed lines of the file:
@@
 RXD
 Wire Wire Line
-	2300 4200 3100 4200
+	2300 4200 2500 4200
 Wire Wire Line
 	2900 4500 2900 4400
@@
 	2900 3800 3100 3800
 Wire Wire Line
-	1700 4000 3100 4000
+	1700 4000 1800 4000
 Connection ~ 1800 4000
 Wire Wire Line
@@
 	2900 3400 2800 3400
 Wire Wire Line
-	2900 2900 2900 3800
+	2900 2900 2900 3000
 Connection ~ 2900 3400
 $Comp
@@
 	2500 3000 2400 3000
 Wire Wire Line
-	2400 3000 2400 3500
+	2400 3000 2400 3400
 Connection ~ 2400 3400
 $Comp
@@
 	6200 4700 6200 4800
 Wire Wire Line
-	3800 4200 6400 4200
-Wire Wire Line
-	3800 4000 6400 4000
+	3800 4200 4200 4200
+Wire Wire Line
+	3800 4000 4200 4000
 Connection ~ 6300 4000
 Wire Wire Line
@@
 Wire Wire Line
 	8100 3100 8100 3300
+Wire Wire Line
+	1800 4000 1900 4000
+Wire Wire Line
+	2900 3400 2900 3800
+Wire Wire Line
+	2900 3000 2900 3400
+Wire Wire Line
+	2400 3400 2400 3500
+Wire Wire Line
+	6300 4000 6400 4000
+Wire Wire Line
+	4400 4000 6200 4000
+Wire Wire Line
+	4800 4200 5600 4200
+Wire Wire Line
+	4200 4200 4800 4200
+Wire Wire Line
+	4200 4000 4400 4000
+Wire Wire Line
+	1900 4000 3100 4000
+Wire Wire Line
+	2500 4200 3100 4200
+Wire Wire Line
+	5600 4200 6100 4200
+Wire Wire Line
+	6100 4200 6400 4200
+Wire Wire Line
+	6200 4000 6300 4000
 $EndSCHEMATC
