File: Master_Board/V4/CAN2.sch (KiCad schematic (older format))
At the start: 13 parts, among them U501 SN65HVD232DR

Commit message: Repair broken librairy references
Parts:
- C501: symbol 885012207080 -> Capacitors:885012207080
- C502: symbol 885012107015 -> Capacitors:885012107015
- C503: symbol 885012207098 -> Capacitors:885012207098
- C504, C505: symbol 885012007053 -> Capacitors:885012007053
- D501: symbol D1213A-02SOL-7 -> Diodes:D1213A-02SOL-7
- R501: symbol RC0805JR-07100RL -> Resistors:RC0805JR-07100RL
- R502: symbol RC1206JR-07120RL -> Resistors:RC1206JR-07120RL
- TP501, TP502, TP503, TP504: symbol Test_Point_THM -> Connectors:Test_Point_THM
- U501: symbol SN65HVD232DR -> Interface:SN65HVD232DR
Changed lines of the file:
@@
 $EndDescr
 $Comp
-L VDD #PWR0503
+L Power_Port:VDD #PWR0503
 U 1 1 597095FA
 P 2900 2900
@@
 $EndComp
 $Comp
-L DGND #PWR0504
+L Power_Port:DGND #PWR0504
 U 1 1 58F7D8B1
 P 2900 4600
@@
 $EndComp
 $Comp
-L DGND #PWR0501
+L Power_Port:DGND #PWR0501
 U 1 1 597095FE
 P 1800 4600
@@
 RXD
 $Comp
-L 885012207098 C503
+L Capacitors:885012207098 C503
 U 1 1 597095FF
 P 2700 3400
@@
 $EndComp
 $Comp
-L DGND #PWR0502
+L Power_Port:DGND #PWR0502
 U 1 1 59709600
 P 2400 3600
@@
 $EndComp
 $Comp
-L 885012107015 C502
+L Capacitors:885012107015 C502
 U 1 1 58F7F5F6
 P 2700 3000
@@
 $EndComp
 $Comp
-L D1213A-02SOL-7 D501
+L Diodes:D1213A-02SOL-7 D501
 U 1 1 58F808C0
 P 7000 4100
@@
 $EndComp
 $Comp
-L DGND #PWR0506
+L Power_Port:DGND #PWR0506
 U 1 1 58F808C6
 P 6050 4900
@@
 $EndComp
 $Comp
-L DGND #PWR0505
+L Power_Port:DGND #PWR0505
 U 1 1 58F808CC
 P 5350 4900
@@
 $EndComp
 $Comp
-L DGND #PWR0507
+L Power_Port:DGND #PWR0507
 U 1 1 58F81672
 P 7500 4400
@@
 NoConn ~ 3800 4400
 $Comp
-L Test_Point_THM TP503
+L Connectors:Test_Point_THM TP503
 U 1 1 59709602
 P 4200 3600
@@
 $EndComp
 $Comp
-L Test_Point_THM TP504
+L Connectors:Test_Point_THM TP504
 U 1 1 58F8F64E
 P 4200 4500
@@
 CAN_H
 $Comp
-L Test_Point_THM TP501
+L Connectors:Test_Point_THM TP501
 U 1 1 59709604
 P 1900 3700
@@
 $EndComp
 $Comp
-L Test_Point_THM TP502
+L Connectors:Test_Point_THM TP502
 U 1 1 58F8FE19
 P 2500 4600
@@
 $EndComp
 $Comp
-L RC1206JR-07120RL R502
+L Resistors:RC1206JR-07120RL R502
 U 1 1 58FBF6A8
 P 4600 5100
@@
 $EndComp
 $Comp
-L SN65HVD232DR U501
+L Interface:SN65HVD232DR U501
 U 1 1 59709607
 P 3500 4400
@@
 	7500 4100 7500 4300
 $Comp
-L RC0805JR-07100RL R501
+L Resistors:RC0805JR-07100RL R501
 U 1 1 597A6225
 P 1500 4000
@@
 $EndComp
 $Comp
-L 885012207080 C501
+L Capacitors:885012207080 C501
 U 1 1 597A62A4
 P 1800 4300
@@
 $EndComp
 $Comp
-L 885012007053 C504
+L Capacitors:885012007053 C504
 U 1 1 597A66F1
 P 5350 4600
@@
 $EndComp
 $Comp
-L 885012007053 C505
+L Capacitors:885012007053 C505
 U 1 1 597A67AE
 P 6050 4600

Commit message: Remove big crappy connector and remap 12V
Connections:
- wire segments 32 -> 46
Changed lines of the file:
@@
 $Descr USLetter 11000 8500
 encoding utf-8
-Sheet 5 11
+Sheet 5 9
 Title "CAN2"
 Date "2017-06-25"
@@
 	1200 4000 1300 4000
 Wire Wire Line
-	2300 4200 3100 4200
+	2300 4200 2500 4200
 Wire Wire Line
 	2900 4500 2900 4400
@@
 	2900 3800 3100 3800
 Wire Wire Line
-	1700 4000 3100 4000
+	1700 4000 1800 4000
 Connection ~ 1800 4000
 Wire Wire Line
@@
 	2900 3400 2800 3400
 Wire Wire Line
-	2900 2900 2900 3800
+	2900 2900 2900 3000
 Connection ~ 2900 3400
 Wire Wire Line
@@
 	2500 3000 2400 3000
 Wire Wire Line
-	2400 3000 2400 3500
+	2400 3000 2400 3400
 Connection ~ 2400 3400
 Wire Wire Line
@@
 	5350 4000 5350 4400
 Wire Wire Line
-	3800 4200 6700 4200
+	3800 4200 4200 4200
 Wire Wire Line
 	6050 4200 6050 4400
@@
 Connection ~ 2500 4200
 Wire Wire Line
-	3800 4000 6700 4000
+	3800 4000 4200 4000
 Connection ~ 6050 4200
 Connection ~ 5350 4000
@@
 	0    1    1    0
 $EndComp
+Wire Wire Line
+	1800 4000 1900 4000
+Wire Wire Line
+	2900 3400 2900 3800
+Wire Wire Line
+	2900 3000 2900 3400
+Wire Wire Line
+	2400 3400 2400 3500
+Wire Wire Line
+	4400 4000 5350 4000
+Wire Wire Line
+	4800 4200 6050 4200
+Wire Wire Line
+	4200 4200 4800 4200
+Wire Wire Line
+	4200 4000 4400 4000
+Wire Wire Line
+	1900 4000 3100 4000
+Wire Wire Line
+	2500 4200 3100 4200
+Wire Wire Line
+	6050 4200 6450 4200
+Wire Wire Line
+	5350 4000 6450 4000
+Wire Wire Line
+	6450 4000 6700 4000
+Wire Wire Line
+	6450 4200 6700 4200
 $EndSCHEMATC
