File: Master_Board/V4/VoltageSense.sch (KiCad schematic (older format))
At the start: 41 parts, among them J901 649002227222, J902 649002227222, J903 649002227222, J904 649002227222, U901 ACPL-C87A-500E, U902 NCS1S2405SC, U903 ACPL-C87A-500E, U904 LMV321RILT, U905 LMV321RILT

Commit message: Repair broken librairy references
Parts:
- C901, C902, C912, C913, C914, C915: symbol 885012207080 -> Capacitors:885012207080
- C903, C910: symbol 860020472006 -> Capacitors:860020472006
- C904, C905, C906, C907, C908, C909: symbol 885012207098 -> Capacitors:885012207098
- C911: symbol 885012207075 -> Capacitors:885012207075
- D901, D902: symbol NRVBS3200T3G -> Diodes:NRVBS3200T3G
- D903: symbol SD0805S020S1R0 -> Capacitors:SD0805S020S1R0
- J901, J902, J903, J904: symbol 649002227222 -> Connectors:649002227222
- L901: symbol 744052471 -> Inductors:744052471
- R901, R903: symbol RC0805JR-071ML -> Resistors:RC0805JR-071ML
- R902, R904, R905, R906, R907, R908: symbol RC0805JR-0710KL -> Resistors:RC0805JR-0710KL
- R909, R910, R911, R912: symbol RC0805JR-0715KL -> Resistors:RC0805JR-0715KL
- R913: symbol RC0805JR-07470RL -> Resistors:RC0805JR-07470RL
- U901, U903: symbol ACPL-C87A-500E -> Sensors:ACPL-C87A-500E
- U902: symbol NCS1S2405SC -> PMIC:NCS1S2405SC
- U904, U905: symbol LMV321RILT -> Amplifiers:LMV321RILT
Changed lines of the file:
@@
 $EndDescr
 $Comp
-L 649002227222 J903
+L Connectors:649002227222 J903
 U 1 1 59455561
 P 1900 4450
@@
 $EndComp
 $Comp
-L 649002227222 J904
+L Connectors:649002227222 J904
 U 1 1 594555CF
 P 1900 6050
@@
 NoConn ~ 2100 5950
 $Comp
-L DGND #PWR01108
+L Power_Port:DGND #PWR01108
 U 1 1 5949C56B
 P 5500 5750
@@
 $EndComp
 $Comp
-L 885012207098 C909
+L Capacitors:885012207098 C909
 U 1 1 5949C815
 P 5800 5250
@@
 $EndComp
 $Comp
-L 885012207098 C905
+L Capacitors:885012207098 C905
 U 1 1 5949CA2A
 P 3950 5250
@@
 $EndComp
 $Comp
-L LMV321RILT U905
+L Amplifiers:LMV321RILT U905
 U 1 1 5949D239
 P 7300 5300
@@
 $EndComp
 $Comp
-L 885012207080 C902
+L Capacitors:885012207080 C902
 U 1 1 5949D391
 P 3500 5350
@@
 $EndComp
 $Comp
-L RC0805JR-0710KL R904
+L Resistors:RC0805JR-0710KL R904
 U 1 1 5949D586
 P 2650 5300
@@
 $EndComp
 $Comp
-L RC0805JR-071ML R903
+L Resistors:RC0805JR-071ML R903
 U 1 1 5949E1E3
 P 2650 4700
@@
 $EndComp
 $Comp
-L 885012207080 C912
+L Capacitors:885012207080 C912
 U 1 1 5949E758
 P 7300 6050
@@
 $EndComp
 $Comp
-L RC0805JR-0710KL R908
+L Resistors:RC0805JR-0710KL R908
 U 1 1 5949EEEC
 P 6400 5650
@@
 $EndComp
 $Comp
-L 885012207080 C914
+L Capacitors:885012207080 C914
 U 1 1 5949F23C
 P 7500 4650
@@
 VSENSE_BP
 $Comp
-L DGND #PWR01114
+L Power_Port:DGND #PWR01114
 U 1 1 5949FCE5
 P 7300 5750
@@
 $EndComp
 $Comp
-L DGND #PWR01116
+L Power_Port:DGND #PWR01116
 U 1 1 594A0EB3
 P 8000 4650
@@
 $EndComp
 $Comp
-L 5V #PWR01107
+L Power_Port:5V #PWR01107
 U 1 1 594A3B0E
 P 5500 4800
@@
 $EndComp
 $Comp
-L NCS1S2405SC U902
+L PMIC:NCS1S2405SC U902
 U 1 1 594A7534
 P 4900 3650
@@
 $EndComp
 $Comp
-L DGND #PWR01104
+L Power_Port:DGND #PWR01104
 U 1 1 594A76E3
 P 5400 4350
@@
 VSENSE_EN
 $Comp
-L 649002227222 J901
+L Connectors:649002227222 J901
 U 1 1 594A896F
 P 1900 850
@@
 $EndComp
 $Comp
-L 649002227222 J902
+L Connectors:649002227222 J902
 U 1 1 594A897A
 P 1900 2450
@@
 NoConn ~ 2100 2350
 $Comp
-L DGND #PWR01106
+L Power_Port:DGND #PWR01106
 U 1 1 594A8995
 P 5500 2150
@@
 $EndComp
 $Comp
-L 885012207098 C908
+L Capacitors:885012207098 C908
 U 1 1 594A89A3
 P 5800 1650
@@
 $EndComp
 $Comp
-L 885012207098 C904
+L Capacitors:885012207098 C904
 U 1 1 594A89B1
 P 3950 1650
@@
 $EndComp
 $Comp
-L LMV321RILT U904
+L Amplifiers:LMV321RILT U904
 U 1 1 594A89BC
 P 7300 1700
@@
 $EndComp
 $Comp
-L 885012207080 C901
+L Capacitors:885012207080 C901
 U 1 1 594A89CA
 P 3500 1750
@@
 $EndComp
 $Comp
-L RC0805JR-0710KL R902
+L Resistors:RC0805JR-0710KL R902
 U 1 1 594A89D8
 P 2650 1700
@@
 $EndComp
 $Comp
-L RC0805JR-071ML R901
+L Resistors:RC0805JR-071ML R901
 U 1 1 594A89E6
 P 2650 1100
@@
 $EndComp
 $Comp
-L RC0805JR-0710KL R905
+L Resistors:RC0805JR-0710KL R905
 U 1 1 594A89F4
 P 6400 1350
@@
 $EndComp
 $Comp
-L 885012207080 C913
+L Capacitors:885012207080 C913
 U 1 1 594A8A02
 P 7350 2750
@@
 $EndComp
 $Comp
-L RC0805JR-0710KL R906
+L Resistors:RC0805JR-0710KL R906
 U 1 1 594A8A10
 P 6400 2050
@@
 $EndComp
 $Comp
-L 885012207080 C915
+L Capacitors:885012207080 C915
 U 1 1 594A8A2C
 P 7550 1000
@@
 VSENSE_MPPT
 $Comp
-L DGND #PWR01112
+L Power_Port:DGND #PWR01112
 U 1 1 594A8A41
 P 7300 2150
@@
 $EndComp
 $Comp
-L DGND #PWR01115
+L Power_Port:DGND #PWR01115
 U 1 1 594A8A81
 P 8000 950
@@
 $EndComp
 $Comp
-L 5V #PWR01105
+L Power_Port:5V #PWR01105
 U 1 1 594A8A88
 P 5500 1200
@@
 5V_ISO
 $Comp
-L RC0805JR-07470RL R913
+L Resistors:RC0805JR-07470RL R913
 U 1 1 594841DD
 P 7750 3450
@@
 	7950 3450 8150 3450
 $Comp
-L 885012207075 C911
+L Capacitors:885012207075 C911
 U 1 1 594853E0
 P 6950 3950
@@
 	6800 3650 7100 3650
 $Comp
-L DGND #PWR01109
+L Power_Port:DGND #PWR01109
 U 1 1 59486B2F
 P 6950 4200
@@
 Isolated
 $Comp
-L SD0805S020S1R0 D903
+L Capacitors:SD0805S020S1R0 D903
 U 1 1 594E14E6
 P 5800 3450
@@
 Connection ~ 4300 5550
 $Comp
-L RC0805JR-0710KL R907
+L Resistors:RC0805JR-0710KL R907
 U 1 1 5949E56D
 P 6400 4950
@@
 $EndComp
 $Comp
-L RC0805JR-0715KL R909
+L Resistors:RC0805JR-0715KL R909
 U 1 1 59539105
 P 7300 2500
@@
 $EndComp
 $Comp
-L RC0805JR-0715KL R910
+L Resistors:RC0805JR-0715KL R910
 U 1 1 59539316
 P 7350 6300
@@
 $EndComp
 $Comp
-L RC0805JR-0715KL R912
+L Resistors:RC0805JR-0715KL R912
 U 1 1 595393DC
 P 7600 800
@@
 $EndComp
 $Comp
-L RC0805JR-0715KL R911
+L Resistors:RC0805JR-0715KL R911
 U 1 1 5953A5C1
 P 7550 4450
@@
 $EndComp
 $Comp
-L ACPL-C87A-500E U901
+L Sensors:ACPL-C87A-500E U901
 U 1 1 59616333
 P 4900 1900
@@
 $EndComp
 $Comp
-L ACPL-C87A-500E U903
+L Sensors:ACPL-C87A-500E U903
 U 1 1 59616A29
 P 4900 5500
@@
 $EndComp
 $Comp
-L 885012207098 C906
+L Capacitors:885012207098 C906
 U 1 1 5962C2AF
 P 4150 3700
@@
 $EndComp
 $Comp
-L 885012207098 C907
+L Capacitors:885012207098 C907
 U 1 1 5962C48A
 P 5600 3950
@@
 Connection ~ 4150 3450
 $Comp
-L 860020472006 C903
+L Capacitors:860020472006 C903
 U 1 1 59632F1A
 P 3700 3700
@@
 $EndComp
 $Comp
-L 860020472006 C910
+L Capacitors:860020472006 C910
 U 1 1 5963389F
 P 6050 3950
@@
 Connection ~ 6050 3650
 $Comp
-L 744052471 L901
+L Inductors:744052471 L901
 U 1 1 5963F05F
 P 6600 3650
@@
 $EndComp
 $Comp
-L NRVBS3200T3G D901
+L Diodes:NRVBS3200T3G D901
 U 1 1 595D8F52
 P 2450 750
@@
 	2250 750  2100 750
 $Comp
-L NRVBS3200T3G D902
+L Diodes:NRVBS3200T3G D902
 U 1 1 595DA6B1
 P 2450 4350
@@
 2V to 3.3V
 $Comp
-L AGND #PWR01103
+L Power_Port:AGND #PWR01103
 U 1 1 59A79917
 P 4350 4350
@@
 $EndComp
 $Comp
-L AGND #PWR01102
+L Power_Port:AGND #PWR01102
 U 1 1 59A799A4
 P 4300 5700
@@
 $EndComp
 $Comp
-L AGND #PWR01101
+L Power_Port:AGND #PWR01101
 U 1 1 59A7A8D9
 P 4300 2100
@@
 Connection ~ 4350 3850
 $Comp
-L PWR_FLAG #FLG01101
+L Power_Port:PWR_FLAG #FLG01101
 U 1 1 59A7E10D
 P 4250 4150
@@
 Connection ~ 4350 4150
 $Comp
-L 12V #PWR01110
+L Power_Port:12V #PWR01110
 U 1 1 594A78A1
 P 7100 3650
@@
 $EndComp
 $Comp
-L VDD #PWR01113
+L Power_Port:VDD #PWR01113
 U 1 1 5A91D90D
 P 7300 5000
@@
 $EndComp
 $Comp
-L VDD #PWR01111
+L Power_Port:VDD #PWR01111
 U 1 1 5A91D973
 P 7300 1400

Commit message: Add pull-up and connector to Master V4 circuit
Connections:
- wire segments 121 -> 165
Changed lines of the file:
@@
 	2650 6050 2100 6050
 Wire Wire Line
-	5400 5450 5800 5450
+	5400 5450 5500 5450
 Wire Wire Line
 	5500 5450 5500 5650
 Wire Wire Line
-	3950 5450 4400 5450
-Wire Wire Line
-	4300 5350 4300 5600
+	3950 5450 4300 5450
+Wire Wire Line
+	4300 5350 4300 5450
 Wire Wire Line
 	5500 4800 5500 5150
 Wire Wire Line
-	5400 5150 5800 5150
+	5400 5150 5500 5150
 Connection ~ 5500 5150
 Connection ~ 5500 5450
@@
 	5650 5350 5650 5650
 Wire Wire Line
-	3950 5150 4400 5150
+	3950 5150 4300 5150
 Connection ~ 4300 5450
 Wire Wire Line
@@
 	4150 5250 4150 5000
 Wire Wire Line
-	4150 5000 2650 5000
+	4150 5000 3500 5000
 Wire Wire Line
 	3500 5000 3500 5150
 Wire Wire Line
-	2650 5550 4300 5550
+	2650 5550 3500 5550
 Wire Wire Line
 	3500 5550 3500 5450
 Wire Wire Line
-	2650 4900 2650 5100
+	2650 4900 2650 5000
 Connection ~ 3500 5000
 Wire Wire Line
-	2650 5500 2650 6050
+	2650 5500 2650 5550
 Connection ~ 3500 5550
 Connection ~ 2650 5550
@@
 	5650 4950 6200 4950
 Wire Wire Line
-	6600 4950 7000 4950
+	6600 4950 6700 4950
 Wire Wire Line
 	7000 4950 7000 5200
@@
 	5650 5650 6200 5650
 Wire Wire Line
-	6600 5650 7000 5650
+	6600 5650 6700 5650
 Wire Wire Line
 	7000 5650 7000 5400
 Wire Wire Line
-	7600 5300 8100 5300
+	7600 5300 7950 5300
 Connection ~ 4300 5150
 Wire Wire Line
-	6700 6050 7200 6050
-Wire Wire Line
-	7500 6050 7950 6050
+	6700 6050 7050 6050
+Wire Wire Line
+	7500 6050 7600 6050
 Connection ~ 6700 4950
 Wire Wire Line
@@
 	7700 4650 7800 4650
 Wire Wire Line
-	6700 4450 7350 4450
+	6700 4450 7300 4450
 Connection ~ 6700 5650
 Wire Wire Line
-	7750 4450 8000 4450
-Wire Wire Line
-	5400 3850 5400 4250
-Wire Wire Line
-	3450 3450 4400 3450
-Wire Wire Line
-	5400 3650 6400 3650
+	7750 4450 7800 4450
+Wire Wire Line
+	5400 3850 5400 4150
+Wire Wire Line
+	3450 3450 3700 3450
+Wire Wire Line
+	5400 3650 5600 3650
 Wire Wire Line
 	2650 2450 2100 2450
 Wire Wire Line
-	5400 1850 5800 1850
+	5400 1850 5500 1850
 Wire Wire Line
 	5500 1850 5500 2050
 Wire Wire Line
-	3950 1850 4400 1850
-Wire Wire Line
-	4300 1750 4300 2000
+	3950 1850 4300 1850
+Wire Wire Line
+	4300 1750 4300 1850
 Wire Wire Line
 	5500 1200 5500 1550
 Wire Wire Line
-	5400 1550 5800 1550
+	5400 1550 5500 1550
 Connection ~ 5500 1550
 Connection ~ 5500 1850
@@
 	5650 1750 5650 2050
 Wire Wire Line
-	3950 1550 4400 1550
+	3950 1550 4300 1550
 Connection ~ 4300 1850
 Wire Wire Line
@@
 	4150 1650 4150 1400
 Wire Wire Line
-	4150 1400 2650 1400
+	4150 1400 3500 1400
 Wire Wire Line
 	3500 1400 3500 1550
 Wire Wire Line
-	2650 1950 4300 1950
+	2650 1950 3500 1950
 Wire Wire Line
 	3500 1950 3500 1850
 Wire Wire Line
-	2650 1300 2650 1500
+	2650 1300 2650 1400
 Connection ~ 3500 1400
 Wire Wire Line
-	2650 1900 2650 2450
+	2650 1900 2650 1950
 Connection ~ 3500 1950
 Connection ~ 2650 1950
@@
 	5650 1350 6200 1350
 Wire Wire Line
-	6600 1350 7000 1350
+	6600 1350 6700 1350
 Wire Wire Line
 	7000 1350 7000 1600
@@
 	5650 2050 6200 2050
 Wire Wire Line
-	6600 2050 7000 2050
+	6600 2050 6700 2050
 Wire Wire Line
 	7000 2050 7000 1800
 Wire Wire Line
-	7600 1700 8100 1700
+	7600 1700 7950 1700
 Connection ~ 4300 1550
 Connection ~ 6700 1350
@@
 	7750 1000 7850 1000
 Wire Wire Line
-	6700 800  7400 800
+	6700 800  7350 800
 Connection ~ 6700 2050
 Wire Wire Line
-	7800 800  8000 800
+	7800 800  7850 800
 Wire Wire Line
 	4300 1550 4300 1200
@@
 $EndComp
 Wire Wire Line
-	6800 3650 7100 3650
+	6800 3650 6950 3650
 $Comp
 L Power_Port:DGND #PWR01109
@@
 	5600 4050 5600 4150
 Wire Wire Line
-	5400 4150 6050 4150
+	5400 4150 5600 4150
 Connection ~ 5400 4150
 Wire Wire Line
-	3700 3850 4400 3850
+	3700 3850 4150 3850
 Wire Wire Line
 	6950 4100 6950 4050
@@
 	7600 6050 7600 6300
 Wire Wire Line
-	7500 2500 7950 2500
+	7500 2500 7700 2500
 Wire Wire Line
 	7950 2500 7950 1700
@@
 	6700 2050 6700 2500
 Wire Wire Line
-	6700 2500 7100 2500
+	6700 2500 6950 2500
 Wire Wire Line
 	6950 2500 6950 2750
@@
 $EndComp
 Wire Wire Line
-	4350 4250 4350 3850
+	4350 4250 4350 4150
 Connection ~ 4350 3850
 $Comp
@@
 	1    0    0    -1
 $EndComp
+Wire Wire Line
+	5500 5150 5800 5150
+Wire Wire Line
+	5500 5450 5800 5450
+Wire Wire Line
+	4300 5450 4400 5450
+Wire Wire Line
+	4300 5450 4300 5550
+Wire Wire Line
+	3500 5000 2650 5000
+Wire Wire Line
+	3500 5550 4300 5550
+Wire Wire Line
+	2650 5550 2650 6050
+Wire Wire Line
+	2650 5000 2650 5100
+Wire Wire Line
+	4300 5150 4400 5150
+Wire Wire Line
+	6700 4950 7000 4950
+Wire Wire Line
+	6700 5650 7000 5650
+Wire Wire Line
+	5500 1550 5800 1550
+Wire Wire Line
+	5500 1850 5800 1850
+Wire Wire Line
+	4300 1850 4400 1850
+Wire Wire Line
+	4300 1850 4300 1950
+Wire Wire Line
+	3500 1400 2650 1400
+Wire Wire Line
+	3500 1950 4300 1950
+Wire Wire Line
+	2650 1950 2650 2450
+Wire Wire Line
+	2650 1400 2650 1500
+Wire Wire Line
+	4300 1550 4400 1550
+Wire Wire Line
+	6700 1350 7000 1350
+Wire Wire Line
+	6700 2050 7000 2050
+Wire Wire Line
+	4300 1950 4300 2000
+Wire Wire Line
+	4300 5550 4300 5600
+Wire Wire Line
+	5400 4150 5400 4250
+Wire Wire Line
+	6950 3650 7100 3650
+Wire Wire Line
+	4150 3850 4350 3850
+Wire Wire Line
+	3700 3450 4150 3450
+Wire Wire Line
+	4150 3450 4400 3450
+Wire Wire Line
+	5600 4150 6050 4150
+Wire Wire Line
+	5600 3650 6050 3650
+Wire Wire Line
+	6050 3650 6400 3650
+Wire Wire Line
+	7300 4450 7350 4450
+Wire Wire Line
+	7800 4450 8000 4450
+Wire Wire Line
+	7350 800  7400 800
+Wire Wire Line
+	7850 800  8000 800
+Wire Wire Line
+	7950 1700 8100 1700
+Wire Wire Line
+	6950 2500 7100 2500
+Wire Wire Line
+	7700 2500 7950 2500
+Wire Wire Line
+	7950 5300 8100 5300
+Wire Wire Line
+	7600 6050 7950 6050
+Wire Wire Line
+	7050 6050 7200 6050
+Wire Wire Line
+	4350 3850 4400 3850
+Wire Wire Line
+	4350 4150 4350 3850
 $EndSCHEMATC

Commit message: add negative contactor reading and start USB feature
Parts:
- added J?: 649002227222, Connectors:649002227222, symbol Connectors:649002227222
- added R? (x2): RC0805JR-074K7L, Resistors:R0805, symbol Resistors:RC0805JR-074K7L
- added U?: CPC1117NTR, IC:4-SOP, symbol Isolators:CPC1117NTR
Connections:
- net labels added: 5V_HP, STATE_RELAY_NEG
- net labels removed: 5V_ISO
- wire segments 165 -> 179

Commit message: Update of schematic for master E10.1
Parts:
- removed J901, J902, J903, J904, J?: 649002227222, Connectors:649002227222, symbol Connectors:649002227222
Connections:
- net labels added: HV_HIGHSIDE-, HV_LOWSIDE+, HV_MPPT+
- net labels removed: BP-HV-, MPPT-HV-
- wire segments 179 -> 174
- no-connect marks 4 -> 0
Changed lines of the file:
@@
 Comment4 ""
 $EndDescr
-$Comp
-L Connectors:649002227222 J903
-U 1 1 59455561
-P 1900 3950
-F 0 "J903" H 1900 4150 60  0000 C CNN
-F 1 "649002227222" H 1900 3800 60  0000 C CNN
-F 2 "Connectors:649002227222" H 1900 3050 60  0001 C CNN
-F 3 "http://katalog.we-online.de/em/datasheet/649016227222.pdf" H 1900 2950 60  0001 C CNN
-F 4 "Digikey" H 1900 3550 60  0001 C CNN "Supplier"
-F 5 "732-1937-ND" H 1900 3450 60  0001 C CNN "Supplier Part Number"
-F 6 "Wurth Electronics Inc." H 1900 3350 60  0001 C CNN "Manufacturer"
-F 7 "649002227222" H 1900 3250 60  0001 C CNN "Manufacturer Part Number"
-F 8 "HEADER MALE DUAL ANGLE W/MNT 2P" H 1900 3150 60  0001 C CNN "Description"
-	1    1900 3950
-	1    0    0    -1
-$EndComp
-$Comp
-L Connectors:649002227222 J904
-U 1 1 594555CF
-P 1900 5550
-F 0 "J904" H 1900 5750 60  0000 C CNN
-F 1 "649002227222" H 1900 5400 60  0000 C CNN
-F 2 "Connectors:649002227222" H 1900 4650 60  0001 C CNN
-F 3 "http://katalog.we-online.de/em/datasheet/649016227222.pdf" H 1900 4550 60  0001 C CNN
-F 4 "Digikey" H 1900 5150 60  0001 C CNN "Supplier"
-F 5 "732-1937-ND" H 1900 5050 60  0001 C CNN "Supplier Part Number"
-F 6 "Wurth Electronics Inc." H 1900 4950 60  0001 C CNN "Manufacturer"
-F 7 "649002227222" H 1900 4850 60  0001 C CNN "Manufacturer Part Number"
-F 8 "HEADER MALE DUAL ANGLE W/MNT 2P" H 1900 4750 60  0001 C CNN "Description"
-	1    1900 5550
-	1    0    0    -1
-$EndComp
 Text Label 2650 3900 0    60   ~ 0
 BP-HV+
-Text Label 2250 5550 0    60   ~ 0
-BP-HV-
-NoConn ~ 2100 3950
-NoConn ~ 2100 5450
 $Comp
 L Power_Port:DGND #PWR01108
@@
 Text HLabel 8150 3050 2    60   Input ~ 0
 VSENSE_EN
-$Comp
-L Connectors:649002227222 J901
-U 1 1 594A896F
-P 1900 800
-F 0 "J901" H 1900 1000 60  0000 C CNN
-F 1 "649002227222" H 1900 650 60  0000 C CNN
-F 2 "Connectors:649002227222" H 1900 -100 60  0001 C CNN
-F 3 "http://katalog.we-online.de/em/datasheet/649016227222.pdf" H 1900 -200 60  0001 C CNN
-F 4 "Digikey" H 1900 400 60  0001 C CNN "Supplier"
-F 5 "732-1937-ND" H 1900 300 60  0001 C CNN "Supplier Part Number"
-F 6 "Wurth Electronics Inc." H 1900 200 60  0001 C CNN "Manufacturer"
-F 7 "649002227222" H 1900 100 60  0001 C CNN "Manufacturer Part Number"
-F 8 "HEADER MALE DUAL ANGLE W/MNT 2P" H 1900 0   60  0001 C CNN "Description"
-	1    1900 800
-	1    0    0    -1
-$EndComp
-$Comp
-L Connectors:649002227222 J902
-U 1 1 594A897A
-P 1900 2400
-F 0 "J902" H 1900 2600 60  0000 C CNN
-F 1 "649002227222" H 1900 2250 60  0000 C CNN
-F 2 "Connectors:649002227222" H 1900 1500 60  0001 C CNN
-F 3 "http://katalog.we-online.de/em/datasheet/649016227222.pdf" H 1900 1400 60  0001 C CNN
-F 4 "Digikey" H 1900 2000 60  0001 C CNN "Supplier"
-F 5 "732-1937-ND" H 1900 1900 60  0001 C CNN "Supplier Part Number"
-F 6 "Wurth Electronics Inc." H 1900 1800 60  0001 C CNN "Manufacturer"
-F 7 "649002227222" H 1900 1700 60  0001 C CNN "Manufacturer Part Number"
-F 8 "HEADER MALE DUAL ANGLE W/MNT 2P" H 1900 1600 60  0001 C CNN "Description"
-	1    1900 2400
-	1    0    0    -1
-$EndComp
 Text Label 2650 800  0    60   ~ 0
 MPPT-HV+
-Text Label 2150 2400 0    60   ~ 0
-MPPT-HV-
-NoConn ~ 2100 800
-NoConn ~ 2100 2300
 $Comp
 L Power_Port:DGND #PWR01106
@@
 $EndComp
 Wire Wire Line
-	2650 5550 2100 5550
-Wire Wire Line
 	5400 4950 5500 4950
 Wire Wire Line
@@
 	2650 5000 2650 5050
 Connection ~ 3500 5050
-Connection ~ 2650 5050
 Connection ~ 2650 4500
 Wire Wire Line
@@
 Wire Wire Line
 	5400 3250 5600 3250
-Wire Wire Line
-	2650 2400 2100 2400
 Wire Wire Line
 	5400 1800 5500 1800
@@
 	2650 1850 2650 1900
 Connection ~ 3500 1900
-Connection ~ 2650 1900
 Connection ~ 2650 1350
 Wire Wire Line
@@
 	1    0    0    -1
 $EndComp
-Text Notes 1750 3200 0    120  ~ 24
+Text Notes 2200 2850 0    120  ~ 24
 Isolated
 $Comp
@@
 	3500 5050 4300 5050
 Wire Wire Line
-	2650 5050 2650 5550
-Wire Wire Line
 	2650 4500 2650 4600
 Wire Wire Line
@@
 Wire Wire Line
 	3500 1900 4300 1900
-Wire Wire Line
-	2650 1900 2650 2400
 Wire Wire Line
 	2650 1350 2650 1450
@@
 Wire Wire Line
 	5500 7100 5500 6900
-$Comp
-L Connectors:649002227222 J?
-U 1 1 5BC9ED44
-P 3250 6450
-F 0 "J?" H 3250 6650 60  0000 C CNN
-F 1 "649002227222" H 3250 6300 60  0000 C CNN
-F 2 "Connectors:649002227222" H 3250 5550 60  0001 C CNN
-F 3 "http://katalog.we-online.de/em/datasheet/649016227222.pdf" H 3250 5450 60  0001 C CNN
-F 4 "Digikey" H 3250 6050 60  0001 C CNN "Supplier"
-F 5 "732-1937-ND" H 3250 5950 60  0001 C CNN "Supplier Part Number"
-F 6 "Wurth Electronics Inc." H 3250 5850 60  0001 C CNN "Manufacturer"
-F 7 "649002227222" H 3250 5750 60  0001 C CNN "Manufacturer Part Number"
-F 8 "HEADER MALE DUAL ANGLE W/MNT 2P" H 3250 5650 60  0001 C CNN "Description"
-	1    3250 6450
-	1    0    0    -1
-$EndComp
 Wire Wire Line
 	3800 5450 3800 5600
 Wire Wire Line
-	3450 6450 3800 6450
-Wire Wire Line
 	3800 6000 3800 6100
 Wire Wire Line
 	4500 6100 3800 6100
-Connection ~ 3800 6100
-Wire Wire Line
-	3800 6100 3800 6450
 Wire Wire Line
 	4500 6250 4400 6250
@@
 	0    1    1    0
 $EndComp
+Text HLabel 2100 700  0    60   Input ~ 0
+HV_MPPT+
+Text HLabel 2100 3850 0    60   Input ~ 0
+HV_HIGHSIDE-
+Connection ~ 3800 6100
+Text HLabel 2200 6100 0    60   Output ~ 0
+HV_LOWSIDE+
+Wire Wire Line
+	2200 6100 3800 6100
 $EndSCHEMATC

Commit message: Master V4 routed
Parts:
- gave numbers to parts that had none: 3
Changed lines of the file:
@@
 	5600 3700 5450 3700
 $Comp
-L Isolators:CPC1117NTR U?
+L Isolators:CPC1117NTR U906
 U 1 1 5BC70C9E
 P 4900 6200
-F 0 "U?" H 4900 6587 60  0000 C CNN
+F 0 "U906" H 4900 6587 60  0000 C CNN
 F 1 "CPC1117NTR" H 4900 6481 60  0000 C CNN
 F 2 "IC:4-SOP" H 4900 5300 60  0001 C CNN
@@
 $EndComp
 $Comp
-L Power_Port:VDD #PWR?
+L Power_Port:VDD #PWR0112
 U 1 1 5BC78429
 P 5500 5900
-F 0 "#PWR?" H 5500 5750 50  0001 C CNN
+F 0 "#PWR0112" H 5500 5750 50  0001 C CNN
 F 1 "VDD" H 5500 6074 50  0000 C CNN
 F 2 "" H 5500 5900 60  0000 C CNN
@@
 	5500 6250 5900 6250
 $Comp
-L Resistors:RC0805JR-074K7L R?
+L Resistors:RC0805JR-074K7L R915
 U 1 1 5BC969DC
 P 5500 6700
-F 0 "R?" V 5455 6758 60  0000 L CNN
+F 0 "R915" V 5455 6758 60  0000 L CNN
 F 1 "RC0805JR-074K7L" H 5500 6400 50  0001 C CNN
 F 2 "Resistors:R0805" H 5500 5800 30  0001 C CNN
@@
 $EndComp
 $Comp
-L Power_Port:DGND #PWR?
+L Power_Port:DGND #PWR0113
 U 1 1 5BC96B76
 P 5500 7200
-F 0 "#PWR?" H 5500 7030 50  0001 C CNN
+F 0 "#PWR0113" H 5500 7030 50  0001 C CNN
 F 1 "DGND" H 5500 7100 50  0000 C CNN
 F 2 "" H 5500 7300 60  0000 C CNN
@@
 	4400 6250 4400 6400
 $Comp
-L Power_Port:AGND #PWR?
+L Power_Port:AGND #PWR0114
 U 1 1 5BDAB935
 P 4400 6500
-F 0 "#PWR?" H 4400 6330 50  0001 C CNN
+F 0 "#PWR0114" H 4400 6330 50  0001 C CNN
 F 1 "AGND" H 4400 6400 50  0000 C CNN
 F 2 "" H 4400 6600 60  0000 C CNN
@@
 $EndComp
 $Comp
-L Power_Port:5V_HP #PWR?
+L Power_Port:5V_HP #PWR0115
 U 1 1 5BDB444E
 P 3550 3050
-F 0 "#PWR?" H 3550 2900 50  0001 C CNN
+F 0 "#PWR0115" H 3550 2900 50  0001 C CNN
 F 1 "5V_HP" H 3550 3224 50  0000 C CNN
 F 2 "" H 3550 3050 60  0000 C CNN
@@
 	3550 3050 3700 3050
 $Comp
-L Power_Port:5V_HP #PWR?
+L Power_Port:5V_HP #PWR0116
 U 1 1 5BDB47F6
 P 3800 5450
-F 0 "#PWR?" H 3800 5300 50  0001 C CNN
+F 0 "#PWR0116" H 3800 5300 50  0001 C CNN
 F 1 "5V_HP" H 3800 5624 50  0000 C CNN
 F 2 "" H 3800 5450 60  0000 C CNN
@@
 $EndComp
 $Comp
-L Power_Port:5V_HP #PWR?
+L Power_Port:5V_HP #PWR0117
 U 1 1 5BDB4AE8
 P 4300 1150
-F 0 "#PWR?" H 4300 1000 50  0001 C CNN
+F 0 "#PWR0117" H 4300 1000 50  0001 C CNN
 F 1 "5V_HP" H 4300 1324 50  0000 C CNN
 F 2 "" H 4300 1150 60  0000 C CNN
@@
 $EndComp
 $Comp
-L Power_Port:5V_HP #PWR?
+L Power_Port:5V_HP #PWR0118
 U 1 1 5BDB4D26
 P 4300 4300
-F 0 "#PWR?" H 4300 4150 50  0001 C CNN
+F 0 "#PWR0118" H 4300 4150 50  0001 C CNN
 F 1 "5V_HP" H 4300 4474 50  0000 C CNN
 F 2 "" H 4300 4300 60  0000 C CNN
@@
 $EndComp
 $Comp
-L Power_Port:PWR_FLAG #FLG?
+L Power_Port:PWR_FLAG #FLG0102
 U 1 1 5BDC6C40
 P 3800 3050
-F 0 "#FLG?" H 3800 2950 60  0001 C CNN
+F 0 "#FLG0102" H 3800 2950 60  0001 C CNN
 F 1 "PWR_FLAG" H 3800 3258 30  0000 C CNN
 F 2 "" H 3800 3050 60  0000 C CNN
@@
 	4900 6400 4900 7750
 $Comp
-L Resistors:RC0805JR-074K7L R?
+L Resistors:RC0805JR-074K7L R914
 U 1 1 5BDD919E
 P 3800 5800
-F 0 "R?" V 3755 5858 60  0000 L CNN
+F 0 "R914" V 3755 5858 60  0000 L CNN
 F 1 "RC0805JR-074K7L" H 3800 5500 50  0001 C CNN
 F 2 "Resistors:R0805" H 3800 4900 30  0001 C CNN
