File: Master_Board/V4/Fan Control.sch (KiCad schematic (older format))
At the start: 9 parts, among them Q1101 BSS806NH6327XTSA1, Q1102 BSS806NH6327XTSA1, Q1103 BSS806NH6327XTSA1

Commit message: add usb schematic
Connections:
- net labels added: GPIO1_EN, GPIO2_EN, GPIO3_EN
- net labels removed: GPO1_EN, GPO2_EN, GPO3_EN
Changed lines of the file:
@@
 $Descr USLetter 11000 8500
 encoding utf-8
-Sheet 10 9
+Sheet 8 10
 Title "BMS_MasterBoard_Fan_Control"
 Date "2018-09-20"
@@
 $EndComp
 Text HLabel 4150 3650 2    60   Input ~ 0
-GPO1_EN
+GPIO1_EN
 Text HLabel 5950 3650 2    60   Input ~ 0
-GPO2_EN
+GPIO2_EN
 Text HLabel 7800 3600 2    60   Input ~ 0
-GPO3_EN
+GPIO3_EN
 Wire Wire Line
 	6850 3150 6850 3300

Commit message: Update of schematic for master E10.1
Parts:
- added J?: 649002227222, Connectors:649002227222, symbol Connectors:649002227222
- added Q?: BSS806NH6327XTSA1, IC:SOT-23-3, symbol Transistors:BSS806NH6327XTSA1
- added R?: RC0805JR-0710KL, Resistors:R0805, symbol Resistors:RC0805JR-0710KL
Connections:
- net labels added: GPIO4_EN
- wire segments 27 -> 36

Commit message: Master V4 routed
Parts:
- gave numbers to parts that had none: 6
Changed lines of the file:
@@
 Connection ~ 6500 3650
 $Comp
-L Connectors:649002227222 J?
+L Connectors:649002227222 J801
 U 1 1 5BA66F80
 P 1900 4050
-F 0 "J?" H 1950 4350 60  0000 C CNN
+F 0 "J801" H 1950 4350 60  0000 C CNN
 F 1 "649002227222" H 1850 4250 60  0000 C CNN
 F 2 "Connectors:649002227222" H 1900 3150 60  0001 C CNN
@@
 $EndComp
 $Comp
-L Connectors:649002227222 J?
+L Connectors:649002227222 J802
 U 1 1 5BA675DC
 P 4200 4050
-F 0 "J?" H 4250 4350 60  0000 C CNN
+F 0 "J802" H 4250 4350 60  0000 C CNN
 F 1 "649002227222" H 4150 4250 60  0000 C CNN
 F 2 "Connectors:649002227222" H 4200 3150 60  0001 C CNN
@@
 $EndComp
 $Comp
-L Connectors:649002227222 J?
+L Connectors:649002227222 J803
 U 1 1 5BA677B8
 P 6450 4050
-F 0 "J?" H 6500 4350 60  0000 C CNN
+F 0 "J803" H 6500 4350 60  0000 C CNN
 F 1 "649002227222" H 6400 4250 60  0000 C CNN
 F 2 "Connectors:649002227222" H 6450 3150 60  0001 C CNN
@@
 $EndComp
 $Comp
-L Power_Port:DGND #PWR?
+L Power_Port:DGND #PWR0106
 U 1 1 5BA67A09
 P 6150 4550
-F 0 "#PWR?" H 6150 4380 50  0001 C CNN
+F 0 "#PWR0106" H 6150 4380 50  0001 C CNN
 F 1 "DGND" H 6150 4450 50  0000 C CNN
 F 2 "" H 6150 4650 60  0000 C CNN
@@
 $EndComp
 $Comp
-L Power_Port:DGND #PWR?
+L Power_Port:DGND #PWR0107
 U 1 1 5BA67A9F
 P 3900 4500
-F 0 "#PWR?" H 3900 4330 50  0001 C CNN
+F 0 "#PWR0107" H 3900 4330 50  0001 C CNN
 F 1 "DGND" H 3900 4400 50  0000 C CNN
 F 2 "" H 3900 4600 60  0000 C CNN
@@
 $EndComp
 $Comp
-L Power_Port:DGND #PWR?
+L Power_Port:DGND #PWR0108
 U 1 1 5BA67C3D
 P 1600 4500
-F 0 "#PWR?" H 1600 4330 50  0001 C CNN
+F 0 "#PWR0108" H 1600 4330 50  0001 C CNN
 F 1 "DGND" H 1600 4400 50  0000 C CNN
 F 2 "" H 1600 4600 60  0000 C CNN
@@
 	8450 4000 8450 4100
 $Comp
-L Power_Port:12V #PWR?
+L Power_Port:12V #PWR0109
 U 1 1 5BC724B1
 P 8450 3250
-F 0 "#PWR?" H 8450 3100 50  0001 C CNN
+F 0 "#PWR0109" H 8450 3100 50  0001 C CNN
 F 1 "12V" H 8440 3390 50  0000 C CNN
 F 2 "" H 8450 3250 60  0000 C CNN
@@
 $EndComp
 $Comp
-L Transistors:BSS806NH6327XTSA1 Q?
+L Transistors:BSS806NH6327XTSA1 Q803
 U 1 1 5BC724BC
 P 8550 3700
-F 0 "Q?" H 8800 3950 60  0000 C CNN
+F 0 "Q803" H 8800 3950 60  0000 C CNN
 F 1 "BSS806NH6327XTSA1" H 9150 3850 60  0000 C CNN
 F 2 "IC:SOT-23-3" H 8700 2800 60  0001 C CNN
@@
 	8750 3700 8800 3700
 $Comp
-L Resistors:RC0805JR-0710KL R?
+L Resistors:RC0805JR-0710KL R807
 U 1 1 5BC724CE
 P 8800 3400
-F 0 "R?" V 8755 3458 60  0000 L CNN
+F 0 "R807" V 8755 3458 60  0000 L CNN
 F 1 "RC0805JR-0710KL" H 8800 3100 50  0001 C CNN
 F 2 "Resistors:R0805" H 8800 2500 30  0001 C CNN
@@
 $EndComp
 $Comp
-L Power_Port:VDD #PWR?
+L Power_Port:VDD #PWR0110
 U 1 1 5BC724D5
 P 8800 3100
-F 0 "#PWR?" H 8800 2950 50  0001 C CNN
+F 0 "#PWR0110" H 8800 2950 50  0001 C CNN
 F 1 "VDD" H 8800 3274 50  0000 C CNN
 F 2 "" H 8800 3100 60  0000 C CNN
@@
 Connection ~ 8800 3700
 $Comp
-L Connectors:649002227222 J?
+L Connectors:649002227222 J804
 U 1 1 5BC724E4
 P 8750 4100
-F 0 "J?" H 8800 4400 60  0000 C CNN
+F 0 "J804" H 8800 4400 60  0000 C CNN
 F 1 "649002227222" H 8700 4300 60  0000 C CNN
 F 2 "Connectors:649002227222" H 8750 3200 60  0001 C CNN
@@
 $EndComp
 $Comp
-L Power_Port:DGND #PWR?
+L Power_Port:DGND #PWR0111
 U 1 1 5BC724EB
 P 8450 4600
-F 0 "#PWR?" H 8450 4430 50  0001 C CNN
+F 0 "#PWR0111" H 8450 4430 50  0001 C CNN
 F 1 "DGND" H 8450 4500 50  0000 C CNN
 F 2 "" H 8450 4700 60  0000 C CNN

Commit message: Reanotate all schematic and finish routing
Parts:
- renumbered Q1101 to Q801, Q1102 to Q802, Q1103 to Q803, Q803 to Q804, R1002 to R801, R1003 to R802, R1004 to R803, R807 to R804
Changed lines of the file:
@@
 	6150 3950 6150 4050
 $Comp
-L Power_Port:12V #PWR01005
+L Power_Port:12V #PWR0807
 U 1 1 5950A06A
 P 6150 3200
-F 0 "#PWR01005" H 6150 3050 50  0001 C CNN
+F 0 "#PWR0807" H 6150 3050 50  0001 C CNN
 F 1 "12V" H 6140 3340 50  0000 C CNN
 F 2 "" H 6150 3200 60  0000 C CNN
@@
 $EndComp
 $Comp
-L Power_Port:12V #PWR01003
+L Power_Port:12V #PWR0804
 U 1 1 59508B4F
 P 3900 3200
-F 0 "#PWR01003" H 3900 3050 50  0001 C CNN
+F 0 "#PWR0804" H 3900 3050 50  0001 C CNN
 F 1 "12V" H 3890 3340 50  0000 C CNN
 F 2 "" H 3900 3200 60  0000 C CNN
@@
 $EndComp
 $Comp
-L Power_Port:12V #PWR01001
+L Power_Port:12V #PWR0801
 U 1 1 594FA6E2
 P 1600 3200
-F 0 "#PWR01001" H 1600 3050 50  0001 C CNN
+F 0 "#PWR0801" H 1600 3050 50  0001 C CNN
 F 1 "12V" H 1590 3340 50  0000 C CNN
 F 2 "" H 1600 3200 60  0000 C CNN
@@
 $EndComp
 $Comp
-L Transistors:BSS806NH6327XTSA1 Q1103
+L Transistors:BSS806NH6327XTSA1 Q803
 U 1 1 5973F4DD
 P 6250 3650
-F 0 "Q1103" H 6500 3900 60  0000 C CNN
+F 0 "Q803" H 6500 3900 60  0000 C CNN
 F 1 "BSS806NH6327XTSA1" H 6850 3800 60  0000 C CNN
 F 2 "IC:SOT-23-3" H 6400 2750 60  0001 C CNN
@@
 $EndComp
 $Comp
-L Transistors:BSS806NH6327XTSA1 Q1102
+L Transistors:BSS806NH6327XTSA1 Q802
 U 1 1 5973DEC3
 P 4000 3650
-F 0 "Q1102" H 4250 3900 60  0000 C CNN
+F 0 "Q802" H 4250 3900 60  0000 C CNN
 F 1 "BSS806NH6327XTSA1" H 4600 3800 60  0000 C CNN
 F 2 "IC:SOT-23-3" H 4150 2750 60  0001 C CNN
@@
 $EndComp
 $Comp
-L Transistors:BSS806NH6327XTSA1 Q1101
+L Transistors:BSS806NH6327XTSA1 Q801
 U 1 1 596C1E1D
 P 1700 3650
-F 0 "Q1101" H 1950 3900 60  0000 C CNN
+F 0 "Q801" H 1950 3900 60  0000 C CNN
 F 1 "BSS806NH6327XTSA1" H 2300 3800 60  0000 C CNN
 F 2 "IC:SOT-23-3" H 1850 2750 60  0001 C CNN
@@
 Fan control circuit
 $Comp
-L Resistors:RC0805JR-0710KL R1002
+L Resistors:RC0805JR-0710KL R801
 U 1 1 5BA60FAF
 P 2000 3350
-F 0 "R1002" V 1955 3408 60  0000 L CNN
+F 0 "R801" V 1955 3408 60  0000 L CNN
 F 1 "RC0805JR-0710KL" H 2000 3050 50  0001 C CNN
 F 2 "Resistors:R0805" H 2000 2450 30  0001 C CNN
@@
 $EndComp
 $Comp
-L Resistors:RC0805JR-0710KL R1003
+L Resistors:RC0805JR-0710KL R802
 U 1 1 5BA61142
 P 4300 3350
-F 0 "R1003" V 4255 3408 60  0000 L CNN
+F 0 "R802" V 4255 3408 60  0000 L CNN
 F 1 "RC0805JR-0710KL" H 4300 3050 50  0001 C CNN
 F 2 "Resistors:R0805" H 4300 2450 30  0001 C CNN
@@
 $EndComp
 $Comp
-L Resistors:RC0805JR-0710KL R1004
+L Resistors:RC0805JR-0710KL R803
 U 1 1 5BA61235
 P 6500 3350
-F 0 "R1004" V 6455 3408 60  0000 L CNN
+F 0 "R803" V 6455 3408 60  0000 L CNN
 F 1 "RC0805JR-0710KL" H 6500 3050 50  0001 C CNN
 F 2 "Resistors:R0805" H 6500 2450 30  0001 C CNN
@@
 $EndComp
 $Comp
-L Power_Port:VDD #PWR01002
+L Power_Port:VDD #PWR0803
 U 1 1 5BA6138F
 P 2000 3050
-F 0 "#PWR01002" H 2000 2900 50  0001 C CNN
+F 0 "#PWR0803" H 2000 2900 50  0001 C CNN
 F 1 "VDD" H 2000 3224 50  0000 C CNN
 F 2 "" H 2000 3050 60  0000 C CNN
@@
 $EndComp
 $Comp
-L Power_Port:VDD #PWR01004
+L Power_Port:VDD #PWR0806
 U 1 1 5BA613CF
 P 4300 3050
-F 0 "#PWR01004" H 4300 2900 50  0001 C CNN
+F 0 "#PWR0806" H 4300 2900 50  0001 C CNN
 F 1 "VDD" H 4300 3224 50  0000 C CNN
 F 2 "" H 4300 3050 60  0000 C CNN
@@
 $EndComp
 $Comp
-L Power_Port:VDD #PWR01006
+L Power_Port:VDD #PWR0809
 U 1 1 5BA61403
 P 6500 3050
-F 0 "#PWR01006" H 6500 2900 50  0001 C CNN
+F 0 "#PWR0809" H 6500 2900 50  0001 C CNN
 F 1 "VDD" H 6500 3224 50  0000 C CNN
 F 2 "" H 6500 3050 60  0000 C CNN
@@
 $EndComp
 $Comp
-L Power_Port:DGND #PWR0106
+L Power_Port:DGND #PWR0808
 U 1 1 5BA67A09
 P 6150 4550
-F 0 "#PWR0106" H 6150 4380 50  0001 C CNN
+F 0 "#PWR0808" H 6150 4380 50  0001 C CNN
 F 1 "DGND" H 6150 4450 50  0000 C CNN
 F 2 "" H 6150 4650 60  0000 C CNN
@@
 $EndComp
 $Comp
-L Power_Port:DGND #PWR0107
+L Power_Port:DGND #PWR0805
 U 1 1 5BA67A9F
 P 3900 4500
-F 0 "#PWR0107" H 3900 4330 50  0001 C CNN
+F 0 "#PWR0805" H 3900 4330 50  0001 C CNN
 F 1 "DGND" H 3900 4400 50  0000 C CNN
 F 2 "" H 3900 4600 60  0000 C CNN
@@
 $EndComp
 $Comp
-L Power_Port:DGND #PWR0108
+L Power_Port:DGND #PWR0802
 U 1 1 5BA67C3D
 P 1600 4500
-F 0 "#PWR0108" H 1600 4330 50  0001 C CNN
+F 0 "#PWR0802" H 1600 4330 50  0001 C CNN
 F 1 "DGND" H 1600 4400 50  0000 C CNN
 F 2 "" H 1600 4600 60  0000 C CNN
@@
 	8450 4000 8450 4100
 $Comp
-L Power_Port:12V #PWR0109
+L Power_Port:12V #PWR0810
 U 1 1 5BC724B1
 P 8450 3250
-F 0 "#PWR0109" H 8450 3100 50  0001 C CNN
+F 0 "#PWR0810" H 8450 3100 50  0001 C CNN
 F 1 "12V" H 8440 3390 50  0000 C CNN
 F 2 "" H 8450 3250 60  0000 C CNN
@@
 $EndComp
 $Comp
-L Transistors:BSS806NH6327XTSA1 Q803
+L Transistors:BSS806NH6327XTSA1 Q804
 U 1 1 5BC724BC
 P 8550 3700
-F 0 "Q803" H 8800 3950 60  0000 C CNN
+F 0 "Q804" H 8800 3950 60  0000 C CNN
 F 1 "BSS806NH6327XTSA1" H 9150 3850 60  0000 C CNN
 F 2 "IC:SOT-23-3" H 8700 2800 60  0001 C CNN
@@
 	8750 3700 8800 3700
 $Comp
-L Resistors:RC0805JR-0710KL R807
+L Resistors:RC0805JR-0710KL R804
 U 1 1 5BC724CE
 P 8800 3400
-F 0 "R807" V 8755 3458 60  0000 L CNN
+F 0 "R804" V 8755 3458 60  0000 L CNN
 F 1 "RC0805JR-0710KL" H 8800 3100 50  0001 C CNN
 F 2 "Resistors:R0805" H 8800 2500 30  0001 C CNN
@@
 $EndComp
 $Comp
-L Power_Port:VDD #PWR0110
+L Power_Port:VDD #PWR0812
 U 1 1 5BC724D5
 P 8800 3100
-F 0 "#PWR0110" H 8800 2950 50  0001 C CNN
+F 0 "#PWR0812" H 8800 2950 50  0001 C CNN
 F 1 "VDD" H 8800 3274 50  0000 C CNN
 F 2 "" H 8800 3100 60  0000 C CNN
@@
 $EndComp
 $Comp
-L Power_Port:DGND #PWR0111
+L Power_Port:DGND #PWR0811
 U 1 1 5BC724EB
 P 8450 4600
-F 0 "#PWR0111" H 8450 4430 50  0001 C CNN
+F 0 "#PWR0811" H 8450 4430 50  0001 C CNN
 F 1 "DGND" H 8450 4500 50  0000 C CNN
 F 2 "" H 8450 4700 60  0000 C CNN
