File: Master_Board/V4/Power Supply.sch (KiCad schematic (older format))
At the start: 19 parts, among them J301 Header_Male_Pin_2.54mm_1X2_,_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, U301 OKI-78SR-5/1.5-W36-C, U302 AZ1117IH-3.3TRG1

Commit message: Repair broken librairy references
Parts:
- C301, C302: symbol 885012107018 -> Capacitors:885012107018
- C303: symbol 885012107014 -> Capacitors:885012107014
- C304: symbol 885012107005 -> Capacitors:885012107005
- D301, D302, D303: symbol 150080VS75000-RESCUE-Master_Board -> Diodes:150080VS75000
- F301: symbol 39511000440 -> Fuses:39511000440
- J301: symbol Header_Male_Pin_2.54mm_1X2_,_Unshrouded -> Connectors:Header_Male_Pin_2.54mm_1X2_,_Unshrouded
- R301: symbol RC0805JR-074K7L -> Resistors:RC0805JR-074K7L
- R302: symbol RC0805JR-071KL -> Resistors:RC0805JR-071KL
- R303: symbol RC0805JR-07470RL -> Resistors:RC0805JR-07470RL
- TP301, TP302, TP303, TP304, TP305: symbol Test_Point_THM -> Connectors:Test_Point_THM
- U301: symbol OKI-78SR-5/1.5-W36-C -> PMIC:OKI-78SR-5_1.5-W36-C
- U302: symbol AZ1117IH-3.3TRG1 -> PMIC:AZ1117IH-3.3TRG1
Changed lines of the file:
@@
 3.3V (LDO)
 $Comp
-L VDD #PWR0312
+L Power_Port:VDD #PWR0312
 U 1 1 58F7F090
 P 8000 3500
@@
 $EndComp
 $Comp
-L PWR_FLAG #FLG0305
+L Power_Port:PWR_FLAG #FLG0305
 U 1 1 58F88B2C
 P 6800 3500
@@
 $EndComp
 $Comp
-L PWR_FLAG #FLG0304
+L Power_Port:PWR_FLAG #FLG0304
 U 1 1 58F88B3E
 P 5100 3600
@@
 $EndComp
 $Comp
-L 5V #PWR0305
+L Power_Port:5V #PWR0305
 U 1 1 58F88B47
 P 4900 3600
@@
 $EndComp
 $Comp
-L OKI-78SR-5/1.5-W36-C U301
+L PMIC:OKI-78SR-5_1.5-W36-C U301
 U 1 1 58F88E7E
 P 4200 3700
@@
 $EndComp
 $Comp
-L DGND #PWR0304
+L Power_Port:DGND #PWR0304
 U 1 1 58F88F61
 P 4200 4400
@@
 Connection ~ 4900 3700
 $Comp
-L 885012107018 C301
+L Capacitors:885012107018 C301
 U 1 1 58F8900A
 P 3600 3900
@@
 $EndComp
 $Comp
-L 885012107018 C302
+L Capacitors:885012107018 C302
 U 1 1 58F89140
 P 4800 3900
@@
 Connection ~ 3600 3700
 $Comp
-L AZ1117IH-3.3TRG1 U302
+L PMIC:AZ1117IH-3.3TRG1 U302
 U 1 1 58F89C4D
 P 6200 3700
@@
 Connection ~ 5100 3700
 $Comp
-L 885012107014 C303
+L Capacitors:885012107014 C303
 U 1 1 58F8A222
 P 5700 3900
@@
 	5700 4100 5700 4200
 $Comp
-L DGND #PWR0307
+L Power_Port:DGND #PWR0307
 U 1 1 58F8A321
 P 5700 4300
@@
 $EndComp
 $Comp
-L DGND #PWR0308
+L Power_Port:DGND #PWR0308
 U 1 1 58F8A33F
 P 6200 4200
@@
 Connection ~ 6600 3600
 $Comp
-L 885012107005 C304
+L Capacitors:885012107005 C304
 U 1 1 58F8A3EF
 P 7000 3800
@@
 $EndComp
 $Comp
-L DGND #PWR0309
+L Power_Port:DGND #PWR0309
 U 1 1 58F8A4C9
 P 7000 4200
@@
 Connection ~ 7000 3600
 $Comp
-L PWR_FLAG #FLG0301
+L Power_Port:PWR_FLAG #FLG0301
 U 1 1 58F8B845
 P 1900 3600
@@
 Connection ~ 1900 3700
 $Comp
-L PWR_FLAG #FLG0303
+L Power_Port:PWR_FLAG #FLG0303
 U 1 1 58F8B88C
 P 3900 4300
@@
 Connection ~ 3900 4200
 $Comp
-L 150080VS75000-RESCUE-Master_Board D302
+L Diodes:150080VS75000 D302
 U 1 1 58F8E86A
 P 5000 4800
@@
 $EndComp
 $Comp
-L DGND #PWR0306
+L Power_Port:DGND #PWR0306
 U 1 1 58F8E9CC
 P 5000 5100
@@
 Connection ~ 5000 3700
 $Comp
-L RC0805JR-07470RL R303
+L Resistors:RC0805JR-07470RL R303
 U 1 1 58F8EBE0
 P 7500 4300
@@
 $EndComp
 $Comp
-L 150080VS75000-RESCUE-Master_Board D303
+L Diodes:150080VS75000 D303
 U 1 1 58F8EC30
 P 7500 4800
@@
 $EndComp
 $Comp
-L DGND #PWR0311
+L Power_Port:DGND #PWR0311
 U 1 1 58F8EC42
 P 7500 5100
@@
 Connection ~ 7500 3600
 $Comp
-L 150080VS75000-RESCUE-Master_Board D301
+L Diodes:150080VS75000 D301
 U 1 1 58F8E204
 P 3200 4800
@@
 $EndComp
 $Comp
-L DGND #PWR0303
+L Power_Port:DGND #PWR0303
 U 1 1 58F8E20A
 P 3200 5100
@@
 Connection ~ 3200 3700
 $Comp
-L Test_Point_THM TP301
+L Connectors:Test_Point_THM TP301
 U 1 1 58F8E348
 P 3400 3400
@@
 Connection ~ 3400 3700
 $Comp
-L Test_Point_THM TP303
+L Connectors:Test_Point_THM TP303
 U 1 1 58F8E842
 P 5400 3400
@@
 Connection ~ 5400 3700
 $Comp
-L Test_Point_THM TP304
+L Connectors:Test_Point_THM TP304
 U 1 1 58F8E9A6
 P 7300 3300
@@
 Connection ~ 7300 3600
 $Comp
-L Test_Point_THM TP302
+L Connectors:Test_Point_THM TP302
 U 1 1 58F8EB6B
 P 3600 4500
@@
 DGND
 $Comp
-L 39511000440 F301
+L Fuses:39511000440 F301
 U 1 1 58FAFE80
 P 2300 3700
@@
 	6500 3600 7700 3600
 $Comp
-L 12V #PWR0302
+L Power_Port:12V #PWR0302
 U 1 1 58FEC80D
 P 2600 3600
@@
 $EndComp
 $Comp
-L PWR_FLAG #FLG0302
+L Power_Port:PWR_FLAG #FLG0302
 U 1 1 58FEC813
 P 2900 3600
@@
 	1600 3600 1600 3700
 $Comp
-L CAN_PWR #PWR0301
+L Power_Port:CAN_PWR #PWR0301
 U 1 1 58FEC94F
 P 1600 3600
@@
 $EndComp
 $Comp
-L 3.3V #PWR0310
+L Power_Port:3.3V #PWR0310
 U 1 1 58FF65C4
 P 7100 3500
@@
 Connection ~ 7100 3600
 $Comp
-L Header_Male_Pin_2.54mm_1X2_,_Unshrouded J301
+L Connectors:Header_Male_Pin_2.54mm_1X2_,_Unshrouded J301
 U 1 1 58FF6649
 P 7700 3400
@@
 	8000 3600 8000 3500
 $Comp
-L Test_Point_THM TP305
+L Connectors:Test_Point_THM TP305
 U 1 1 58FF725D
 P 8300 3300
@@
 Connection ~ 8000 3600
 $Comp
-L PWR_FLAG #FLG0306
+L Power_Port:PWR_FLAG #FLG0306
 U 1 1 58FF7333
 P 8500 3500
@@
 Connection ~ 8300 3600
 $Comp
-L RC0805JR-071KL R302
+L Resistors:RC0805JR-071KL R302
 U 1 1 59347B67
 P 5000 4300
@@
 $EndComp
 $Comp
-L RC0805JR-074K7L R301
+L Resistors:RC0805JR-074K7L R301
 U 1 1 59347DB4
 P 3200 4300

Commit message: Add pull-up and connector to Master V4 circuit
Connections:
- wire segments 44 -> 68
Changed lines of the file:
@@
 $EndComp
 Wire Wire Line
-	4200 4000 4200 4300
-Wire Wire Line
-	4500 3700 5900 3700
+	4200 4000 4200 4100
+Wire Wire Line
+	4500 3700 4800 3700
 Wire Wire Line
 	4900 3700 4900 3600
@@
 $EndComp
 Wire Wire Line
-	3600 4100 3600 4300
-Wire Wire Line
-	3600 4200 4200 4200
+	3600 4100 3600 4200
+Wire Wire Line
+	3600 4200 3900 4200
 Connection ~ 4200 4200
 Wire Wire Line
@@
 $EndComp
 Wire Wire Line
-	2500 3700 3900 3700
-Wire Wire Line
-	1600 3700 2100 3700
-Wire Wire Line
-	6500 3600 7700 3600
+	2500 3700 2600 3700
+Wire Wire Line
+	1600 3700 1900 3700
+Wire Wire Line
+	6500 3600 6600 3600
 $Comp
 L Power_Port:12V #PWR0302
@@
 	7800 3500 7800 3600
 Wire Wire Line
-	7800 3600 8500 3600
+	7800 3600 8000 3600
 Wire Wire Line
 	8000 3600 8000 3500
@@
 	0    -1   -1   0
 $EndComp
+Wire Wire Line
+	4900 3700 5000 3700
+Wire Wire Line
+	4200 4200 4200 4300
+Wire Wire Line
+	4200 4100 4200 4200
+Wire Wire Line
+	4800 3700 4900 3700
+Wire Wire Line
+	3600 3700 3900 3700
+Wire Wire Line
+	5100 3700 5400 3700
+Wire Wire Line
+	5700 3700 5900 3700
+Wire Wire Line
+	6600 3600 6800 3600
+Wire Wire Line
+	6800 3600 7000 3600
+Wire Wire Line
+	7000 3600 7100 3600
+Wire Wire Line
+	1900 3700 2100 3700
+Wire Wire Line
+	3900 4200 4200 4200
+Wire Wire Line
+	5000 3700 5100 3700
+Wire Wire Line
+	7500 3600 7700 3600
+Wire Wire Line
+	3200 3700 3400 3700
+Wire Wire Line
+	3400 3700 3600 3700
+Wire Wire Line
+	5400 3700 5700 3700
+Wire Wire Line
+	7300 3600 7500 3600
+Wire Wire Line
+	3600 4200 3600 4300
+Wire Wire Line
+	2600 3700 2900 3700
+Wire Wire Line
+	2900 3700 3200 3700
+Wire Wire Line
+	7100 3600 7300 3600
+Wire Wire Line
+	8000 3600 8300 3600
+Wire Wire Line
+	8300 3600 8500 3600
 $EndSCHEMATC

Commit message: Remove big crappy connector and remap 12V
Connections:
- wire segments 68 -> 66
Changed lines of the file:
@@
 $Descr USLetter 11000 8500
 encoding utf-8
-Sheet 3 11
+Sheet 3 9
 Title "Power Supply"
 Date ""
@@
 Connection ~ 7000 3600
 $Comp
-L Power_Port:PWR_FLAG #FLG0301
-U 1 1 58F8B845
-P 1900 3600
-F 0 "#FLG0301" H 1900 3500 60  0001 C CNN
-F 1 "PWR_FLAG" H 1900 3800 30  0000 C CNN
-F 2 "" H 1900 3600 60  0000 C CNN
-F 3 "" H 1900 3600 60  0000 C CNN
-	1    1900 3600
-	1    0    0    -1
-$EndComp
-Wire Wire Line
-	1900 3600 1900 3700
-Connection ~ 1900 3700
-$Comp
 L Power_Port:PWR_FLAG #FLG0303
 U 1 1 58F8B88C
@@
 	2500 3700 2600 3700
 Wire Wire Line
-	1600 3700 1900 3700
-Wire Wire Line
 	6500 3600 6600 3600
 $Comp
@@
 	7000 3600 7100 3600
 Wire Wire Line
-	1900 3700 2100 3700
-Wire Wire Line
 	3900 4200 4200 4200
 Wire Wire Line
@@
 Wire Wire Line
 	8300 3600 8500 3600
+Wire Wire Line
+	1600 3700 2100 3700
 $EndSCHEMATC

Commit message: Update of schematic for master E10.1
Parts:
- removed U301: OKI-78SR-5/1.5-W36-C, Assembly:OKI-78SR_Vertical, symbol PMIC:OKI-78SR-5_1.5-W36-C
- added U?: OKI-78SR-5_1.5-W36H-C, Assembly:OKI-78SR_Horizontal, symbol PMIC:OKI-78SR-5_1.5-W36H-C
Changed lines of the file:
@@
-$EndComp
-$Comp
-L PMIC:OKI-78SR-5_1.5-W36-C U301
-U 1 1 58F88E7E
-P 4200 3700
-F 0 "U301" H 4200 3850 50  0000 C CNN
-F 1 "OKI-78SR-5/1.5-W36-C" H 4200 2900 60  0001 C CNN
-F 2 "Assembly:OKI-78SR_Vertical" H 4200 1575 60  0001 C CNN
-F 3 "http://power.murata.com/data/power/oki-78sr.pdf" H 4200 1475 60  0001 C CNN
-F 4 "Digikey" H 4200 2075 60  0001 C CNN "Supplier"
-F 5 "811-2196-5-ND" H 4200 1975 60  0001 C CNN "Supplier Part Number"
-F 6 "Murata Power Solutions Inc." H 4200 1875 60  0001 C CNN "Manufacturer"
-F 7 "OKI-78SR-5/1.5-W36H-C" H 4200 1775 60  0001 C CNN "Manufacturer Part Number"
-F 8 "DC/DC CONVERTER 5V 8W" H 4200 1675 60  0001 C CNN "Description"
-F 9 "7V" H 4190 2785 50  0001 C CNN "Voltage - Input (Min)"
-F 10 "36V" H 4190 2705 50  0001 C CNN "Voltage - Input (Max)"
-F 11 "5V" H 4190 2615 50  0001 C CNN "Voltage - Output (Min/Fixed)"
-F 12 "1.5A" H 4205 2400 50  0001 C CNN "Current - Output"
-	1    4200 3700
-	1    0    0    -1
 $EndComp
 $Comp
@@
 Wire Wire Line
 	1600 3700 2100 3700
+$Comp
+L PMIC:OKI-78SR-5_1.5-W36H-C U?
+U 1 1 5BD0EA6F
+P 4200 3700
+F 0 "U?" H 4200 3987 60  0000 C CNN
+F 1 "OKI-78SR-5_1.5-W36H-C" H 4200 3881 60  0000 C CNN
+F 2 "Assembly:OKI-78SR_Horizontal" H 4200 1575 60  0001 C CNN
+F 3 "http://power.murata.com/data/power/oki-78sr.pdf" H 4200 1475 60  0001 C CNN
+F 4 "Digikey" H 4200 2075 60  0001 C CNN "Supplier"
+F 5 "811-2692-ND" H 4200 1975 60  0001 C CNN "Supplier Part Number"
+F 6 "Murata Power Solutions Inc." H 4200 1875 60  0001 C CNN "Manufacturer"
+F 7 "OKI-78SR-5/1.5-W36H-C" H 4200 1775 60  0001 C CNN "Manufacturer Part Number"
+F 8 "DC/DC CONVERTER 5V 8W" H 4200 1675 60  0001 C CNN "Description"
+F 9 "7V" H 4190 2785 50  0001 C CNN "Voltage - Input (Min)"
+F 10 "36V" H 4190 2705 50  0001 C CNN "Voltage - Input (Max)"
+F 11 "5V" H 4190 2615 50  0001 C CNN "Voltage - Output (Min/Fixed)"
+F 12 "1.5A" H 4205 2400 50  0001 C CNN "Current - Output"
+	1    4200 3700
+	1    0    0    -1
+$EndComp
 $EndSCHEMATC

Commit message: Master V4 routed
Parts:
- removed D301, D302, D303: 150080VS75000, Diodes:LED_0805_GREEN, symbol Diodes:150080VS75000
- added D301, D302, D303: 150080BS75000, Diodes:LED_0805_BLUE, symbol Diodes:150080BS75000
- gave numbers to parts that had none: 1
Changed lines of the file:
@@
 Connection ~ 3900 4200
-$Comp
-L Diodes:150080VS75000 D302
-U 1 1 58F8E86A
-P 5000 4800
-F 0 "D302" V 4900 5000 60  0000 C CNN
-F 1 "150080VS75000" H 5000 4600 60  0001 C CNN
-F 2 "Diodes:LED_0805_GREEN" H 5010 3720 60  0001 C CNN
-F 3 "http://katalog.we-online.de/led/datasheet/150080VS75000.pdf" H 5010 3620 60  0001 C CNN
-F 4 "Digikey" H 5010 4220 60  0001 C CNN "Supplier"
-F 5 "732-4986-1-ND" H 5010 4120 60  0001 C CNN "Supplier Part Number"
-F 6 "Wurth Electronics Inc." H 5010 4020 60  0001 C CNN "Manufacturer"
-F 7 "150080VS75000" H 5010 3920 60  0001 C CNN "Manufacturer Part Number"
-F 8 "LED GREEN CLEAR 0805 SMD" H 5010 3820 60  0001 C CNN "Description"
-F 9 "GREEN" V 5000 5025 60  0000 C CNN "Color"
-F 10 "2V" H 5000 4400 60  0001 C CNN "Voltage - Forward (Vf) (Typ)"
-	1    5000 4800
-	0    -1   1    0
-$EndComp
 $Comp
 L Power_Port:DGND #PWR0306
@@
 $EndComp
 $Comp
-L Diodes:150080VS75000 D303
-U 1 1 58F8EC30
-P 7500 4800
-F 0 "D303" V 7400 5000 60  0000 C CNN
-F 1 "150080VS75000" H 7500 4600 60  0001 C CNN
-F 2 "Diodes:LED_0805_GREEN" H 7510 3720 60  0001 C CNN
-F 3 "http://katalog.we-online.de/led/datasheet/150080VS75000.pdf" H 7510 3620 60  0001 C CNN
-F 4 "Digikey" H 7510 4220 60  0001 C CNN "Supplier"
-F 5 "732-4986-1-ND" H 7510 4120 60  0001 C CNN "Supplier Part Number"
-F 6 "Wurth Electronics Inc." H 7510 4020 60  0001 C CNN "Manufacturer"
-F 7 "150080VS75000" H 7510 3920 60  0001 C CNN "Manufacturer Part Number"
-F 8 "LED GREEN CLEAR 0805 SMD" H 7510 3820 60  0001 C CNN "Description"
-F 9 "GREEN" V 7500 5025 60  0000 C CNN "Color"
-F 10 "2V" H 7500 4400 60  0001 C CNN "Voltage - Forward (Vf) (Typ)"
-	1    7500 4800
-	0    -1   1    0
-$EndComp
-$Comp
 L Power_Port:DGND #PWR0311
 U 1 1 58F8EC42
@@
 	7500 3600 7500 4100
 Connection ~ 7500 3600
-$Comp
-L Diodes:150080VS75000 D301
-U 1 1 58F8E204
-P 3200 4800
-F 0 "D301" V 3100 5000 60  0000 C CNN
-F 1 "150080VS75000" H 3200 4600 60  0001 C CNN
-F 2 "Diodes:LED_0805_GREEN" H 3210 3720 60  0001 C CNN
-F 3 "http://katalog.we-online.de/led/datasheet/150080VS75000.pdf" H 3210 3620 60  0001 C CNN
-F 4 "Digikey" H 3210 4220 60  0001 C CNN "Supplier"
-F 5 "732-4986-1-ND" H 3210 4120 60  0001 C CNN "Supplier Part Number"
-F 6 "Wurth Electronics Inc." H 3210 4020 60  0001 C CNN "Manufacturer"
-F 7 "150080VS75000" H 3210 3920 60  0001 C CNN "Manufacturer Part Number"
-F 8 "LED GREEN CLEAR 0805 SMD" H 3210 3820 60  0001 C CNN "Description"
-F 9 "GREEN" V 3200 5025 60  0000 C CNN "Color"
-F 10 "2V" H 3200 4400 60  0001 C CNN "Voltage - Forward (Vf) (Typ)"
-	1    3200 4800
-	0    -1   1    0
-$EndComp
 $Comp
 L Power_Port:DGND #PWR0303
@@
 	1600 3700 2100 3700
 $Comp
-L PMIC:OKI-78SR-5_1.5-W36H-C U?
+L PMIC:OKI-78SR-5_1.5-W36H-C U301
 U 1 1 5BD0EA6F
 P 4200 3700
-F 0 "U?" H 4200 3987 60  0000 C CNN
+F 0 "U301" H 4200 3987 60  0000 C CNN
 F 1 "OKI-78SR-5_1.5-W36H-C" H 4200 3881 60  0000 C CNN
 F 2 "Assembly:OKI-78SR_Horizontal" H 4200 1575 60  0001 C CNN
@@
 	1    0    0    -1
 $EndComp
+$Comp
+L Diodes:150080BS75000 D301
+U 1 1 5BDFDA3F
+P 3200 4800
+F 0 "D301" V 3097 4883 60  0000 L CNN
+F 1 "150080BS75000" V 3203 4883 60  0000 L CNN
+F 2 "Diodes:LED_0805_BLUE" H 3210 3720 60  0001 C CNN
+F 3 "http://katalog.we-online.de/led/datasheet/150080BS75000.pdf" H 3210 3620 60  0001 C CNN
+F 4 "Digikey" H 3210 4220 60  0001 C CNN "Supplier"
+F 5 "732-4982-1-ND" H 3210 4120 60  0001 C CNN "Supplier Part Number"
+F 6 "Wurth Electronics Inc." H 3210 4020 60  0001 C CNN "Manufacturer"
+F 7 "150080BS75000" H 3210 3920 60  0001 C CNN "Manufacturer Part Number"
+F 8 "LED BLUE CLEAR 0805 SMD" H 3210 3820 60  0001 C CNN "Description"
+F 9 "BLUE" H 3200 4500 60  0001 C CNN "Color"
+F 10 "3.2V" H 3200 4400 60  0001 C CNN "Voltage - Forward (Vf) (Typ)"
+	1    3200 4800
+	0    1    1    0
+$EndComp
+$Comp
+L Diodes:150080BS75000 D302
+U 1 1 5BDFDBAF
+P 5000 4800
+F 0 "D302" V 4897 4883 60  0000 L CNN
+F 1 "150080BS75000" V 5003 4883 60  0000 L CNN
+F 2 "Diodes:LED_0805_BLUE" H 5010 3720 60  0001 C CNN
+F 3 "http://katalog.we-online.de/led/datasheet/150080BS75000.pdf" H 5010 3620 60  0001 C CNN
+F 4 "Digikey" H 5010 4220 60  0001 C CNN "Supplier"
+F 5 "732-4982-1-ND" H 5010 4120 60  0001 C CNN "Supplier Part Number"
+F 6 "Wurth Electronics Inc." H 5010 4020 60  0001 C CNN "Manufacturer"
+F 7 "150080BS75000" H 5010 3920 60  0001 C CNN "Manufacturer Part Number"
+F 8 "LED BLUE CLEAR 0805 SMD" H 5010 3820 60  0001 C CNN "Description"
+F 9 "BLUE" H 5000 4500 60  0001 C CNN "Color"
+F 10 "3.2V" H 5000 4400 60  0001 C CNN "Voltage - Forward (Vf) (Typ)"
+	1    5000 4800
+	0    1    1    0
+$EndComp
+$Comp
+L Diodes:150080BS75000 D303
+U 1 1 5BDFDCEA
+P 7500 4800
+F 0 "D303" V 7397 4883 60  0000 L CNN
+F 1 "150080BS75000" V 7503 4883 60  0000 L CNN
+F 2 "Diodes:LED_0805_BLUE" H 7510 3720 60  0001 C CNN
+F 3 "http://katalog.we-online.de/led/datasheet/150080BS75000.pdf" H 7510 3620 60  0001 C CNN
+F 4 "Digikey" H 7510 4220 60  0001 C CNN "Supplier"
+F 5 "732-4982-1-ND" H 7510 4120 60  0001 C CNN "Supplier Part Number"
+F 6 "Wurth Electronics Inc." H 7510 4020 60  0001 C CNN "Manufacturer"
+F 7 "150080BS75000" H 7510 3920 60  0001 C CNN "Manufacturer Part Number"
+F 8 "LED BLUE CLEAR 0805 SMD" H 7510 3820 60  0001 C CNN "Description"
+F 9 "BLUE" H 7500 4500 60  0001 C CNN "Color"
+F 10 "3.2V" H 7500 4400 60  0001 C CNN "Voltage - Forward (Vf) (Typ)"
+	1    7500 4800
+	0    1    1    0
+$EndComp
 $EndSCHEMATC
