File: Master_Board/V4/STM32F446.sch (KiCad schematic (older format))
At the start: 45 parts, among them J201 Header_Male_Pin_2.54mm_1X3_,_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, J202 Header_Male_Pin_2.54mm_1X6_,_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, SW201 PTS645SM43SMTR92, SW202 PTS645SM43SMTR92, U201 STM32F446RE

Commit message: Repair broken librairy references
Parts:
- C201, C203, C205, C212: symbol 885012007053 -> Capacitors:885012007053
- C202, C210, C211, C214, C215, C216: symbol 885012207098 -> Capacitors:885012207098
- C204, C208: symbol 885012007027 -> Capacitors:885012007027
- C206, C209: symbol 885012107015 -> Capacitors:885012107015
- C207: symbol 885012207092 -> Capacitors:885012207092
- C213: symbol 885012107018 -> Capacitors:885012107018
- D201: symbol 150080VS75000 -> Diodes:150080VS75000
- D202: symbol 150080YS75000 -> Diodes:150080YS75000
- D203: symbol 150080RS75000 -> Diodes:150080RS75000
- J201: symbol Header_Male_Pin_2.54mm_1X3_,_Unshrouded -> Connectors:Header_Male_Pin_2.54mm_1X3_,_Unshrouded
- J202: symbol Header_Male_Pin_2.54mm_1X6_,_Unshrouded -> Connectors:Header_Male_Pin_2.54mm_1X6_,_Unshrouded
- R201, R204, R207, R212: symbol RC0805JR-074K7L -> Resistors:RC0805JR-074K7L
- R202, R206: symbol RC0805JR-070RL -> Resistors:RC0805JR-070RL
- R203, R211: symbol RC0805JR-07100RL -> Resistors:RC0805JR-07100RL
- R205, R208: symbol RC0805JR-071KL -> Resistors:RC0805JR-071KL
- R209, R210, R213: symbol RC0805JR-07470RL -> Resistors:RC0805JR-07470RL
- SW201, SW202: symbol PTS645SM43SMTR92 -> Switches:PTS645SM43SMTR92
- TP201, TP202, TP203, TP204, TP205, TP206: symbol Test_Point_THM -> Connectors:Test_Point_THM
- U201: symbol STM32F446RE -> STMicroelectronics:STM32F446RE
- XTAL201: symbol ABLS-8.000MHZ-D-T -> Crystals:ABLS-8.000MHZ-D-T
- XTAL202: symbol ABS25-32.768KHZ-6-T -> Crystals:ABS25-32.768KHZ-6-T

Commit message: Add pull-up and connector to Master V4 circuit
Connections:
- wire segments 168 -> 195
Changed lines of the file:
@@
 	6000 5200 6000 4800
 Wire Wire Line
-	2600 4500 2600 4700
-Wire Wire Line
-	2600 4600 3300 4600
+	2600 4500 2600 4600
+Wire Wire Line
+	2600 4600 3100 4600
 Wire Wire Line
 	3100 4600 3100 4500
@@
 	3100 4200 3100 4100
 Wire Wire Line
-	2600 4100 4300 4100
-Wire Wire Line
-	2600 4000 2600 4200
+	2600 4100 3100 4100
+Wire Wire Line
+	2600 4000 2600 4100
 Connection ~ 3100 4100
 Wire Wire Line
@@
 Connection ~ 3100 4600
 Wire Wire Line
-	6100 4800 6100 5700
-Wire Wire Line
-	6200 4800 6200 5200
+	6100 4800 6100 5500
+Wire Wire Line
+	6200 4800 6200 4900
 Wire Wire Line
 	6400 4900 6200 4900
@@
 Connection ~ 6100 5500
 Wire Wire Line
-	4200 5800 4400 5800
+	4200 5800 4300 5800
 Wire Wire Line
 	4300 5800 4300 5900
@@
 	4600 1800 4700 1800
 Wire Wire Line
-	4700 1700 4700 2500
-Wire Wire Line
-	4200 1800 4200 2100
+	4700 1700 4700 1800
+Wire Wire Line
+	4200 1800 4200 2000
 Wire Wire Line
 	4200 1800 4300 1800
@@
 	6900 2800 6800 2800
 Wire Wire Line
-	6800 2700 6800 2900
+	6800 2700 6800 2800
 Wire Wire Line
 	6800 2900 6600 2900
 Wire Wire Line
-	7200 2800 7600 2800
+	7200 2800 7400 2800
 Wire Wire Line
 	7400 3000 7400 2800
@@
 	1000 4300 1000 4400
 Wire Wire Line
-	1000 4800 1000 5000
+	1000 4800 1000 4900
 Connection ~ 1000 4900
 Wire Wire Line
 	1100 4900 1000 4900
 Wire Wire Line
-	1000 5400 1000 5600
+	1000 5400 1000 5500
 Wire Wire Line
 	1600 5500 1000 5500
@@
 	4300 3500 4000 3500
 Wire Wire Line
-	1500 4900 1700 4900
+	1500 4900 1600 4900
 Wire Notes Line
 	500  4000 500  5900
@@
 	2000 4000 500  4000
 Wire Wire Line
-	4000 2900 4300 2900
+	4000 2900 4200 2900
 Wire Wire Line
 	3700 3000 4300 3000
@@
 	5500 2500 5500 2400
 Wire Wire Line
-	5400 1550 5400 2500
+	5400 1550 5400 1600
 Wire Wire Line
 	5300 2500 5300 2400
@@
 	2600 3200 4300 3200
 Wire Wire Line
-	2500 1700 2700 1700
+	2500 1700 2600 1700
 Wire Wire Line
 	2600 1900 2600 1700
 Connection ~ 2600 1700
 Wire Wire Line
-	3100 1700 3300 1700
+	3100 1700 3200 1700
 Wire Wire Line
 	2200 1700 2100 1700
@@
 	2600 2300 2600 3200
 Wire Wire Line
-	1100 2800 1300 2800
-Wire Wire Line
-	1700 2800 1900 2800
+	1100 2800 1200 2800
+Wire Wire Line
+	1700 2800 1800 2800
 Wire Wire Line
 	700  2900 700  2800
@@
 	3900 1400 1900 1400
 Wire Wire Line
-	2300 6600 2500 6600
+	2300 6600 2400 6600
 Wire Wire Line
 	2300 7500 2500 7500
@@
 	1200 7500 1900 7500
 Wire Wire Line
-	4400 5100 4400 5400
+	4400 5100 4400 5300
 Wire Wire Line
 	4400 5100 4900 5100
@@
 	9900 4800 9900 4900
 Wire Wire Line
-	9900 5300 9900 5500
+	9900 5300 9900 5400
 Connection ~ 9900 5400
 Wire Wire Line
 	9800 5400 9900 5400
 Wire Wire Line
-	9900 5900 9900 6100
+	9900 5900 9900 6000
 Wire Wire Line
 	9300 6000 9900 6000
@@
 Connection ~ 9300 5400
 Wire Wire Line
-	9200 5400 9400 5400
+	9200 5400 9300 5400
 Wire Notes Line
 	8700 4500 8700 6400
@@
 	4250 4400 4250 4550
 Wire Wire Line
-	5050 6600 5250 6600
+	5050 6600 5150 6600
 Wire Wire Line
 	5050 7500 5250 7500
@@
 Text Label 9950 2550 3    60   ~ 0
 LED_ASSERT
+Wire Wire Line
+	3100 4100 4300 4100
+Wire Wire Line
+	3100 4600 3300 4600
+Wire Wire Line
+	6200 4900 6200 5200
+Wire Wire Line
+	6100 5600 6100 5700
+Wire Wire Line
+	6100 5500 6100 5600
+Wire Wire Line
+	4300 5800 4400 5800
+Wire Wire Line
+	4400 5300 4400 5400
+Wire Wire Line
+	2600 4100 2600 4200
+Wire Wire Line
+	4200 2000 4200 2100
+Wire Wire Line
+	4700 1800 4700 2500
+Wire Wire Line
+	6800 2800 6800 2900
+Wire Wire Line
+	2600 4600 2600 4700
+Wire Wire Line
+	1000 4900 1000 5000
+Wire Wire Line
+	1000 5500 1000 5600
+Wire Wire Line
+	1600 4900 1700 4900
+Wire Wire Line
+	2600 1700 2700 1700
+Wire Wire Line
+	3200 1700 3300 1700
+Wire Wire Line
+	1200 2800 1300 2800
+Wire Wire Line
+	1800 2800 1900 2800
+Wire Wire Line
+	7400 2800 7600 2800
+Wire Wire Line
+	9900 5400 9900 5500
+Wire Wire Line
+	9900 6000 9900 6100
+Wire Wire Line
+	9300 5400 9400 5400
+Wire Wire Line
+	4200 2900 4300 2900
+Wire Wire Line
+	2400 6600 2500 6600
+Wire Wire Line
+	5150 6600 5250 6600
+Wire Wire Line
+	5400 1600 5400 2500
 $EndSCHEMATC

Commit message: Remove big crappy connector and remap 12V
Connections:
- net labels added: LED_ERROR
- net labels removed: LED_ASSERT
Changed lines of the file:
@@
 $Descr USLetter 11000 8500
 encoding utf-8
-Sheet 2 11
+Sheet 2 9
 Title "STM32F446RE"
 Date ""
@@
 $EndComp
 Text Label 7050 4200 0    60   ~ 0
-LED_ASSERT
+LED_ERROR
 $Comp
 L Resistors:RC0805JR-07470RL R213
@@
 $EndComp
 Text Label 9950 2550 3    60   ~ 0
-LED_ASSERT
+LED_ERROR
 Wire Wire Line
 	3100 4100 4300 4100

Commit message: Update of schematic for master E10.1
Parts:
- added R?: RC0805JR-0710KL, Resistors:R0805, symbol Resistors:RC0805JR-0710KL
Connections:
- wire segments 195 -> 199
Changed lines of the file:
@@
 Text HLabel 4000 2900 0    60   BiDi ~ 0
 VBat
-Text HLabel 4200 3600 0    60   Output ~ 0
+Text HLabel 3700 3600 0    60   Output ~ 0
 PC0
 Text Label 4000 3500 0    60   ~ 0
@@
 Text Notes 1000 3900 0    100  ~ 0
 RESET
-Text HLabel 4200 3700 0    60   Output ~ 0
+Text HLabel 3700 3700 0    60   Output ~ 0
 PC1
-Text HLabel 4200 3800 0    60   Output ~ 0
+Text HLabel 3700 3800 0    60   Output ~ 0
 PC2
 Text HLabel 4200 3900 0    60   BiDi ~ 0
@@
 Text HLabel 5900 4900 3    60   Output ~ 0
 PB10
-Text HLabel 7600 4200 2    60   Output ~ 0
+Text HLabel 6750 4200 2    60   BiDi ~ 0
 PB14
-Text HLabel 7600 4100 2    60   Output ~ 0
+Text HLabel 6750 4100 2    60   BiDi ~ 0
 PB15
-Text HLabel 7600 4000 2    60   Output ~ 0
+Text HLabel 6750 4000 2    60   BiDi ~ 0
 PC6
 Text HLabel 6750 3900 2    60   BiDi ~ 0
@@
 Text HLabel 5200 2400 1    60   BiDi ~ 0
 PB7
-Text HLabel 5100 2400 1    60   BiDi ~ 0
+Text HLabel 5100 1300 1    60   BiDi ~ 0
 BOOT0
 Text HLabel 5000 2400 1    60   Output ~ 0
@@
 	0    -1   -1   0
 $EndComp
-Text Label 7050 4000 0    60   ~ 0
-LED_BLINK
 Text Label 8550 2550 3    60   ~ 0
 LED_BLINK
@@
 	1    0    0    -1
 $EndComp
-Text Label 7050 4200 0    60   ~ 0
-LED_ERROR
 $Comp
 L Resistors:RC0805JR-07470RL R213
@@
 	1    0    0    -1
 $EndComp
-Text Label 7050 4100 0    60   ~ 0
-LED_DEBUG
 Text Notes 8200 2450 0    60   ~ 0
 LED : BLINK, DEBUG, ASSERT
@@
 Text HLabel 5600 4900 3    60   BiDi ~ 0
 PB0
-Text HLabel 4000 3500 0    60   Input ~ 0
+Text HLabel 3700 3500 0    60   Input ~ 0
 NRST
 $Comp
@@
 Connection ~ 1600 4900
 Wire Wire Line
-	4300 3500 4000 3500
+	4300 3500 3700 3500
 Wire Wire Line
 	1500 4900 1600 4900
@@
 	3700 3000 4300 3000
 Wire Wire Line
-	4300 3600 4200 3600
-Wire Wire Line
-	4200 3700 4300 3700
-Wire Wire Line
 	4300 3900 4200 3900
 Wire Wire Line
-	4200 3800 4300 3800
-Wire Wire Line
 	4200 4200 4300 4200
 Wire Wire Line
@@
 	6600 4300 7600 4300
 Wire Wire Line
-	6600 4200 7600 4200
-Wire Wire Line
-	6600 4100 7600 4100
-Wire Wire Line
-	6600 4000 7600 4000
+	6600 4200 6750 4200
+Wire Wire Line
+	6600 4100 6750 4100
+Wire Wire Line
+	6600 4000 6750 4000
 Wire Wire Line
 	6600 3900 6750 3900
@@
 Wire Wire Line
 	5200 2400 5200 2500
-Wire Wire Line
-	5100 2500 5100 2400
 Wire Wire Line
 	5000 2400 5000 2500
@@
 Wire Wire Line
 	5400 1600 5400 2500
+Wire Wire Line
+	5100 1400 4850 1400
+$Comp
+L Power_Port:DGND #PWR?
+U 1 1 5BD344F6
+P 4200 1550
+F 0 "#PWR?" H 4200 1380 50  0001 C CNN
+F 1 "DGND" H 4200 1450 50  0000 C CNN
+F 2 "" H 4200 1650 60  0000 C CNN
+F 3 "" H 4180 1460 60  0000 C CNN
+	1    4200 1550
+	1    0    0    -1
+$EndComp
+Wire Wire Line
+	5100 1400 5100 2500
+$Comp
+L Resistors:RC0805JR-0710KL R?
+U 1 1 5BD5F8F8
+P 4650 1400
+F 0 "R?" H 4650 1601 60  0000 C CNN
+F 1 "RC0805JR-0710KL" H 4650 1100 50  0001 C CNN
+F 2 "Resistors:R0805" H 4650 500 30  0001 C CNN
+F 3 "http://www.yageo.com/documents/recent/PYu-RC_Group_51_RoHS_L_7.pdf" H 4650 450 30  0001 C CNN
+F 4 "Digikey" H 4650 1000 60  0001 C CNN "Supplier"
+F 5 "311-10KARCT-ND" H 4650 900 60  0001 C CNN "Supplier Part Number"
+F 6 "Yageo" H 4650 800 60  0001 C CNN "Manufacturer"
+F 7 "RC0805JR-0710KL" H 4650 700 60  0001 C CNN "Manufacturer Part Number"
+F 8 "RES SMD 10K OHM 5% 1/8W 0805" H 4650 600 60  0001 C CNN "Description"
+F 9 "10k" H 4650 1503 50  0000 C CNN "Resistance (Ohms)"
+F 10 "±5%" H 5060 1320 50  0001 C CNN "Tolerance (%)"
+F 11 "1/8W" H 4650 1260 50  0001 C CNN "Puissance (Watts)"
+	1    4650 1400
+	1    0    0    -1
+$EndComp
+Wire Wire Line
+	4450 1400 4200 1400
+Wire Wire Line
+	4200 1400 4200 1450
+Wire Wire Line
+	5100 1400 5100 1300
+Connection ~ 5100 1400
+Text Label 3700 3800 0    60   ~ 0
+LED_BLINK
+Text Label 3700 3700 0    60   ~ 0
+LED_DEBUG
+Text Label 3700 3600 0    60   ~ 0
+LED_ERROR
+Wire Wire Line
+	3700 3600 4300 3600
+Wire Wire Line
+	3700 3700 4300 3700
+Wire Wire Line
+	3700 3800 4300 3800
 $EndSCHEMATC

Commit message: Master V4 routed
Parts:
- removed XTAL201: ABLS-8.000MHZ-D-T, Crystals:HC49_US, symbol Crystals:ABLS-8.000MHZ-D-T
- added XTAL201: 7A-8.000MAHJ-T, Crystals:TXC_7A_Series, symbol Crystals:7A-8.000MAHJ-T
- gave numbers to parts that had none: 1
Changed lines of the file:
@@
-$EndComp
-$Comp
-L Crystals:ABLS-8.000MHZ-D-T XTAL201
-U 1 1 58F3DBC0
-P 1500 2800
-F 0 "XTAL201" H 1500 3000 60  0000 C CNN
-F 1 "ABLS-8.000MHZ-D-T" H 1500 2600 30  0000 C CNN
-F 2 "Crystals:HC49_US" H 1500 1900 60  0001 C CNN
-F 3 "http://www.abracon.com/Resonators/abls.pdf" H 1500 1800 60  0001 C CNN
-F 4 "Digikey" H 1500 2400 60  0001 C CNN "Supplier"
-F 5 "535-13445-2-ND" H 1500 2300 60  0001 C CNN "Supplier Part Number"
-F 6 "Abracon LLC" H 1500 2200 60  0001 C CNN "Manufacturer"
-F 7 "ABLS-8.000MHZ-D-T" H 1500 2100 60  0001 C CNN "Manufacturer Part Number"
-F 8 "CRYSTAL 8.0000MHZ 18PF SMD" H 1500 2000 60  0001 C CNN "Description"
-	1    1500 2800
-	1    0    0    -1
 $EndComp
 $Comp
@@
 	5150 7000 5150 7100
 Wire Wire Line
-	3950 6600 4650 6600
-Wire Wire Line
 	3950 7500 4650 7500
 Wire Notes Line
@@
 	-1   0    0    1
 $EndComp
-Wire Wire Line
-	7600 3600 7550 3600
-Wire Wire Line
-	7550 3600 7550 3650
 $Comp
 L Power_Port:DGND #PWR0221
@@
 	5100 1400 4850 1400
 $Comp
-L Power_Port:DGND #PWR?
+L Power_Port:DGND #PWR0104
 U 1 1 5BD344F6
 P 4200 1550
-F 0 "#PWR?" H 4200 1380 50  0001 C CNN
+F 0 "#PWR0104" H 4200 1380 50  0001 C CNN
 F 1 "DGND" H 4200 1450 50  0000 C CNN
 F 2 "" H 4200 1650 60  0000 C CNN
@@
 	5100 1400 5100 2500
 $Comp
-L Resistors:RC0805JR-0710KL R?
+L Resistors:RC0805JR-0710KL R214
 U 1 1 5BD5F8F8
 P 4650 1400
-F 0 "R?" H 4650 1601 60  0000 C CNN
+F 0 "R214" H 4650 1601 60  0000 C CNN
 F 1 "RC0805JR-0710KL" H 4650 1100 50  0001 C CNN
 F 2 "Resistors:R0805" H 4650 500 30  0001 C CNN
@@
 Wire Wire Line
 	3700 3800 4300 3800
+$Comp
+L Crystals:7A-8.000MAHJ-T XTAL201
+U 1 1 5BD212B3
+P 1500 2800
+F 0 "XTAL201" H 1500 3000 60  0000 C CNN
+F 1 "7A-8.000MAHJ-T" H 1500 2650 39  0000 C CNN
+F 2 "Crystals:TXC_7A_Series" H 1500 2000 60  0001 C CNN
+F 3 "http://www.txccorp.com/download/products/quartz_crystals/2015TXC_7A_28.pdf" H 1500 2000 60  0001 C CNN
+F 4 "Digikey" H 1500 2500 60  0001 C CNN "Supplier"
+F 5 "887-2634-1-ND" H 1500 2400 60  0001 C CNN "Supplier Part Number"
+F 6 "TXC CORPORATION" H 1500 2300 60  0001 C CNN "Manufacturer"
+F 7 "ABLS-8.000MHZ-D-T" H 1500 2200 60  0001 C CNN "Manufacturer Part Number"
+F 8 "CRYSTAL 8.000MHZ 18PF SMT" H 1500 2100 60  0001 C CNN "Description"
+	1    1500 2800
+	1    0    0    -1
+$EndComp
+Wire Wire Line
+	3950 6600 4650 6600
+Wire Wire Line
+	7600 3600 7550 3600
+Wire Wire Line
+	7550 3600 7550 3650
 $EndSCHEMATC

Commit message: Reanotate all schematic and finish routing
Parts:
- renumbered R214 to R207, R207 to R208, R208 to R209, R209 to R210, R210 to R211, R211 to R212, R212 to R213, R213 to R214
Changed lines of the file:
@@
 $EndComp
 $Comp
-L Power_Port:VDD #PWR0219
+L Power_Port:VDD #PWR0220
 U 1 1 58F2D98D
 P 6400 4900
-F 0 "#PWR0219" H 6400 4750 50  0001 C CNN
+F 0 "#PWR0220" H 6400 4750 50  0001 C CNN
 F 1 "VDD" H 6390 5040 50  0000 C CNN
 F 2 "" H 6400 4900 60  0000 C CNN
@@
 $EndComp
 $Comp
-L Power_Port:DGND #PWR0218
+L Power_Port:DGND #PWR0219
 U 1 1 58F2DBB5
 P 6100 5800
-F 0 "#PWR0218" H 6100 5630 50  0001 C CNN
+F 0 "#PWR0219" H 6100 5630 50  0001 C CNN
 F 1 "DGND" H 6100 5700 50  0000 C CNN
 F 2 "" H 6100 5900 60  0000 C CNN
@@
 $EndComp
 $Comp
-L Power_Port:DGND #PWR0214
+L Power_Port:DGND #PWR0215
 U 1 1 58F2E125
 P 4300 6000
-F 0 "#PWR0214" H 4300 5830 50  0001 C CNN
+F 0 "#PWR0215" H 4300 5830 50  0001 C CNN
 F 1 "DGND" H 4300 5900 50  0000 C CNN
 F 2 "" H 4300 6100 60  0000 C CNN
@@
 $EndComp
 $Comp
-L Power_Port:VDD #PWR0215
+L Power_Port:VDD #PWR0216
 U 1 1 58F2E176
 P 4600 5300
-F 0 "#PWR0215" H 4600 5150 50  0001 C CNN
+F 0 "#PWR0216" H 4600 5150 50  0001 C CNN
 F 1 "VDD" H 4590 5440 50  0000 C CNN
 F 2 "" H 4600 5300 60  0000 C CNN
@@
 $EndComp
 $Comp
-L Power_Port:DGND #PWR0213
+L Power_Port:DGND #PWR0214
 U 1 1 58F2E533
 P 4200 2200
-F 0 "#PWR0213" H 4200 2030 50  0001 C CNN
+F 0 "#PWR0214" H 4200 2030 50  0001 C CNN
 F 1 "DGND" H 4200 2100 50  0000 C CNN
 F 2 "" H 4200 2300 60  0000 C CNN
@@
 $EndComp
 $Comp
-L Power_Port:DGND #PWR0222
+L Power_Port:DGND #PWR0223
 U 1 1 58F2E754
 P 7600 2900
-F 0 "#PWR0222" H 7600 2730 50  0001 C CNN
+F 0 "#PWR0223" H 7600 2730 50  0001 C CNN
 F 1 "DGND" H 7600 2800 50  0000 C CNN
 F 2 "" H 7600 3000 60  0000 C CNN
@@
 $EndComp
 $Comp
-L Power_Port:VDD #PWR0216
+L Power_Port:VDD #PWR0217
 U 1 1 58F2E95B
 P 4700 1700
-F 0 "#PWR0216" H 4700 1550 50  0001 C CNN
+F 0 "#PWR0217" H 4700 1550 50  0001 C CNN
 F 1 "VDD" H 4690 1840 50  0000 C CNN
 F 2 "" H 4700 1700 60  0000 C CNN
@@
 $EndComp
 $Comp
-L Power_Port:VDD #PWR0220
+L Power_Port:VDD #PWR0221
 U 1 1 58F2EA08
 P 6800 2700
-F 0 "#PWR0220" H 6800 2550 50  0001 C CNN
+F 0 "#PWR0221" H 6800 2550 50  0001 C CNN
 F 1 "VDD" H 6790 2840 50  0000 C CNN
 F 2 "" H 6800 2700 60  0000 C CNN
@@
 $EndComp
 $Comp
-L Resistors:RC0805JR-07470RL R209
+L Resistors:RC0805JR-07470RL R210
 U 1 1 58F8F74B
 P 8550 3600
-F 0 "R209" V 8650 3800 60  0000 C CNN
+F 0 "R210" V 8650 3800 60  0000 C CNN
 F 1 "RC0805JR-07470RL" H 8550 3300 50  0001 C CNN
 F 2 "Resistors:R0805" H 8550 2700 30  0001 C CNN
@@
 LED_BLINK
 $Comp
-L Power_Port:DGND #PWR0223
+L Power_Port:DGND #PWR0224
 U 1 1 58F90369
 P 8550 3950
-F 0 "#PWR0223" H 8550 3780 50  0001 C CNN
+F 0 "#PWR0224" H 8550 3780 50  0001 C CNN
 F 1 "DGND" H 8550 3850 50  0000 C CNN
 F 2 "" H 8550 4050 60  0000 C CNN
@@
 $EndComp
 $Comp
-L Resistors:RC0805JR-07470RL R210
+L Resistors:RC0805JR-07470RL R211
 U 1 1 58F904BD
 P 9250 3600
-F 0 "R210" V 9350 3800 60  0000 C CNN
+F 0 "R211" V 9350 3800 60  0000 C CNN
 F 1 "RC0805JR-07470RL" H 9250 3300 50  0001 C CNN
 F 2 "Resistors:R0805" H 9250 2700 30  0001 C CNN
@@
 LED_DEBUG
 $Comp
-L Power_Port:DGND #PWR0224
+L Power_Port:DGND #PWR0225
 U 1 1 58F904C6
 P 9250 3950
-F 0 "#PWR0224" H 9250 3780 50  0001 C CNN
+F 0 "#PWR0225" H 9250 3780 50  0001 C CNN
 F 1 "DGND" H 9250 3850 50  0000 C CNN
 F 2 "" H 9250 4050 60  0000 C CNN
@@
 $EndComp
 $Comp
-L Resistors:RC0805JR-07470RL R213
+L Resistors:RC0805JR-07470RL R214
 U 1 1 58F90B78
 P 9950 3600
-F 0 "R213" V 10050 3800 60  0000 C CNN
+F 0 "R214" V 10050 3800 60  0000 C CNN
 F 1 "RC0805JR-07470RL" H 9950 3300 50  0001 C CNN
 F 2 "Resistors:R0805" H 9950 2700 30  0001 C CNN
@@
 $EndComp
 $Comp
-L Power_Port:DGND #PWR0229
+L Power_Port:DGND #PWR0230
 U 1 1 58F90B81
 P 9950 3950
-F 0 "#PWR0229" H 9950 3780 50  0001 C CNN
+F 0 "#PWR0230" H 9950 3780 50  0001 C CNN
 F 1 "DGND" H 9950 3850 50  0000 C CNN
 F 2 "" H 9950 4050 60  0000 C CNN
@@
 $EndComp
 $Comp
-L Power_Port:DGND #PWR0228
+L Power_Port:DGND #PWR0229
 U 1 1 58FAAF19
 P 9900 6200
-F 0 "#PWR0228" H 9900 6030 50  0001 C CNN
+F 0 "#PWR0229" H 9900 6030 50  0001 C CNN
 F 1 "DGND" H 9900 6100 50  0000 C CNN
 F 2 "" H 9900 6300 60  0000 C CNN
@@
 $EndComp
 $Comp
-L Power_Port:VDD #PWR0227
+L Power_Port:VDD #PWR0228
 U 1 1 58FAAF1F
 P 9900 4800
-F 0 "#PWR0227" H 9900 4650 50  0001 C CNN
+F 0 "#PWR0228" H 9900 4650 50  0001 C CNN
 F 1 "VDD" H 9890 4940 50  0000 C CNN
 F 2 "" H 9900 4800 60  0000 C CNN
@@
 USER BUTTON
 $Comp
-L Resistors:RC0805JR-074K7L R212
+L Resistors:RC0805JR-074K7L R213
 U 1 1 58FAAF2F
 P 9900 5100
-F 0 "R212" V 9975 5275 60  0000 C CNN
+F 0 "R213" V 9975 5275 60  0000 C CNN
 F 1 "RC0805JR-074K7L" H 9900 4800 50  0001 C CNN
 F 2 "Resistors:R0805" H 9900 4200 30  0001 C CNN
@@
 $EndComp
 $Comp
-L Resistors:RC0805JR-07100RL R211
+L Resistors:RC0805JR-07100RL R212
 U 1 1 58FAAF3D
 P 9600 5400
-F 0 "R211" H 9600 5500 60  0000 C CNN
+F 0 "R212" H 9600 5500 60  0000 C CNN
 F 1 "RC0805JR-07100RL" H 9600 5100 50  0001 C CNN
 F 2 "Resistors:R0805" H 9600 4500 30  0001 C CNN
@@
 $EndComp
 $Comp
-L Power_Port:VDD #PWR0226
+L Power_Port:VDD #PWR0227
 U 1 1 58FBA992
 P 9900 1000
-F 0 "#PWR0226" H 9900 850 50  0001 C CNN
+F 0 "#PWR0227" H 9900 850 50  0001 C CNN
 F 1 "VDD" H 9890 1140 50  0000 C CNN
 F 2 "" H 9900 1000 60  0000 C CNN
@@
 SWO
 $Comp
-L Power_Port:DGND #PWR0225
+L Power_Port:DGND #PWR0226
 U 1 1 58FBB473
 P 9500 1500
-F 0 "#PWR0225" H 9500 1330 50  0001 C CNN
+F 0 "#PWR0226" H 9500 1330 50  0001 C CNN
 F 1 "DGND" H 9500 1400 50  0000 C CNN
 F 2 "" H 9500 1600 60  0000 C CNN
@@
 USART1_TX
 $Comp
-L Resistors:RC0805JR-074K7L R207
+L Resistors:RC0805JR-074K7L R208
 U 1 1 59843533
 P 4850 6600
-F 0 "R207" H 4850 6700 60  0000 C CNN
+F 0 "R208" H 4850 6700 60  0000 C CNN
 F 1 "RC0805JR-074K7L" H 4850 6300 50  0001 C CNN
 F 2 "Resistors:R0805" H 4850 5700 30  0001 C CNN
@@
 USART1_RX
 $Comp
-L Power_Port:DGND #PWR0217
+L Power_Port:DGND #PWR0218
 U 1 1 5984353A
 P 5150 7200
-F 0 "#PWR0217" H 5150 7030 50  0001 C CNN
+F 0 "#PWR0218" H 5150 7030 50  0001 C CNN
 F 1 "DGND" H 5150 7100 50  0000 C CNN
 F 2 "" H 5150 7300 60  0000 C CNN
@@
 PA10_RX
 $Comp
-L Resistors:RC0805JR-071KL R208
+L Resistors:RC0805JR-071KL R209
 U 1 1 5984354A
 P 4850 7500
-F 0 "R208" H 4850 7600 60  0000 C CNN
+F 0 "R209" H 4850 7600 60  0000 C CNN
 F 1 "RC0805JR-071KL" H 4850 7200 50  0001 C CNN
 F 2 "Resistors:R0805" H 4850 6600 30  0001 C CNN
@@
 $EndComp
 $Comp
-L Power_Port:DGND #PWR0221
+L Power_Port:DGND #PWR0222
 U 1 1 59A40ED8
 P 7550 3750
-F 0 "#PWR0221" H 7550 3580 50  0001 C CNN
+F 0 "#PWR0222" H 7550 3580 50  0001 C CNN
 F 1 "DGND" H 7550 3650 50  0000 C CNN
 F 2 "" H 7550 3850 60  0000 C CNN
@@
 	5100 1400 4850 1400
 $Comp
-L Power_Port:DGND #PWR0104
+L Power_Port:DGND #PWR0213
 U 1 1 5BD344F6
 P 4200 1550
-F 0 "#PWR0104" H 4200 1380 50  0001 C CNN
+F 0 "#PWR0213" H 4200 1380 50  0001 C CNN
 F 1 "DGND" H 4200 1450 50  0000 C CNN
 F 2 "" H 4200 1650 60  0000 C CNN
@@
 	5100 1400 5100 2500
 $Comp
-L Resistors:RC0805JR-0710KL R214
+L Resistors:RC0805JR-0710KL R207
 U 1 1 5BD5F8F8
 P 4650 1400
-F 0 "R214" H 4650 1601 60  0000 C CNN
+F 0 "R207" H 4650 1601 60  0000 C CNN
 F 1 "RC0805JR-0710KL" H 4650 1100 50  0001 C CNN
 F 2 "Resistors:R0805" H 4650 500 30  0001 C CNN
