File: Master_Board/E10.1/V1/STM32F446.sch (KiCad schematic (older format))
At the start: 46 parts, among them J201 Header_Male_Pin_2.54mm_1X3_,_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, J202 Header_Male_Pin_2.54mm_1X6_,_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, SW201 PTS645SM43SMTR92, SW202 PTS645SM43SMTR92, U201 STM32F446RE

Commit message: add Vusb_sense
Connections:
- net labels removed: CAN1_RX, CAN1_TX
Changed lines of the file:
@@
 	1    0    0    -1
 $EndComp
-Text Label 7000 3200 0    60   ~ 0
-CAN1_TX
-Text Label 7000 3300 0    60   ~ 0
-CAN1_RX
 $Comp
 L Switches:PTS645SM43SMTR92 SW202
