File: Master_Board/E10.1/V1/USB.sch (KiCad schematic (older format))
At the start: 8 parts, among them J1001 61400416121

Commit message: add Vusb_sense
Parts:
- added D1002: B240AQ-13-F, Diodes:DO-214AC_SMA, symbol Diodes:B240AQ-13-F
- added Q1001: BSS806NH6327XTSA1, IC:SOT-23-3, symbol Transistors:BSS806NH6327XTSA1
- added R1004: RC0805JR-074K7L, Resistors:R0805, symbol Resistors:RC0805JR-074K7L
Connections:
- net labels added: 5V_EXT, USB_DETECT, VDD
- wire segments 40 -> 47
Changed lines of the file:
@@
 L Power_Port:5V #PWR01003
 U 1 1 5BDF1730
-P 7400 2450
-F 0 "#PWR01003" H 7400 2300 50  0001 C CNN
-F 1 "5V" H 7400 2624 50  0000 C CNN
-F 2 "" H 7400 2450 60  0000 C CNN
-F 3 "" H 7400 2450 60  0000 C CNN
-	1    7400 2450
+P 8400 2450
+F 0 "#PWR01003" H 8400 2300 50  0001 C CNN
+F 1 "5V" H 8400 2624 50  0000 C CNN
+F 2 "" H 8400 2450 60  0000 C CNN
+F 3 "" H 8400 2450 60  0000 C CNN
+	1    8400 2450
 	1    0    0    -1
 $EndComp
@@
 Connection ~ 5200 2600
 Wire Wire Line
-	6600 2600 7400 2600
-Wire Wire Line
-	7400 2600 7400 2450
+	8400 2600 8400 2450
 $Comp
 L Resistors:RC0805JR-070RL R1003
@@
 	0    -1   -1   0
 $EndComp
+$Comp
+L Diodes:B240AQ-13-F D1002
+U 1 1 5C098C05
+P 7550 2600
+F 0 "D1002" H 7500 2842 60  0000 C CNN
+F 1 "B240AQ-13-F" H 7500 2736 60  0000 C CNN
+F 2 "Diodes:DO-214AC_SMA" H 7550 1580 60  0001 C CNN
+F 3 "https://www.diodes.com/assets/Datasheets/ds13004.pdf" H 7550 1480 60  0001 C CNN
+F 4 "Digikey" H 7550 2080 60  0001 C CNN "Supplier"
+F 5 "B240AQ-13-FDICT-ND" H 7550 1980 60  0001 C CNN "Supplier Part Number"
+F 6 "Diode Incorporated" H 7550 1880 60  0001 C CNN "Manufacturer"
+F 7 "B240AQ-13-F" H 7550 1780 60  0001 C CNN "Manufacturer Part Number"
+F 8 "DIODE SCHOTTKY 40V 2A SMA" H 7550 1680 60  0001 C CNN "Description"
+	1    7550 2600
+	1    0    0    -1
+$EndComp
+Wire Wire Line
+	7650 2600 8400 2600
+Wire Wire Line
+	6600 2600 7350 2600
+Text Label 6800 2600 0    60   ~ 0
+5V_EXT
+Text Label 3700 5100 0    60   ~ 0
+5V_EXT
+$Comp
+L Transistors:BSS806NH6327XTSA1 Q1001
+U 1 1 5C09C1FD
+P 4300 5100
+F 0 "Q1001" H 4528 5153 60  0000 L CNN
+F 1 "BSS806NH6327XTSA1" H 4528 5047 60  0000 L CNN
+F 2 "IC:SOT-23-3" H 4450 4200 60  0001 C CNN
+F 3 "D" H 4450 4100 60  0001 C CNN
+F 4 "Digikey" H 4450 4700 60  0001 C CNN "Supplier"
+F 5 "BSS806NH6327XTSA1CT-ND" H 4450 4600 60  0001 C CNN "Supplier Part Number"
+F 6 "Infineon Technologies" H 4450 4500 60  0001 C CNN "Manufacturer"
+F 7 "BSS806NH6327XTSA1" H 4400 4400 60  0001 C CNN "Manufacturer Part Number"
+F 8 "MOSFET N-CH 20V 2.3A SOT23" H 4450 4300 60  0001 C CNN "Description"
+	1    4300 5100
+	1    0    0    -1
+$EndComp
+Wire Wire Line
+	4100 5100 3700 5100
+Wire Wire Line
+	4400 5400 4400 5500
+Wire Wire Line
+	4400 5500 5000 5500
+Wire Wire Line
+	4400 4800 4400 4700
+$Comp
+L Power_Port:VDD #PWR0107
+U 1 1 5C09DA3C
+P 4400 4700
+F 0 "#PWR0107" H 4400 4550 50  0001 C CNN
+F 1 "VDD" H 4400 4874 50  0000 C CNN
+F 2 "" H 4400 4700 60  0000 C CNN
+F 3 "" H 4400 4550 60  0000 C CNN
+	1    4400 4700
+	1    0    0    -1
+$EndComp
+$Comp
+L Resistors:RC0805JR-074K7L R1004
+U 1 1 5C09DB22
+P 4400 5800
+F 0 "R1004" V 4355 5858 60  0000 L CNN
+F 1 "RC0805JR-074K7L" H 4400 5500 50  0001 C CNN
+F 2 "Resistors:R0805" H 4400 4900 30  0001 C CNN
+F 3 "http://www.yageo.com/documents/recent/PYu-RC_Group_51_RoHS_L_7.pdf" H 4400 4850 30  0001 C CNN
+F 4 "Digikey" H 4400 5400 60  0001 C CNN "Supplier"
+F 5 "311-4.7KARCT-ND" H 4400 5300 60  0001 C CNN "Supplier Part Number"
+F 6 "Yageo" H 4400 5200 60  0001 C CNN "Manufacturer"
+F 7 "RC0805JR-074K7L" H 4400 5100 60  0001 C CNN "Manufacturer Part Number"
+F 8 "RES SMD 4.7K OHM 5% 1/8W 0805" H 4400 5000 60  0001 C CNN "Description"
+F 9 "4.7k" V 4453 5858 50  0000 L CNN "Resistance (Ohms)"
+F 10 "±5%" H 4600 5700 50  0001 C CNN "Tolerance (%)"
+F 11 "1/8W" H 4400 5660 50  0001 C CNN "Puissance (Watts)"
+	1    4400 5800
+	0    1    1    0
+$EndComp
+Wire Wire Line
+	4400 5600 4400 5500
+Connection ~ 4400 5500
+Wire Wire Line
+	4400 6000 4400 6100
+$Comp
+L Power_Port:DGND #PWR0108
+U 1 1 5C09FEE3
+P 4400 6200
+F 0 "#PWR0108" H 4400 6030 50  0001 C CNN
+F 1 "DGND" H 4400 6100 50  0000 C CNN
+F 2 "" H 4400 6300 60  0000 C CNN
+F 3 "" H 4380 6110 60  0000 C CNN
+	1    4400 6200
+	1    0    0    -1
+$EndComp
+Text HLabel 5000 5500 2    60   Output ~ 0
+USB_DETECT
 $EndSCHEMATC

Commit message: last minute change
Parts:
- removed J1001: 61400416121, Connectors:61400416121, symbol Connectors:61400416121
- added J1001: 61400413321, Connectors:61400413321, symbol Connectors:61400413321
Changed lines of the file:
@@
-	1    0    0    -1
-$EndComp
-$Comp
-L Connectors:61400416121 J1001
-U 1 1 5BB76F3B
-P 4000 3000
-F 0 "J1001" H 3850 3450 60  0000 C CNN
-F 1 "61400416121" H 3850 3350 60  0000 C CNN
-F 2 "Connectors:61400416121" H 4000 2100 60  0001 C CNN
-F 3 "https://media.digikey.com/pdf/Data%20Sheets/Wurth%20Electronics%20PDFs/Communication%20Conn%20WR-COM.pdf" H 4000 2000 60  0001 C CNN
-F 4 "Digikey" H 4000 2600 60  0001 C CNN "Supplier"
-F 5 "732-2108-ND" H 4000 2500 60  0001 C CNN "Supplier Part Number"
-F 6 "Wurth Electronics Inc." H 4000 2400 60  0001 C CNN "Manufacturer"
-F 7 "61400416121" H 4000 2300 60  0001 C CNN "Manufacturer Part Number"
-F 8 "CONN COM TYPE B USB HORZ 4POS" H 4000 2200 60  0001 C CNN "Description"
-	1    4000 3000
 	1    0    0    -1
 $EndComp
@@
 Text HLabel 5000 5500 2    60   Output ~ 0
 USB_DETECT
+$Comp
+L Connectors:61400413321 J1001
+U 1 1 5C40BE5F
+P 4000 3000
+F 0 "J1001" H 4000 3437 60  0000 C CNN
+F 1 "61400413321" H 4000 3331 60  0000 C CNN
+F 2 "Connectors:61400413321" H 4000 2100 60  0001 C CNN
+F 3 "https://katalog.we-online.com/em/datasheet/61400413321.pdf" H 4000 2000 60  0001 C CNN
+F 4 "Digikey" H 4000 2600 60  0001 C CNN "Supplier"
+F 5 "732-2734-ND" H 4000 2500 60  0001 C CNN "Supplier Part Number"
+F 6 "Wurth Electronics Inc." H 4000 2400 60  0001 C CNN "Manufacturer"
+F 7 "61400413321" H 4000 2300 60  0001 C CNN "Manufacturer Part Number"
+F 8 "CONN COM TYPE B USB HORZ 4POS" H 4000 2200 60  0001 C CNN "Description"
+	1    4000 3000
+	1    0    0    -1
+$EndComp
 $EndSCHEMATC
