File: Master_Board/E10.1/V2/VoltageSense.sch (KiCad schematic (older format))
At the start: 42 parts, among them U901 ACPL-C87A-500E, U902 NCS1S2405SC, U903 ACPL-C87A-500E, U904 CPC1117NTR, U905 LMV321RILT, U906 LMV321RILT

Commit message: Routing of the patch
Parts:
- gave numbers to parts that had none: 2
Changed lines of the file:
@@
 	2200 6100 3800 6100
 $Comp
-L Capacitors:885012207098 C?
+L Capacitors:885012207098 C917
 U 1 1 5C3B0325
 P 7950 1400
-F 0 "C?" H 7900 1648 60  0000 C CNN
+F 0 "C917" H 7900 1648 60  0000 C CNN
 F 1 "885012207098" H 7900 1050 60  0001 C CNN
 F 2 "Capacitors:C0805" H 7900 450 60  0001 C CNN
@@
 $EndComp
 $Comp
-L Capacitors:885012207098 C?
+L Capacitors:885012207098 C916
 U 1 1 5C3C9B58
 P 7900 4550
-F 0 "C?" H 7850 4798 60  0000 C CNN
+F 0 "C916" H 7850 4798 60  0000 C CNN
 F 1 "885012207098" H 7850 4200 60  0001 C CNN
 F 2 "Capacitors:C0805" H 7850 3600 60  0001 C CNN
@@
 	7300 1400 7300 1450
 $Comp
-L Power_Port:DGND #PWR?
+L Power_Port:DGND #PWR0109
 U 1 1 5C3E330F
 P 8200 1500
-F 0 "#PWR?" H 8200 1330 50  0001 C CNN
+F 0 "#PWR0109" H 8200 1330 50  0001 C CNN
 F 1 "DGND" H 8350 1450 50  0000 C CNN
 F 2 "" H 8200 1600 60  0000 C CNN
@@
 	8200 1400 8050 1400
 $Comp
-L Power_Port:DGND #PWR?
+L Power_Port:DGND #PWR0110
 U 1 1 5C3F4D71
 P 8150 4650
-F 0 "#PWR?" H 8150 4480 50  0001 C CNN
+F 0 "#PWR0110" H 8150 4480 50  0001 C CNN
 F 1 "DGND" H 8300 4600 50  0000 C CNN
 F 2 "" H 8150 4750 60  0000 C CNN

Commit message: Update repo
Parts:
- added D904, D905: D1213A-02SOL-7, IC:SOT-23-3, symbol Diodes:D1213A-02SOL-7
Connections:
- net DGND: now also D904.3 (GND), D905.3 (GND)
- net at R909.1, U903.7 (VOUT+): now also D905.1 (CH1)
- net at R910.1, U903.6 (VOUT-): now also D905.2 (CH2)
- net at R907.1, U901.7 (VOUT+): now also D904.1 (CH1)
- net at R908.1, U901.6 (VOUT-): now also D904.2 (CH2)
Changed lines of the file:
@@
 EESchema Schematic File Version 4
 LIBS:Master_Board-cache
-EELAYER 26 0
+EELAYER 29 0
 EELAYER END
 $Descr A4 11693 8268
@@
 F 7 "885012207098" H 5750 4000 60  0001 C CNN "Manufacturer Part Number"
 F 8 "CAP CER 0.1UF 50V X7R 0805" H 5750 3900 60  0001 C CNN "Description"
-F 9 "100nF" V 5750 4500 50  0000 C CNN "Capacitance (Farad)"
+F 9 "100nF" V 5750 4550 50  0000 C CNN "Capacitance (Farad)"
 F 10 "±10%" H 6010 4630 50  0001 C CNN "Tolerance (%)"
 F 11 "50V" H 5750 4560 50  0001 C CNN "Voltage Rated (Volt)"
@@
 F 7 "885012207098" H 5750 850 60  0001 C CNN "Manufacturer Part Number"
 F 8 "CAP CER 0.1UF 50V X7R 0805" H 5750 750 60  0001 C CNN "Description"
-F 9 "100nF" V 5750 1350 50  0000 C CNN "Capacitance (Farad)"
+F 9 "100nF" V 5750 1400 50  0000 C CNN "Capacitance (Farad)"
 F 10 "±10%" H 6010 1480 50  0001 C CNN "Tolerance (%)"
 F 11 "50V" H 5750 1410 50  0001 C CNN "Voltage Rated (Volt)"
@@
 	2650 3850 2650 4000
 Wire Wire Line
-	5650 4450 6200 4450
+	5650 4450 6150 4450
 Wire Wire Line
 	6600 4450 6700 4450
@@
 	7000 4450 7000 4700
 Wire Wire Line
-	5650 5150 6200 5150
+	5650 5150 5950 5150
 Wire Wire Line
 	6600 5150 6700 5150
@@
 	2650 700  2650 850
 Wire Wire Line
-	5650 1300 6200 1300
+	5650 1300 6150 1300
 Wire Wire Line
 	6600 1300 6700 1300
@@
 	7000 1300 7000 1550
 Wire Wire Line
-	5650 2000 6200 2000
+	5650 2000 5950 2000
 Wire Wire Line
 	6600 2000 6700 2000
@@
 Wire Wire Line
 	8150 4550 8000 4550
+$Comp
+L Diodes:D1213A-02SOL-7 D904
+U 1 1 5CD40D41
+P 6050 2350
+F 0 "D904" V 6300 2400 60  0000 L CNN
+F 1 "D1213A-02SOL-7" V 6400 2400 60  0000 L CNN
+F 2 "IC:SOT-23-3" H 6050 1330 60  0001 C CNN
+F 3 "https://www.diodes.com/assets/Datasheets/D1213A_02SOL.pdf" H 6050 1230 60  0001 C CNN
+F 4 "Digikey" H 6050 1830 60  0001 C CNN "Supplier"
+F 5 "D1213A-02SOL-7DICT-ND" H 6050 1730 60  0001 C CNN "Supplier Part Number"
+F 6 "Diodes Incorporated" H 6050 1630 60  0001 C CNN "Manufacturer"
+F 7 "D1213A-02SOL-7" H 6050 1530 60  0001 C CNN "Manufacturer Part Number"
+F 8 "TVS DIODE 3.3VWM 10VC SOT23" H 6050 1430 60  0001 C CNN "Description"
+	1    6050 2350
+	0    1    1    0
+$EndComp
+Wire Wire Line
+	6150 2050 6150 1300
+Connection ~ 6150 1300
+Wire Wire Line
+	6150 1300 6200 1300
+Wire Wire Line
+	5950 2050 5950 2000
+Connection ~ 5950 2000
+Wire Wire Line
+	5950 2000 6200 2000
+$Comp
+L Power_Port:DGND #PWR0111
+U 1 1 5CD5B24C
+P 6050 2800
+F 0 "#PWR0111" H 6050 2630 50  0001 C CNN
+F 1 "DGND" H 6050 2700 50  0000 C CNN
+F 2 "" H 6050 2900 60  0000 C CNN
+F 3 "" H 6030 2710 60  0000 C CNN
+	1    6050 2800
+	1    0    0    -1
+$EndComp
+Wire Wire Line
+	6050 2700 6050 2650
+$Comp
+L Diodes:D1213A-02SOL-7 D905
+U 1 1 5CD7A6E2
+P 6050 5500
+F 0 "D905" V 6200 5650 60  0000 L CNN
+F 1 "D1213A-02SOL-7" V 6300 5600 60  0000 L CNN
+F 2 "IC:SOT-23-3" H 6050 4480 60  0001 C CNN
+F 3 "https://www.diodes.com/assets/Datasheets/D1213A_02SOL.pdf" H 6050 4380 60  0001 C CNN
+F 4 "Digikey" H 6050 4980 60  0001 C CNN "Supplier"
+F 5 "D1213A-02SOL-7DICT-ND" H 6050 4880 60  0001 C CNN "Supplier Part Number"
+F 6 "Diodes Incorporated" H 6050 4780 60  0001 C CNN "Manufacturer"
+F 7 "D1213A-02SOL-7" H 6050 4680 60  0001 C CNN "Manufacturer Part Number"
+F 8 "TVS DIODE 3.3VWM 10VC SOT23" H 6050 4580 60  0001 C CNN "Description"
+	1    6050 5500
+	0    1    1    0
+$EndComp
+$Comp
+L Power_Port:DGND #PWR0112
+U 1 1 5CD7A6E8
+P 6050 5950
+F 0 "#PWR0112" H 6050 5780 50  0001 C CNN
+F 1 "DGND" H 6050 5850 50  0000 C CNN
+F 2 "" H 6050 6050 60  0000 C CNN
+F 3 "" H 6030 5860 60  0000 C CNN
+	1    6050 5950
+	1    0    0    -1
+$EndComp
+Wire Wire Line
+	6050 5850 6050 5800
+Wire Wire Line
+	6150 5200 6150 4450
+Connection ~ 6150 4450
+Wire Wire Line
+	6150 4450 6200 4450
+Wire Wire Line
+	5950 5200 5950 5150
+Connection ~ 5950 5150
+Wire Wire Line
+	5950 5150 6200 5150
 $EndSCHEMATC
