File: Master_Board/E10.1/V2/CAN1.sch (KiCad schematic (older format))
At the start: 15 parts, among them J401 649006227222, U401 SN65HVD232DR

Commit message: Modification after review of @gabChouin - Gabriel Chouinard
Other:
- note added: "To solder in E10.1 race package"
- note removed: "Solder only if needed"
Changed lines of the file:
@@
 Text Notes 4200 4875 0    60   ~ 0
 BUS TERMINATION
-Text Notes 4100 5400 0    60   ~ 0
-Solder only if needed
+Text Notes 3850 5450 0    60   ~ 0
+To solder in E10.1 race package
 Text Notes 7700 2700 0    60   ~ 0
 TVS and Capacitor need to be routed \nas close as possible to the connector
