File: Master_Board/E10.1/V3/ContactorControl.sch (KiCad schematic (older format))
At the start: 38 parts, among them J601 649004227222, J602 649004227222, J603 649004227222, J604 649004227222, J605 649002227222, Q601 BC849BLT1G, Q602 BC849BLT1G, Q603 BC849BLT1G, Q604 BC849BLT1G, Q605 BC849BLT1G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

Commit message: 2 new fuses added. PCB traces overhaul to support more current. Some small layout changes.
Parts:
- U601, U602, U603, U604, U605: symbol Isolators:TLP3543A(TP1,F -> Master_Board-rescue:TLP3543A(TP1,F-Isolators
- U606: symbol Isolators:CPC1117NTR -> Master_Board-rescue:CPC1117NTR-Isolators
Changed lines of the file:
@@
 EESchema Schematic File Version 4
 LIBS:Master_Board-cache
-EELAYER 29 0
+EELAYER 30 0
 EELAYER END
 $Descr A4 11693 8268
@@
 $EndComp
 $Comp
-L Isolators:CPC1117NTR U606
+L Master_Board-rescue:CPC1117NTR-Isolators U606
 U 1 1 5A88CE19
 P 9200 2350
@@
 Connection ~ 8800 1750
 $Comp
-L Isolators:TLP3543A(TP1,F U601
+L Master_Board-rescue:TLP3543A(TP1,F-Isolators U601
 U 1 1 5BC34945
 P 3450 1100
@@
 NoConn ~ 2950 1300
 $Comp
-L Isolators:TLP3543A(TP1,F U602
+L Master_Board-rescue:TLP3543A(TP1,F-Isolators U602
 U 1 1 5BC8294A
 P 3450 2400
@@
 $EndComp
 $Comp
-L Isolators:TLP3543A(TP1,F U603
+L Master_Board-rescue:TLP3543A(TP1,F-Isolators U603
 U 1 1 5BC863FC
 P 3450 3600
@@
 $EndComp
 $Comp
-L Isolators:TLP3543A(TP1,F U604
+L Master_Board-rescue:TLP3543A(TP1,F-Isolators U604
 U 1 1 5BC89EB4
 P 3450 5150
@@
 	5450 6300 5650 6300
 $Comp
-L Isolators:TLP3543A(TP1,F U605
+L Master_Board-rescue:TLP3543A(TP1,F-Isolators U605
 U 1 1 5BD4B22C
 P 3450 6650
