File: Master_Board/E10.1/V3/Master_Board.sch (KiCad schematic (older format))
At the start: 7 parts, among them J101 649002227222, J102 649002227222, J103 649002227222

Commit message: 2 new fuses added. PCB traces overhaul to support more current. Some small layout changes.
Parts:
- H101, H102, H103, H104: symbol Mechanicals:Mounting-Hole-M3 -> Master_Board-rescue:Mounting-Hole-M3-Mechanicals
Changed lines of the file:
@@
 EESchema Schematic File Version 4
 LIBS:Master_Board-cache
-EELAYER 29 0
+EELAYER 30 0
 EELAYER END
 $Descr USLetter 11000 8500
@@
 	7750 5000 9000 5000
 $Comp
-L Mechanicals:Mounting-Hole-M3 H104
+L Master_Board-rescue:Mounting-Hole-M3-Mechanicals H104
 U 1 1 5BD5CAFE
 P 4950 7250
@@
 $EndComp
 $Comp
-L Mechanicals:Mounting-Hole-M3 H103
+L Master_Board-rescue:Mounting-Hole-M3-Mechanicals H103
 U 1 1 5BD5CD8E
 P 4600 7250
@@
 $EndComp
 $Comp
-L Mechanicals:Mounting-Hole-M3 H102
+L Master_Board-rescue:Mounting-Hole-M3-Mechanicals H102
 U 1 1 5BD5CDD1
 P 4250 7250
@@
 $EndComp
 $Comp
-L Mechanicals:Mounting-Hole-M3 H101
+L Master_Board-rescue:Mounting-Hole-M3-Mechanicals H101
 U 1 1 5BD5CE2D
 P 3900 7250
