File: Master_Board/E10.1/V3/USB.sch (KiCad schematic (older format))
At the start: 11 parts, among them J1001 61400413321, Q1001 BSS806NH6327XTSA1

Commit message: 2 new fuses added. PCB traces overhaul to support more current. Some small layout changes.
Parts:
- FB1001: symbol Filter:742792605 -> Master_Board-rescue:742792605-Filter
- FL1001: symbol Filter:744230900 -> Master_Board-rescue:744230900-Filter
Changed lines of the file:
@@
 EESchema Schematic File Version 4
 LIBS:Master_Board-cache
-EELAYER 29 0
+EELAYER 30 0
 EELAYER END
 $Descr A4 11693 8268
@@
 $EndComp
 $Comp
-L Filter:744230900 FL1001
+L Master_Board-rescue:744230900-Filter FL1001
 U 1 1 5BBC3D6A
 P 6400 2950
@@
 	4250 2600 4300 2600
 $Comp
-L Filter:742792605 FB1001
+L Master_Board-rescue:742792605-Filter FB1001
 U 1 1 5BD3226B
 P 6400 2600
