File: Master_Board/E10.1/V3/VoltageSense.sch (KiCad schematic (older format))
At the start: 44 parts, among them U901 ACPL-C87A-500E, U902 NCS1S2405SC, U903 ACPL-C87A-500E, U904 CPC1117NTR, U905 LMV321RILT, U906 LMV321RILT

Commit message: 2 new fuses added. PCB traces overhaul to support more current. Some small layout changes.
Parts:
- U904: symbol Isolators:CPC1117NTR -> Master_Board-rescue:CPC1117NTR-Isolators
Changed lines of the file:
@@
 EESchema Schematic File Version 4
 LIBS:Master_Board-cache
-EELAYER 29 0
+EELAYER 30 0
 EELAYER END
 $Descr A4 11693 8268
@@
 	5600 3700 5450 3700
 $Comp
-L Isolators:CPC1117NTR U904
+L Master_Board-rescue:CPC1117NTR-Isolators U904
 U 1 1 5BC70C9E
 P 4900 6200
